Commit message: Fixed axis of kinect

File: urdf/kinect_v1/kinect.urdf.xacro (robot description, xacro)
@@ -1,36 +1,36 @@
 <?xml version="1.0"?>
 <robot xmlns:xacro="http://ros.org/wiki/xacro" >
-   <xacro:include filename="$(find sara_description)/urdf/kinect_v1/kinect.gazebo.xacro" />
-   <xacro:macro name="kinect2" params="name parent">
-       <xacro:kinect2_gazebo name="${name}" parent="${parent}"/>
-       <link name="${name}_link">
-         <visual>
-            <geometry>
-               <mesh filename="package://sara_description/meshes/kinect.STL" scale="0.001 0.001 0.001"/>
-            </geometry>
-            <origin xyz="-0.0269875 0.1321628 0" rpy="0 0 -1.5708"/>
-            <material name="black">
-               <color rgba="0.12 0.12 0.12 1"/>
-            </material>
-         </visual>
-         <collision>
-            <geometry>
-               <mesh filename="package://sara_description/meshes/kinect.STL" scale="0.001 0.001 0.001"/>
-            </geometry>
-            <origin xyz="-0.0269875 0.1321628 0" rpy="0 0 -1.5708"/>
-         </collision>
-         <inertial>
-            <mass value="10"/>
-            <origin xyz="0 0 0" rpy="1.5708 0 1.5708"/>
-            <inertia ixx="0.001" ixy="0" ixz="0" iyy="0.001" iyz="0" izz="0.001"/>
-         </inertial>
-     </link>
-     <joint name="${parent}_${name}_joint" type="fixed">
-         <parent link="${parent}_link"/>
-         <child link="${name}_link"/>
-         <limit effort="1000.0" lower="0" upper="0.5" velocity="0.2"/>
-         <origin xyz="0.177374 0 0.65676" rpy="0 0 0" />
-         <axis xyz="0 0 1" />
-    </joint>
-  </xacro:macro>
+  <xacro:include filename="$(find sara_description)/urdf/kinect_v1/kinect.gazebo.xacro" />
+  <xacro:macro name="kinect2" params="name parent">
+      <xacro:kinect2_gazebo name="${name}" parent="${parent}"/>
+      <link name="${name}_link">
+        <visual>
+           <geometry>
+              <mesh filename="package://sara_description/meshes/kinect.STL" scale="0.001 0.001 0.001"/>
+           </geometry>
+           <origin xyz="-0.13466 0 -0.028975" rpy="1.5708 0 0"/>
+           <material name="black">
+              <color rgba="0.12 0.12 0.12 1"/>
+           </material>
+        </visual>
+        <collision>
+           <geometry>
+              <mesh filename="package://sara_description/meshes/kinect.STL" scale="0.001 0.001 0.001"/>
+           </geometry>
+           <origin xyz="-0.0269875 0.1321628 0" rpy="0 0 -1.5708"/>
+        </collision>
+        <inertial>
+           <mass value="10"/>
+           <origin xyz="0 0 0" rpy="1.5708 0 1.5708"/>
+           <inertia ixx="0.001" ixy="0" ixz="0" iyy="0.001" iyz="0" izz="0.001"/>
+        </inertial>
+    </link>
+    <joint name="${parent}_${name}_joint" type="fixed">
+        <parent link="${parent}_link"/>
+        <child link="${name}_link"/>
+        <limit effort="1000.0" lower="0" upper="0.5" velocity="0.2"/>
+        <origin xyz="0.177374 0 0.65676" rpy="-1.5708 0 -1.5708" />
+        <axis xyz="0 0 1" />
+   </joint>
+ </xacro:macro>
 </robot>
