Commit message: launch file deplace dans sara_gazebo + ajout des coeficiens de friction des roues

File: urdf/wheels_v1/wheels.gazebo.xacro (robot description, xacro)
@@ -3,5 +3,11 @@
    <xacro:macro name="sara_wheels_gazebo_v1" params="name parent">
       <gazebo reference="${name}_link">
-         <gravity>false</gravity>
+      <mu1 value="1.0"/>
+      <mu2 value="1.0"/>
+      <kp value="1000000.0" />
+      <kd value="100.0" />
+      <fdir1 value="0 0 1"/>
+      <material>Gazebo/Orange</material>
+      <turnGravityOff>false</turnGravityOff>
       </gazebo>
    </xacro:macro>

Commit message: mu a zero

File: urdf/wheels_v1/wheels.gazebo.xacro (robot description, xacro)
@@ -3,11 +3,11 @@
    <xacro:macro name="sara_wheels_gazebo_v1" params="name parent">
       <gazebo reference="${name}_link">
-      <mu1 value="1.0"/>
-      <mu2 value="1.0"/>
-      <kp value="1000000.0" />
-      <kd value="100.0" />
-      <fdir1 value="0 0 1"/>
-      <material>Gazebo/Orange</material>
-      <turnGravityOff>false</turnGravityOff>
+        <mu1 value="0"/>
+        <mu2 value="0"/>
+        <kp value="0" />
+        <kd value="0" />
+        <fdir1 value="1 0 0"/>
+        <material>Gazebo/Orange</material>
+        <turnGravityOff>false</turnGravityOff>
       </gazebo>
    </xacro:macro>
