Commit message: WIP for gazebo + moveit

File: urdf/arm_v1/arm.gazebo.xacro (robot description, xacro)
@@ -1,23 +1,118 @@
 <?xml version="1.0"?>
 <robot xmlns:xacro="http://ros.org/wiki/xacro">
-   <xacro:macro name="sara_arm_gazebo_v1" params="name parent">
-       <gazebo reference="${name}_clavicular_link">
-         <gravity>false</gravity>
-       </gazebo>
-       <gazebo reference="$${name}_fix_upper_link">
-         <gravity>false</gravity>
-       </gazebo>
-       <gazebo reference="${name}_rot_upper_link">
-         <gravity>false</gravity>
-       </gazebo>
-       <gazebo reference="${name}_fix_lower_link">
-         <gravity>false</gravity>
-       </gazebo>
-       <gazebo reference="${name}_rot_lower_link">
-         <gravity>false</gravity>
-       </gazebo>
-       <gazebo reference="grasp_link">
-         <gravity>false</gravity>
-       </gazebo>
+  <xacro:macro name="sara_arm_gazebo_v1" params="name parent">
+    <transmission name="${parent}_${name}_trans" type="SimpleTransmission">
+      <type>transmission_interface/SimpleTransmission</type>
+      <actuator name="${parent}_${name}_motor">
+        <mechanicalReduction>1</mechanicalReduction>
+      </actuator>
+      <joint name="${parent}_${name}_joint">
+  	     <hardwareInterface>VelocityJointInterface</hardwareInterface>
+      </joint>
+    </transmission>
+    <gazebo reference="${name}_clavicular_link">
+        <turnGravityOff>false</turnGravityOff>
+    </gazebo>
+    <transmission name="${name}_shoulder_trans" type="SimpleTransmission">
+      <type>transmission_interface/SimpleTransmission</type>
+      <actuator name="${name}_shoulder_motor">
+  	     <mechanicalReduction>1</mechanicalReduction>
+      </actuator>
+      <joint name="${name}_shoulder_joint">
+      	 <hardwareInterface>VelocityJointInterface</hardwareInterface>
+      </joint>
+    </transmission>
+    <gazebo reference="$${name}_fix_upper_link">
+      <turnGravityOff>false</turnGravityOff>
+    </gazebo>
+    <transmission name="${name}_rot_elbow_trans" type="SimpleTransmission">
+      <type>transmission_interface/SimpleTransmission</type>
+      <actuator name="${name}_rot_elbow_motor">
+        <mechanicalReduction>1</mechanicalReduction>
+      </actuator>
+      <joint name="${name}_rot_elbow_joint">
+        <hardwareInterface>VelocityJointInterface</hardwareInterface>
+      </joint>
+    </transmission>
+    <gazebo reference="${name}_rot_upper_link">
+      <turnGravityOff>false</turnGravityOff>
+    </gazebo>
+    <transmission name="${name}_elbow_trans" type="SimpleTransmission">
+      <type>transmission_interface/SimpleTransmission</type>
+      <actuator name="${name}_elbow_motor">
+        <mechanicalReduction>1</mechanicalReduction>
+      </actuator>
+      <joint name="${name}_elbow_joint">
+        <hardwareInterface>VelocityJointInterface</hardwareInterface>
+      </joint>
+    </transmission>
+    <gazebo reference="${name}_fix_lower_link">
+      <turnGravityOff>false</turnGravityOff>
+    </gazebo>
+    <transmission name="${name}_rot_wrist_trans" type="SimpleTransmission">
+      <type>transmission_interface/SimpleTransmission</type>
+      <actuator name="${name}_rot_wrist_motor">
+   	 <mechanicalReduction>1</mechanicalReduction>
+      </actuator>
+      <joint name="${name}_rot_wrist_joint">
+      	 <hardwareInterface>VelocityJointInterface</hardwareInterface>
+      </joint>
+    </transmission>
+    <gazebo reference="${name}_rot_lower_link">
+      <turnGravityOff>false</turnGravityOff>
+    </gazebo>
+    <transmission name="${name}_forarm-wrist_trans" type="SimpleTransmission">
+      <type>transmission_interface/SimpleTransmission</type>
+      <actuator name="${name}_forarm-wrist_motor">
+      	 <mechanicalReduction>1</mechanicalReduction>
+      </actuator>
+      <joint name="${name}_forarm_wrist_joint">
+      	 <hardwareInterface>VelocityJointInterface</hardwareInterface>
+      </joint>
+    </transmission>
+    <gazebo reference="${name}_high_wrist_link">
+      <turnGravityOff>false</turnGravityOff>
+    </gazebo>
+    <transmission name="${name}_high_low_wrist_trans" type="SimpleTransmission">
+      <type>transmission_interface/SimpleTransmission</type>
+      <actuator name="${name}_high_low_wrist_motor">
+      	 <mechanicalReduction>1</mechanicalReduction>
+      </actuator>
+      <joint name="${name}_high_low_wrist_joint">
+      	 <hardwareInterface>VelocityJointInterface</hardwareInterface>
+      </joint>
+    </transmission>
+    <gazebo reference="${name}_low_wrist_link">
+      <turnGravityOff>false</turnGravityOff>
+    </gazebo>
+    <transmission name="${name}_low_wrist_grasp_socket_trans" type="SimpleTransmission">
+      <type>transmission_interface/SimpleTransmission</type>
+      <actuator name="${name}_low_wrist_grasp_socket_motor">
+      	 <mechanicalReduction>1</mechanicalReduction>
+      </actuator>
+      <joint name="${name}_low_wrist_grasp_socket_joint">
+      	 <hardwareInterface>VelocityJointInterface</hardwareInterface>
+      </joint>
+    </transmission>
+    <gazebo reference="${name}_socket_link">
+      <turnGravityOff>false</turnGravityOff>
+    </gazebo>
+    <transmission name="${name}_end_effector_trans" type="SimpleTransmission">
+      <type>transmission_interface/SimpleTransmission</type>
+      <actuator name="${name}_end_effector_motor">
+        <mechanicalReduction>1</mechanicalReduction>
+      </actuator>
+      <joint name="${name}_end_effector_joint">
+        <hardwareInterface>VelocityJointInterface</hardwareInterface>
+      </joint>
+    </transmission>
+    <gazebo reference="grasp_link">
+      <turnGravityOff>false</turnGravityOff>
+    </gazebo>
+    <gazebo>
+      <plugin name="gazebo_ros_control" filename="libgazebo_ros_control.so">
+        <robotNamespace>/</robotNamespace>
+      </plugin>
+    </gazebo>
   </xacro:macro>
 </robot>
