Commit message: WIP for gazebo + moveit

File: urdf/arm_v1/arm.urdf.xacro (robot description, xacro)
@@ -3,253 +3,247 @@
    <xacro:include filename="$(find sara_description)/urdf/arm_v1/arm.gazebo.xacro" />
    <xacro:macro name="sara_arm_v1" params="name parent end_effector">
-       <xacro:sara_arm_gazebo_v1 name="${name}" parent="${parent}"/>
-       <joint name="${parent}_${name}_joint" type="revolute">
-          <parent link="${parent}_link"/>
-          <child link="${name}_clavicular_link"/>
-          <limit effort="1000.0" lower="-0.18" upper="1.21" velocity="0.5"/>
-          <origin xyz="0 -0.145 0.189" rpy="0 -1.57 0" />
-          <axis xyz="0 0 1" />
-       </joint>
-       <!-- Link and joint to raise arm at shoulder level -->
-      <link name="${name}_clavicular_link">
-         <visual>
-            <geometry>
-               <mesh filename="package://sara_description/meshes/epaule.STL" scale="0.001 0.001 0.001"/>
-            </geometry>
-            <origin xyz="0 0 0" rpy="0 3.1416 0"/>
+     <xacro:sara_arm_gazebo_v1 name="${name}" parent="${parent}"/>
+     <joint name="${parent}_${name}_joint" type="revolute">
+       <parent link="${parent}_link"/>
+       <child link="${name}_clavicular_link"/>
+       <limit effort="1000.0" lower="-0.18" upper="1.21" velocity="0.5"/>
+       <origin xyz="0 -0.145 0.189" rpy="0 -1.57 0"/>
+       <axis xyz="0 0 1" />
+     </joint>
+     <link name="${name}_clavicular_link">
+       <visual>
+         <geometry>
+           <mesh filename="package://sara_description/meshes/epaule.STL" scale="0.001 0.001 0.001"/>
+           </geometry>
+           <origin xyz="0 0 0" rpy="0 3.1416 0"/>
+           <material name="black">
+             <color rgba="0.12 0.12 0.12 1"/>
+           </material>
+       </visual>
+       <collision>
+         <geometry>
+           <mesh filename="package://sara_description/meshes/epaule.STL" scale="0.001 0.001 0.001"/>
+         </geometry>
+           <origin xyz="0 0 0" rpy="0 3.1416 0"/>
+       </collision>
+       <inertial>
+         <mass value="1" />
+         <origin xyz="0 0 0" rpy="0 3.1416 0" />
+         <inertia ixx="0.001" ixy="0" ixz="0" iyy="0.001" iyz="0" izz="0.001" />
+       </inertial>
+     </link>
+     <joint name="${name}_shoulder_joint" type="revolute">
+       <parent link="${name}_clavicular_link"/>
+       <child link="${name}_fix_upper_link"/>
+       <limit effort="1000.0" lower="-3.29" upper="0.37" velocity="0.5"/>
+       <origin xyz="0 -0.085 0" rpy="-1.57 0 0" />
+       <axis xyz="0 0 1" />
+     </joint>
+     <link name="${name}_fix_upper_link">
+       <visual>
+         <geometry>
+           <mesh filename="package://sara_description/meshes/epaule.STL" scale="0.001 0.001 0.001"/>
+         </geometry>
+           <origin xyz="0 0 0" rpy="3.1416 0 1.5708"/>
+           <material name="black">
+             <color rgba="0.12 0.12 0.12 1"/>
+           </material>
+       </visual>
+       <collision>
+         <geometry>
+           <mesh filename="package://sara_description/meshes/epaule.STL" scale="0.001 0.001 0.001"/>
+         </geometry>
+           <origin xyz="0 0 0" rpy="3.1416 0 1.5708"/>
+         </collision>
+         <inertial>
+           <mass value="1" />
+           <origin xyz="0 0 0" rpy="3.1416 0 1.5708" />
+           <inertia ixx="0.001" ixy="0" ixz="0" iyy="0.001" iyz="0" izz="0.001" />
+         </inertial>
+     </link>
+     <joint name="${name}_rot_elbow_joint" type="revolute">
+       <parent link="${name}_fix_upper_link"/>
+       <child link="${name}_rot_upper_link"/>
+       <limit effort="1000.0" lower="-2.14" upper="1.00" velocity="0.5"/>
+       <origin xyz="-0.085 0 0" rpy="1.5708 0 1.5708" />
+       <axis xyz="0 0 1" />
+     </joint>
+     <link name="${name}_rot_upper_link">
+       <visual>
+         <geometry>
+           <mesh filename="package://sara_description/meshes/bras_haut.STL" scale="0.001 0.001 0.001"/>
+         </geometry>
+         <origin xyz="0 0 0" rpy="1.5708 3.1416 3.1416"/>
+         <material name="black">
+           <color rgba="0.12 0.12 0.12 1"/>
+         </material>
+       </visual>
+       <collision>
+         <geometry>
+           <mesh filename="package://sara_description/meshes/bras_haut.STL" scale="0.001 0.001 0.001"/>
+         </geometry>
+         <origin xyz="0 0 0" rpy="1.5708 3.1416 3.1416"/>
+       </collision>
+       <inertial>
+         <mass value="1" />
+         <origin xyz="0 0 0" rpy="1.5708 3.1416 3.1416" />
+         <inertia ixx="0.001" ixy="0" ixz="0" iyy="0.001" iyz="0" izz="0.001" />
+       </inertial>
+     </link>
+      <joint name="${name}_elbow_joint" type="revolute">
+        <parent link="${name}_rot_upper_link"/>
+        <child link="${name}_fix_lower_link"/>
+        <limit effort="1000.0" lower="-2.20" upper="1.90" velocity="0.5"/>
+        <origin xyz="0 0 -0.31" rpy="-1.5708 0 0" />
+        <axis xyz="0 0 1" />
+      </joint>
+      <link name="${name}_fix_lower_link">
+        <visual>
+          <geometry>
+            <mesh filename="package://sara_description/meshes/coude.STL" scale="0.001 0.001 0.001"/>
+          </geometry>
+            <origin xyz="0 0 -0.0005" rpy="3.1416 0 0"/>
             <material name="black">
-               <color rgba="0.12 0.12 0.12 1"/>
+              <color rgba="0.12 0.12 0.12 1"/>
             </material>
-         </visual>
-         <collision>
-            <geometry>
-               <mesh filename="package://sara_description/meshes/epaule.STL" scale="0.001 0.001 0.001"/>
-            </geometry>
-            <origin xyz="0 0 0" rpy="0 3.1416 0"/>
+        </visual>
+        <collision>
+          <geometry>
+            <mesh filename="package://sara_description/meshes/coude.STL" scale="0.001 0.001 0.001"/>
+          </geometry>
+          <origin xyz="0 0 -0.0005" rpy="3.1416 0 0"/>
         </collision>
         <inertial>
-            <mass value="1" />
-            <origin xyz="0 0 0" rpy="0 3.1416 0" />
-            <inertia ixx="0.001" ixy="0" ixz="0" iyy="0.001" iyz="0" izz="0.001" />
+          <mass value="1" />
+          <origin xyz="0 0 0" rpy="0 3.1416 0" />
+          <inertia ixx="0.001" ixy="0" ixz="0" iyy="0.001" iyz="0" izz="0.001" />
         </inertial>
       </link>
-      <joint name="${name}_shoulder_joint" type="revolute">
-         <parent link="${name}_clavicular_link"/>
-         <child link="${name}_fix_upper_link"/>
-         <limit effort="1000.0" lower="-3.29" upper="0.37" velocity="0.5"/>
-         <origin xyz="0 -0.085 0" rpy="-1.57 0 0" />
-         <axis xyz="0 0 1" />
-      </joint>
-      <!-- Link and joint to rotate the upper part of the arm at shoulder level -->
-      <link name="${name}_fix_upper_link">
-         <visual>
-            <geometry>
-               <mesh filename="package://sara_description/meshes/epaule.STL" scale="0.001 0.001 0.001"/>
-            </geometry>
-            <origin xyz="0 0 0" rpy="3.1416 0 1.5708"/>
-            <material name="black">
-               <color rgba="0.12 0.12 0.12 1"/>
-            </material>
-         </visual>
-         <collision>
-            <geometry>
-               <mesh filename="package://sara_description/meshes/epaule.STL" scale="0.001 0.001 0.001"/>
-            </geometry>
-            <origin xyz="0 0 0" rpy="3.1416 0 1.5708"/>
-         </collision>
-         <inertial>
-            <mass value="1" />
-            <origin xyz="0 0 0" rpy="3.1416 0 1.5708" />
-            <inertia ixx="0.001" ixy="0" ixz="0" iyy="0.001" iyz="0" izz="0.001" />
-        </inertial>
-      </link>
-      <joint name="${name}_rot_elbow_joint" type="revolute">
-         <parent link="${name}_fix_upper_link"/>
-         <child link="${name}_rot_upper_link"/>
-         <limit effort="1000.0" lower="-2.14" upper="1.00" velocity="0.5"/>
-         <origin xyz="-0.085 0 0" rpy="1.5708 0 1.5708" />
-         <axis xyz="0 0 1" />
-      </joint>
-      <!-- Link and joint to rotate the lower part of the arm at shoulder level -->
-      <link name="${name}_rot_upper_link">
-         <visual>
-            <geometry>
-               <mesh filename="package://sara_description/meshes/bras_haut.STL" scale="0.001 0.001 0.001"/>
-            </geometry>
-            <origin xyz="0 0 0" rpy="1.5708 3.1416 3.1416"/>
-            <material name="black">
-               <color rgba="0.12 0.12 0.12 1"/>
-            </material>
-         </visual>
-         <collision>
-            <geometry>
-               <mesh filename="package://sara_description/meshes/bras_haut.STL" scale="0.001 0.001 0.001"/>
-            </geometry>
-            <origin xyz="0 0 0" rpy="1.5708 3.1416 3.1416"/>
-         </collision>
-        <inertial>
-            <mass value="1" />
-            <origin xyz="0 0 0" rpy="1.5708 3.1416 3.1416" />
-            <inertia ixx="0.001" ixy="0" ixz="0" iyy="0.001" iyz="0" izz="0.001" />
-        </inertial>
-      </link>
-      <joint name="${name}_elbow_joint" type="revolute">
-         <parent link="${name}_rot_upper_link"/>
-         <child link="${name}_fix_lower_link"/>
-         <limit effort="1000.0" lower="-2.20" upper="1.90" velocity="0.5"/>
-         <origin xyz="0 0 -0.31" rpy="-1.5708 0 0" />
-         <axis xyz="0 0 1" />
-      </joint>
-       <!-- Link and joint to raise arm at elbow level -->
-      <link name="${name}_fix_lower_link">
-         <visual>
-            <geometry>
-               <mesh filename="package://sara_description/meshes/coude.STL" scale="0.001 0.001 0.001"/>
-            </geometry>
-            <origin xyz="0 0 -0.0005" rpy="3.1416 0 0"/>
-            <material name="black">
-               <color rgba="0.12 0.12 0.12 1"/>
-            </material>
-         </visual>
-         <collision>
-            <geometry>
-               <mesh filename="package://sara_description/meshes/coude.STL" scale="0.001 0.001 0.001"/>
-            </geometry>
-            <origin xyz="0 0 -0.0005" rpy="3.1416 0 0"/>
-         </collision>
-         <inertial>
-            <mass value="1" />
-            <origin xyz="0 0 0" rpy="0 3.1416 0" />
-            <inertia ixx="0.001" ixy="0" ixz="0" iyy="0.001" iyz="0" izz="0.001" />
-        </inertial>
-     </link>
      <joint name="${name}_rot_wrist_joint" type="revolute">
-        <parent link="${name}_fix_lower_link"/>
-        <child link="${name}_rot_lower_link"/>
-        <limit effort="1000.0" lower="-3.1416" upper="3.1416" velocity="0.5"/>
-        <origin xyz="0 0.0945 0" rpy="1.5708 -1.5708 0" />
-        <axis xyz="0 0 1" />
-    </joint>
-      <!-- Link and joint to rotate arm at elbow level -->
-      <link name="${name}_rot_lower_link">
-         <visual>
-            <geometry>
-               <mesh filename="package://sara_description/meshes/avant-bras.STL" scale="0.001 0.001 0.001"/>
-            </geometry>
-            <origin xyz="-0.0338 0.0338 0" rpy="-1.5708 0 -1.5708" />
-            <material name="black">
-               <color rgba="0.12 0.12 0.12 1"/>
-            </material>
-         </visual>
-         <collision>
-            <geometry>
-               <mesh filename="package://sara_description/meshes/avant-bras.STL" scale="0.001 0.001 0.001"/>
-            </geometry>
-            <origin xyz="-0.0338 0.0338 0" rpy="-1.5708 0 -1.5708" />
-         </collision>
-          <inertial>
-            <mass value="1" />
-            <origin xyz="-0.0676 0.0676 0" rpy="-1.5708 0 -1.5708" />
-            <inertia ixx="0.001" ixy="0" ixz="0" iyy="0.001" iyz="0" izz="0.001" />
-        </inertial>
-     </link>
-     <joint name="${name}_forarm-wrist_joint" type="fixed">
-        <parent link="${name}_rot_lower_link"/>
-        <child link="${name}_high_wrist_link"/>
-        <limit effort="1000.0" lower="-3.1416" upper="3.1416" velocity="0.5"/>
-        <origin xyz="0 0 -0.11184" rpy="1.5708 -1.5708 0" />
-        <axis xyz="0 1 0" />
-    </joint>
+       <parent link="${name}_fix_lower_link"/>
+       <child link="${name}_rot_lower_link"/>
+       <limit effort="1000.0" lower="-3.1416" upper="3.1416" velocity="0.5"/>
+       <origin xyz="0 0.0945 0" rpy="1.5708 -1.5708 0" />
+       <axis xyz="0 0 1" />
+     </joint>
+     <link name="${name}_rot_lower_link">
+       <visual>
+         <geometry>
+           <mesh filename="package://sara_description/meshes/avant-bras.STL" scale="0.001 0.001 0.001"/>
+         </geometry>
+         <origin xyz="-0.0338 0.0338 0" rpy="-1.5708 0 -1.5708" />
+           <material name="black">
+             <color rgba="0.12 0.12 0.12 1"/>
+           </material>
+       </visual>
+       <collision>
+         <geometry>
+           <mesh filename="package://sara_description/meshes/avant-bras.STL" scale="0.001 0.001 0.001"/>
+         </geometry>
+           <origin xyz="-0.0338 0.0338 0" rpy="-1.5708 0 -1.5708" />
+       </collision>
+       <inertial>
+         <mass value="1" />
+         <origin xyz="-0.0676 0.0676 0" rpy="-1.5708 0 -1.5708" />
+         <inertia ixx="0.001" ixy="0" ixz="0" iyy="0.001" iyz="0" izz="0.001" />
+       </inertial>
+     </link>
+     <joint name="${name}_forarm_wrist_joint" type="fixed">
+       <parent link="${name}_rot_lower_link"/>
+       <child link="${name}_high_wrist_link"/>
+       <limit effort="1000.0" lower="-3.1416" upper="3.1416" velocity="0.5"/>
+       <origin xyz="0 0 -0.11184" rpy="1.5708 -1.5708 0" />
+       <axis xyz="0 1 0" />
+     </joint>
      <link name="${name}_high_wrist_link">
-          <visual>
-              <geometry>
-                  <mesh filename="package://sara_description/meshes/poignet_haut.STL" scale="0.001 0.001 0.001"/>
-              </geometry>
-              <origin xyz="0.0706 0.0283 -0.030" rpy="1.5708 -1.5708 0"/>
-              <material name="black">
-              </material>
-              <color rgba="0 0 1 .06"/>
-          </visual>
-          <collision>
-             <geometry>
-                <mesh filename="package://sara_description/meshes/poignet_haut.STL" scale="0.001 0.001 0.001"/>
-             </geometry>
-             <origin xyz="0.0706 0.0283 -0.030" rpy="1.5708 -1.5708 0"/>
-          </collision>
+       <visual>
+         <geometry>
+           <mesh filename="package://sara_description/meshes/poignet_haut.STL" scale="0.001 0.001 0.001"/>
+         </geometry>
+         <origin xyz="0.0706 0.0283 -0.030" rpy="1.5708 -1.5708 0"/>
+         <material name="blue">
+           <color rgba="0 0 1 .06"/>
+         </material>
+       </visual>
+       <collision>
+         <geometry>
+           <mesh filename="package://sara_description/meshes/poignet_haut.STL" scale="0.001 0.001 0.001"/>
+         </geometry>
+         <origin xyz="0.0706 0.0283 -0.030" rpy="1.5708 -1.5708 0"/>
+       </collision>
      </link>
      <joint name="${name}_high_low_wrist_joint" type="revolute">
-        <parent link="${name}_high_wrist_link"/>
-        <child link="${name}_low_wrist_link"/>
-        <limit effort="1000.0" lower="-3.1416" upper="3.1416" velocity="0.5"/>
-        <origin xyz="0 0 0" rpy="1.5708 -1.5708 0" />
-        <axis xyz="0 0 1" />
-    </joint>
+       <parent link="${name}_high_wrist_link"/>
+       <child link="${name}_low_wrist_link"/>
+       <limit effort="1000.0" lower="-3.1416" upper="3.1416" velocity="0.5"/>
+       <origin xyz="0 0 0" rpy="1.5708 -1.5708 0" />
+       <axis xyz="0 0 1" />
+     </joint>
      <link name="${name}_low_wrist_link">
-          <visual>
-              <geometry>
-                  <mesh filename="package://sara_description/meshes/poignet_bas.STL" scale="0.001 0.001 0.001"/>
-              </geometry>
-              <origin xyz="-0.02575  -0.01375 0.0305448" rpy=" 0 1.5708 0"/>
-              <material name="black">
-                 <color rgba="0.12 0.12 0.12 1"/>
-              </material>
-          </visual>
-          <collision>
-             <geometry>
-                <mesh filename="package://sara_description/meshes/poignet_bas.STL" scale="0.001 0.001 0.001"/>
-             </geometry>
-             <origin xyz="-0.02575  -0.01375 0.0305448" rpy=" 0 1.5708 0"/>
-          </collision>
-     </link>
-          <joint name="${name}_low_wrist_grasp_socket_joint" type="revolute">
-             <parent link="${name}_low_wrist_link"/>
-             <child link="${name}_socket_link"/>
-             <limit effort="1000.0" lower="-3.1416" upper="3.1416" velocity="0.5"/>
-             <origin xyz="0 0.084375 0" rpy="1.5708 0 0" />
-             <axis xyz="1 0 0" />
-          </joint>
-      <link name="${name}_socket_link">
-      <visual>
-          <geometry>
-              <mesh filename="package://sara_description/meshes/attache-pince.STL" scale="0.001 0.001 0.001"/>
-          </geometry>
-          <origin xyz="0.028925 -0.025 -0.0362070" rpy="0 0 1.5708"/>
-          <material name="black">
-             <color rgba="0.12 0.12 0.12 1"/>
-          </material>
-      </visual>
-      <collision>
-         <geometry>
-            <mesh filename="package://sara_description/meshes/attache-pince.STL" scale="0.001 0.001 0.001"/>
+       <visual>
+         <geometry>
+           <mesh filename="package://sara_description/meshes/poignet_bas.STL" scale="0.001 0.001 0.001"/>
+         </geometry>
+         <origin xyz="-0.02575  -0.01375 0.0305448" rpy=" 0 1.5708 0"/>
+         <material name="black">
+           <color rgba="0.12 0.12 0.12 1"/>
+         </material>
+       </visual>
+       <collision>
+         <geometry>
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
File: urdf/base_v1/base.gazebo.xacro (robot description, xacro)
@@ -3,12 +3,12 @@
    <xacro:macro name="sara_base_gazebo_v1" params="name parent">
        <gazebo reference="{name}_link">
-         <gravity>false</gravity>
+         <turnGravityOff>false</turnGravityOff>
       </gazebo>
       <gazebo reference="spine_link">
-          <gravity>false</gravity>
+          <turnGravityOff>false</turnGravityOff>
       </gazebo>
       <!-- hokuyo -->
       <gazebo reference="lidar_link">
-         <gravity>false</gravity>
+         <turnGravityOff>false</turnGravityOff>
          <sensor type="ray" name="base_hokuyo_sensor">
             <pose>0 0 0 0 0 0</pose>

File: urdf/base_v1/base.urdf.xacro (robot description, xacro)
@@ -35,4 +35,18 @@
         <origin xyz="-0.055 0 0.227" rpy="0 0 0"/>
       </collision>
+      <inertial>
+        <mass value="100"/>
+        <origin xyz="-0.055 0 0.227" rpy="0 0 0"/>
+        <inertia ixx="0.1" ixy="0.1" ixz="0.1"
+                 iyy="0.1" iyz="0.1"
+                 izz="0.1"/>
+      </inertial>
+      <inertial>
+        <mass value="30"/>
+        <origin xyz="0 0 0" rpy="0 0 0"/>
+        <inertia ixx="0.1" ixy="0.1" ixz="0.1"
+                 iyy="0.1" iyz="0.1"
+                 izz="0.1"/>
+      </inertial>
     </link>
     <!-- Lidar -->

File: urdf/head_v1/head.gazebo.xacro (robot description, xacro)
@@ -3,11 +3,11 @@
    <xacro:macro name="sara_head_gazebo_v1" params="name parent">
       <gazebo reference="neck_dynamixel_link">
-         <gravity>false</gravity>
+         <turnGravityOff>false</turnGravityOff>
       </gazebo>
       <gazebo reference="head_link">
-         <gravity>false</gravity>
+         <turnGravityOff>false</turnGravityOff>
       </gazebo>
       <gazebo reference="camera_link">
-         <gravity>false</gravity>
+         <turnGravityOff>false</turnGravityOff>
          <sensor type="depth" name="camera">
             <visualize>true</visualize>

File: urdf/kinect_v1/kinect.gazebo.xacro (robot description, xacro)
@@ -3,5 +3,5 @@
    <xacro:macro name="kinect2_gazebo" params="name parent">
       <gazebo reference="${name}_link">
-         <gravity>false</gravity>
+         <turnGravityOff>false</turnGravityOff>
       </gazebo>
    </xacro:macro>

File: urdf/kinect_v1/kinect.urdf.xacro (robot description, xacro)
@@ -34,4 +34,3 @@
    </joint>
  </xacro:macro>
->>>>>>> ec39a350ad45b017363f201bf2bc936c8fdd3bdb
 </robot>

File: urdf/neck_v1/neck.gazebo.xacro (robot description, xacro)
@@ -3,5 +3,5 @@
    <xacro:macro name="sara_neck_gazebo_v1" params="name parent">
       <gazebo reference="${name}_link">
-         <gravity>false</gravity>
+         <turnGravityOff>false</turnGravityOff>
       </gazebo>
    </xacro:macro>

File: urdf/robotiq_c2_model/robotiq_c2_model.gazebo.xacro (robot description, xacro)
@@ -3,30 +3,30 @@
    <xacro:macro name="robotiq_c2_model_gazebo" params="prefix">
       <gazebo reference="${prefix}robotiq_85_base_link">
-         <gravity>false</gravity>
+         <turnGravityOff>false</turnGravityOff>
       </gazebo>
       <gazebo reference="${prefix}robotiq_85_left_knuckle_link">
-         <gravity>false</gravity>
+         <turnGravityOff>false</turnGravityOff>
       </gazebo>
       <gazebo reference="${prefix}robotiq_85_right_knuckle_link">
-         <gravity>false</gravity>
+         <turnGravityOff>false</turnGravityOff>
       </gazebo>
       <gazebo reference="${prefix}robotiq_85_left_finger_link">
-         <gravity>false</gravity>
+         <turnGravityOff>false</turnGravityOff>
       </gazebo>
       <gazebo reference="${prefix}robotiq_85_right_finger_link">
-         <gravity>false</gravity>
+         <turnGravityOff>false</turnGravityOff>
       </gazebo>
       <gazebo reference="${prefix}robotiq_85_left_inner_knuckle_link">
-         <gravity>false</gravity>
+         <turnGravityOff>false</turnGravityOff>
       </gazebo>
       <gazebo reference="${prefix}robotiq_85_right_inner_knuckle_link">
-         <gravity>false</gravity>
+         <turnGravityOff>false</turnGravityOff>
       </gazebo>
       <gazebo reference="${prefix}robotiq_85_left_finger_tip_link">
-         <gravity>false</gravity>
+         <turnGravityOff>false</turnGravityOff>
       </gazebo>
       <gazebo reference="${prefix}robotiq_85_right_finger_tip_link">
-         <gravity>false</gravity>
+         <turnGravityOff>false</turnGravityOff>
       </gazebo>
-</xacro:macro>
+   </xacro:macro>
 </robot>

File: urdf/torso_v1/torso.gazebo.xacro (robot description, xacro)
@@ -3,5 +3,5 @@
    <xacro:macro name="sara_torso_gazebo_v1" params="name parent">
       <gazebo reference="${name}_link">
-         <gravity>false</gravity>
+         <turnGravityOff>false</turnGravityOff>
       </gazebo>
    </xacro:macro>
