Commit message: fix arm urdf for moveit

File: urdf/arm_v1/arm.gazebo.xacro (robot description, xacro)
@@ -62,13 +62,4 @@
       <turnGravityOff>false</turnGravityOff>
     </gazebo>
-    <transmission name="${name}_forarm-wrist_trans" type="SimpleTransmission">
-      <type>transmission_interface/SimpleTransmission</type>
-      <actuator name="${name}_forarm-wrist_motor">
-      	 <mechanicalReduction>1</mechanicalReduction>
-      </actuator>
-      <joint name="${name}_forarm_wrist_joint">
-      	 <hardwareInterface>VelocityJointInterface</hardwareInterface>
-      </joint>
-    </transmission>
     <gazebo reference="${name}_high_wrist_link">
       <turnGravityOff>false</turnGravityOff>
@@ -98,13 +89,4 @@
       <turnGravityOff>false</turnGravityOff>
     </gazebo>
-    <transmission name="${name}_end_effector_trans" type="SimpleTransmission">
-      <type>transmission_interface/SimpleTransmission</type>
-      <actuator name="${name}_end_effector_motor">
-        <mechanicalReduction>1</mechanicalReduction>
-      </actuator>
-      <joint name="${name}_end_effector_joint">
-        <hardwareInterface>VelocityJointInterface</hardwareInterface>
-      </joint>
-    </transmission>
     <gazebo reference="grasp_link">
       <turnGravityOff>false</turnGravityOff>

File: urdf/arm_v1/arm.urdf.xacro (robot description, xacro)
@@ -172,4 +172,9 @@
          <origin xyz="0.0706 0.0283 -0.030" rpy="1.5708 -1.5708 0"/>
        </collision>
+       <inertial>
+         <mass value="1" />
+         <origin xyz="-0.0676 0.0676 0" rpy="-1.5708 0 -1.5708" />
+         <inertia ixx="0.001" ixy="0" ixz="0" iyy="0.001" iyz="0" izz="0.001" />
+       </inertial>
      </link>
      <joint name="${name}_high_low_wrist_joint" type="revolute">
@@ -196,4 +201,9 @@
          <origin xyz="-0.02575  -0.01375 0.0305448" rpy=" 0 1.5708 0"/>
        </collision>
+       <inertial>
+         <mass value="1" />
+         <origin xyz="-0.0676 0.0676 0" rpy="-1.5708 0 -1.5708" />
+         <inertia ixx="0.001" ixy="0" ixz="0" iyy="0.001" iyz="0" izz="0.001" />
+       </inertial>
      </link>
      <joint name="${name}_low_wrist_grasp_socket_joint" type="revolute">
@@ -220,4 +230,9 @@
          <origin xyz="0.028925 -0.025 -0.0362070" rpy="0 0 1.5708"/>
        </collision>
+       <inertial>
+         <mass value="1" />
+         <origin xyz="-0.0676 0.0676 0" rpy="-1.5708 0 -1.5708" />
+         <inertia ixx="0.001" ixy="0" ixz="0" iyy="0.001" iyz="0" izz="0.001" />
+       </inertial>
      </link>
      <joint name="${name}_end_effector_joint" type="fixed">

File: urdf/kinect_v1/kinect.urdf.xacro (robot description, xacro)
@@ -18,9 +18,9 @@
               <mesh filename="package://sara_description/meshes/kinect.STL" scale="0.001 0.001 0.001"/>
            </geometry>
-           <origin xyz="-0.0269875 0.1321628 0" rpy="0 0 -1.5708"/>
+           <origin xyz="-0.0269875 0.1321628 0" rpy="1.5708 0 0"/>
         </collision>
         <inertial>
            <mass value="10"/>
-           <origin xyz="0 0 0" rpy="1.5708 0 1.5708"/>
+           <origin xyz="0 0 0" rpy="1.5708 0 0"/>
            <inertia ixx="0.001" ixy="0" ixz="0" iyy="0.001" iyz="0" izz="0.001"/>
         </inertial>
