Commit message: Fix joint limits

File: urdf/arm_v1/arm.urdf.xacro (robot description, xacro)
@@ -7,5 +7,5 @@
        <parent link="${parent}_link"/>
        <child link="${name}_clavicular_link"/>
-       <limit effort="1000.0" lower="-0.18" upper="1.21" velocity="0.5"/>
+       <limit effort="1000.0" lower="-1.6" upper="1.4" velocity="0.5"/>
        <origin xyz="0 -0.145 0.189" rpy="0 -1.57 0"/>
        <axis xyz="0 0 1" />
@@ -36,5 +36,5 @@
        <parent link="${name}_clavicular_link"/>
        <child link="${name}_fix_upper_link"/>
-       <limit effort="1000.0" lower="-3.29" upper="0.37" velocity="0.5"/>
+       <limit effort="1000.0" lower="-4.7124" upper="1.5708" velocity="0.5"/>
        <origin xyz="0 -0.085 0" rpy="-1.57 0 0" />
        <axis xyz="0 0 1" />
@@ -65,5 +65,5 @@
        <parent link="${name}_fix_upper_link"/>
        <child link="${name}_rot_upper_link"/>
-       <limit effort="1000.0" lower="-2.14" upper="1.00" velocity="0.5"/>
+       <limit effort="1000.0" lower="-3.1416" upper="3.1416" velocity="0.5"/>
        <origin xyz="-0.085 0 0" rpy="1.5708 0 1.5708" />
        <axis xyz="0 0 1" />
@@ -176,5 +176,5 @@
        <parent link="${name}_high_wrist_link"/>
        <child link="${name}_low_wrist_link"/>
-       <limit effort="1000.0" lower="-3.1416" upper="3.1416" velocity="0.5"/>
+       <limit effort="1000.0" lower="-1.5708" upper="1.5708" velocity="0.5"/>
        <origin xyz="0 0 0" rpy="1.5708 -1.5708 0" />
        <axis xyz="0 0 1" />
@@ -200,5 +200,5 @@
        <parent link="${name}_low_wrist_link"/>
        <child link="${name}_socket_link"/>
-       <limit effort="1000.0" lower="-3.1416" upper="3.1416" velocity="0.5"/>
+       <limit effort="1000.0" lower="-1.49" upper="1.49" velocity="0.5"/>
        <origin xyz="0 0.084375 0" rpy="1.5708 0 0" />
        <axis xyz="1 0 0" />

Commit message: Removed gripper from sara_description, change urdf of the arm to fit both gripper

File: urdf/arm_v1/arm.urdf.xacro (robot description, xacro)
@@ -2,5 +2,5 @@
 <robot xmlns:xacro="http://ros.org/wiki/xacro" >
    <xacro:include filename="$(find sara_description)/urdf/arm_v1/arm.gazebo.xacro" />
-   <xacro:macro name="sara_arm_v1" params="name parent end_effector">
+   <xacro:macro name="sara_arm_v1" params="name parent">
      <xacro:sara_arm_gazebo_v1 name="${name}" parent="${parent}"/>
      <joint name="${parent}_${name}_joint" type="revolute">
@@ -236,29 +236,4 @@
        </inertial>
      </link>
-     <joint name="${name}_end_effector_joint" type="fixed">
-       <parent link="${name}_socket_link"/>
-       <child link="${end_effector}_link"/>
-       <limit effort="1000.0" lower="-0.26" upper="0.26" velocity="0.5" />
-       <axis xyz="0 1 0"/>
-       <origin xyz="0 0 -0.02989" rpy="0 1.5708 0"/>
-     </joint>
-     <link name="grasp_link" >
-       <visual>
-         <geometry>
-           <sphere radius="0.01" />
-         </geometry>
-         <origin xyz="0 0.05 0" rpy="0 0 0" />
-       </visual>
-       <inertial>
-         <mass value="0" />
-         <origin xyz="0 0 0" rpy="0 0 0" />
-         <inertia ixx="0.001" ixy="0" ixz="0" iyy="0.001" iyz="0" izz="0.001" />
-       </inertial>
-     </link>
-     <joint name="grasp_joint" type="fixed" >
-       <parent link="${end_effector}_link" />
-       <child link="grasp_link" />
-       <origin xyz="0.075 0 -0.012" rpy="3.1416 0 1.5708" />
-     </joint>
    </xacro:macro>
 </robot>

File: urdf/sara.urdf.xacro (robot description, xacro)
@@ -6,8 +6,9 @@
     <xacro:include filename="$(find sara_description)/urdf/kinect_v1/kinect.urdf.xacro"/>
     <xacro:include filename="$(find sara_description)/urdf/head_v1/head.urdf.xacro"/>
-    <xacro:include filename="$(find sara_description)/urdf/robotiq_c2_model/robotiq_c2_model_macro.xacro"/>
     <xacro:include filename="$(find sara_description)/urdf/arm_v1/arm.urdf.xacro"/>
     <xacro:include filename="$(find sara_description)/urdf/base_v1/base.urdf.xacro"/>
     <xacro:include filename="$(find sara_description)/urdf/wheels_v1/wheels.urdf.xacro"/>
+    <xacro:include filename="$(find robotiq_85_description)/urdf/robotiq_85_gripper.urdf.xacro"/>
+    <xacro:include filename="$(find robotiq_c2_model_visualization)/urdf/robotiq_c2_model_macro.xacro"/>
     <!-- Base -->
     <xacro:sara_base_v1 name="base" parent=""/>
@@ -23,6 +24,13 @@
     <xacro:sara_head_v1 name="head" parent="neck"/>
     <!-- Arm -->
-    <xacro:sara_arm_v1 name="arm" parent="torso" end_effector="robotiq_85_base"/>
-    <!-- End Effector -->
-    <xacro:robotiq_c2_model prefix=""/>
+    <xacro:sara_arm_v1 name="arm" parent="torso"/>
+    <!-- Gripper 85 (new)
+    <xacro:robotiq_85_gripper prefix="" parent="arm_socket_link">
+      <origin xyz="0 0 -0.02989" rpy="0 1.5708 0"/>
+    </xacro:robotiq_85_gripper>
+    -->
+    <!-- Gripper C2 (old)-->
+    <xacro:robotiq_c2_model prefix="" parent="arm_socket_link">
+      <origin xyz="0 0 -0.02989" rpy="0 1.5708 0"/>
+    </xacro:robotiq_c2_model>
 </robot>
