Commit message: fix lidar z, fix kinect colision

File: urdf/base_v1/base.gazebo.xacro (robot description, xacro)
@@ -12,5 +12,5 @@
          <turnGravityOff>false</turnGravityOff>
          <sensor type="ray" name="base_hokuyo_sensor">
-            <pose>0 0 0 0 0 0</pose>
+            <pose>0 0 0 0 0 0.0425</pose>
             <visualize>true</visualize>
             <update_rate>30</update_rate>

File: urdf/base_v1/base.urdf.xacro (robot description, xacro)
@@ -56,5 +56,5 @@
           <cylinder length="0.085" radius="0.03"/>
         </geometry>
-        <origin xyz="0 0 0.0425" rpy="0 0 0"/>
+        <origin xyz="0 0 0" rpy="0 0 0"/>
         <material name="orange">
           <color rgba="1 0.5 0 1"/>
@@ -76,5 +76,5 @@
       <parent link="base_link"/>
       <child link="lidar_link"/>
-      <origin xyz="0.2516879 0 -0.0288348" rpy="0 0 0" />
+      <origin xyz="0.2516879 0 0" rpy="0 0 0" />
     </joint>
     </xacro:macro>

File: urdf/kinect_v1/kinect.urdf.xacro (robot description, xacro)
@@ -18,9 +18,9 @@
               <mesh filename="package://sara_description/meshes/kinect.STL" scale="0.001 0.001 0.001"/>
            </geometry>
-           <origin xyz="-0.0269875 0.1321628 0" rpy="1.5708 0 0"/>
+           <origin xyz="-0.13466 0 -0.028975" rpy="1.5708 0 0"/>
         </collision>
         <inertial>
            <mass value="10"/>
-           <origin xyz="0 0 0" rpy="1.5708 0 0"/>
+           <origin xyz="-0.13466 0 -0.028975" rpy="1.5708 0 0"/>
            <inertia ixx="0.001" ixy="0" ixz="0" iyy="0.001" iyz="0" izz="0.001"/>
         </inertial>
