Commit message: Remove kinect2

File: urdf/sara.urdf (robot description, URDF)
Before this commit: robot sara, 32 links, 31 joints
Links:
- removed link kinect2_link
- removed link right_lower_wrist_link
- removed link right_upper_wrist_link
- added link right_wrist_lower_link, mass 0.18747684; collision mesh filename=package://sara_description/meshes/poignet_bas.STL scale=0.001 0.001 0.001; visual mesh filename=package://sara_description/meshes/poignet_bas.STL scale=0.001 0.001 0.001
- added link right_wrist_upper_link, mass 0.1956991; collision mesh filename=package://sara_description/meshes/poignet_haut.STL scale=0.001 0.001 0.001; visual mesh filename=package://sara_description/meshes/poignet_haut.STL scale=0.001 0.001 0.001
- link base_link: mass 100 -> 40
- link head_link: mass 5 -> 2.60401968
- link head_xtion_link: geometry visual mesh filename=package://sara_description/meshes/xtion.STL scale=0.001 0.001 0.001
- link right_clavicular_link: mass 1 -> 0.28506911; geometry collision mesh filename=package://sara_description/meshes/epaule1.STL scale=0.001 0.001 0.001; visual mesh filename=package://sara_description/meshes/epaule1.STL scale=0.001 0.001 0.001
- link right_forearm_lower_link: mass 1 -> 0.1177; geometry collision mesh filename=package://sara_description/meshes/avant_bras.STL scale=0.001 0.001 0.001; visual mesh filename=package://sara_description/meshes/avant_bras.STL scale=0.001 0.001 0.001
- link right_forearm_upper_link: mass 1 -> 0.28300045
- link right_robotiq_85_base_link: geometry collision mesh filename=package://robotiq_c2_description/meshes/robotiq_c2/collisio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; visual mesh filename=package://robotiq_c2_description/meshes/robotiq_c2/visual/r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
- link right_robotiq_85_left_finger_link: geometry collision mesh filename=package://robotiq_c2_description/meshes/robotiq_c2/collisio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; visual mesh filename=package://robotiq_c2_description/meshes/robotiq_c2/visual/r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
- link right_robotiq_85_left_finger_tip_link: geometry collision mesh filename=package://robotiq_c2_description/meshes/robotiq_c2/collisio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; visual mesh filename=package://robotiq_c2_description/meshes/robotiq_c2/visual/r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
- link right_robotiq_85_left_inner_knuckle_link: geometry collision mesh filename=package://robotiq_c2_description/meshes/robotiq_c2/collisio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; visual mesh filename=package://robotiq_c2_description/meshes/robotiq_c2/visual/r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
- link right_robotiq_85_left_knuckle_link: geometry collision mesh filename=package://robotiq_c2_description/meshes/robotiq_c2/collisio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; visual mesh filename=package://robotiq_c2_description/meshes/robotiq_c2/visual/r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
- link right_robotiq_85_right_finger_link: geometry collision mesh filename=package://robotiq_c2_description/meshes/robotiq_c2/collisio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; visual mesh filename=package://robotiq_c2_description/meshes/robotiq_c2/visual/r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
- link right_robotiq_85_right_finger_tip_link: geometry collision mesh filename=package://robotiq_c2_description/meshes/robotiq_c2/collisio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; visual mesh filename=package://robotiq_c2_description/meshes/robotiq_c2/visual/r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
- link right_robotiq_85_right_inner_knuckle_link: geometry collision mesh filename=package://robotiq_c2_description/meshes/robotiq_c2/collisio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; visual mesh filename=package://robotiq_c2_description/meshes/robotiq_c2/visual/r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
- link right_robotiq_85_right_knuckle_link: geometry collision mesh filename=package://robotiq_c2_description/meshes/robotiq_c2/collisio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; visual mesh filename=package://robotiq_c2_description/meshes/robotiq_c2/visual/r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
- link right_socket_link: mass 1 -> 0.02796; geometry collision mesh filename=package://sara_description/meshes/attache_pince.STL scale=0.001 0.001 0.001; visual mesh filename=package://sara_description/meshes/attache_pince.STL scale=0.001 0.001 0.001
- link right_upper_arm_lower_link: mass 1 -> 0.85240803
- link right_upper_arm_upper_link: mass 1 -> 0.28506911; geometry collision mesh filename=package://sara_description/meshes/epaule2.STL scale=0.001 0.001 0.001; visual mesh filename=package://sara_description/meshes/epaule2.STL scale=0.001 0.001 0.001
- link torso_link: mass 10 -> 4.17008957
Joints:
- removed joint base_kinect2_joint
- removed joint right_wrist_yaw_joint
- added joint right_wrist_roll_joint: type revolute, parent right_wrist_lower_link, child right_socket_link, origin xyz=0 0.084375 0 rpy=1.5708 0 0, axis 1 0 0, limit lower=-1.49 upper=1.49 effort=10000.0 velocity=0.5
- joint right_elbow_pitch_joint: limit lower=-2.20 upper=1.90 effort=1000.0 velocity=0.5 -> lower=-2.20 upper=1.90 effort=10000.0 velocity=0.5
- joint right_elbow_yaw_joint: limit lower=-3.1416 upper=3.1416 effort=1000.0 velocity=0.5 -> lower=-3.1416 upper=3.1416 effort=10000.0 velocity=0.5
- joint right_shoulder_pitch_joint: limit lower=-4.7124 upper=1.5708 effort=1000.0 velocity=0.5 -> lower=-4.7124 upper=1.5708 effort=10000.0 velocity=0.5
- joint right_shoulder_roll_joint: limit lower=-1.6 upper=1.4 effort=1000.0 velocity=0.5 -> lower=-1.6 upper=1.4 effort=10000.0 velocity=0.5
- joint right_shoulder_yaw_joint: limit lower=-3.1416 upper=3.1416 effort=1000.0 velocity=0.5 -> lower=-3.1416 upper=3.1416 effort=10000.0 velocity=0.5
- joint right_wrist_joint: child right_upper_wrist_link -> right_wrist_upper_link; limit lower=-3.1416 upper=3.1416 effort=1000.0 velocity=0.5 -> lower=-3.1416 upper=3.1416 effort=10000.0 velocity=0.5; origin xyz=0 0 -0.11184 rpy=1.5708 -1.5708 0 -> xyz=0 0 -0.05124 rpy=1.5708 -1.5708 0
- joint right_wrist_pitch_joint: child right_lower_wrist_link -> right_wrist_lower_link; limit lower=-1.5708 upper=1.5708 effort=1000.0 velocity=0.5 -> lower=-1.5708 upper=1.5708 effort=10000.0 velocity=0.5; origin xyz=0 0 0 rpy=1.5708 -1.5708 0 -> xyz=-0.0606 0 0 rpy=1.5708 -1.5708 0; parent right_upper_wrist_link -> right_wrist_upper_link

File: urdf/sara.urdf.xacro (robot description, xacro)
@@ -6,5 +6,4 @@
     <xacro:include filename="$(find sara_description)/urdf/torso_v1/torso.urdf.xacro"/>
     <xacro:include filename="$(find sara_description)/urdf/neck_v1/neck.urdf.xacro"/>
-    <xacro:include filename="$(find sara_description)/urdf/kinect2/kinect2.urdf.xacro"/>
     <xacro:include filename="$(find sara_description)/urdf/xtion/xtion.urdf.xacro"/>
     <xacro:include filename="$(find sara_description)/urdf/head_v1/head.urdf.xacro"/>
@@ -29,8 +28,4 @@
         <origin xyz="0.177374 0 0.70531" rpy="0 0 0" />
     </xacro:sara_torso_v1>
-    <!-- Torso Kinect -->
-    <xacro:kinect2 prefix="torso_" parent="base" sim="${sim}">
-        <origin xyz="0.177374 0 0.65676" rpy="-1.5708 0 -1.5708" />
-    </xacro:kinect2>
     <!-- Neck -->
     <xacro:sara_neck_v1 parent="torso" sim="${sim}">
