Commit message: new folder for head_xtion

File: urdf/head_xtion/head_xtion.urdf.xacro (robot description, xacro)
@@ -4,5 +4,5 @@
     <xacro:macro name="asus_xtion" params="prefix parent *origin sim">
         <xacro:if value="${sim}">
-            <xacro:include filename="$(find sara_description)/urdf/xtion/xtion.gazebo.xacro" />
+            <xacro:include filename="$(find sara_description)/urdf/head_xtion/head_xtion.gazebo.xacro" />
             <xacro:xtion_gazebo prefix="${prefix}"/>
         </xacro:if>
@@ -21,5 +21,5 @@
           <origin xyz="0 0 0" rpy="0 0 0" />
           <geometry>
-              <mesh filename="package://sara_description/meshes/xtion.STL" scale="0.001 0.001 0.001"/>
+              <mesh filename="package://sara_description/meshes/head_xtion.STL" scale="0.001 0.001 0.001"/>
           </geometry>
         </visual>

File: urdf/sara.urdf.xacro (robot description, xacro)
@@ -7,5 +7,5 @@
     <xacro:include filename="$(find sara_description)/urdf/neck_v1/neck.urdf.xacro"/>
     <xacro:include filename="$(find sara_description)/urdf/kinect2/kinect2.urdf.xacro"/>
-    <xacro:include filename="$(find sara_description)/urdf/xtion/xtion.urdf.xacro"/>
+    <xacro:include filename="$(find sara_description)/urdf/head_xtion/head_xtion.urdf.xacro"/>
     <xacro:include filename="$(find sara_description)/urdf/head_v1/head.urdf.xacro"/>
     <xacro:include filename="$(find sara_description)/urdf/arm_v2/arm.urdf.xacro"/>
