Commit message: Referentials for arm_xtion are good

File: urdf/arm_xtion/arm_xtion.gazebo.xacro (robot description, xacro)
@@ -9,5 +9,5 @@
       <link name="${prefix}xtion_depth_frame"/>
       <joint name="${prefix}xtion_depth_optical_joint" type="fixed">
-         <origin xyz="0 0 0" rpy="${-M_PI/2} 0.0 ${-M_PI/2}" />
+         <origin xyz="0 0 0" rpy="0 0 0" />
          <parent link="${prefix}xtion_depth_frame" />
          <child link="${prefix}xtion_depth_optical_frame"/>
@@ -21,5 +21,5 @@
       <link name="${prefix}xtion_rgb_frame"/>
       <joint name="${prefix}xtion_rgb_optical_joint" type="fixed">
-         <origin xyz="0 0 0" rpy="${-M_PI/2} 0.0 ${-M_PI/2}" />
+         <origin xyz="0 0 0" rpy="0 0 0" />
          <parent link="${prefix}xtion_rgb_frame" />
          <child link="${prefix}xtion_rgb_optical_frame"/>
