Commit message: removed box from collion

File: urdf/base_v2/base.urdf.xacro (robot description, xacro)
@@ -22,10 +22,4 @@
          <origin xyz="0 0 0" rpy="-1.57 0 1.57"/>
       </collision>
-      <collision>
-        <geometry>
-             <box size="0.4 0.35635 0.454"/>
-        </geometry>
-        <origin xyz="-0.055 0 0.227" rpy="0 0 0"/>
-      </collision>
       <inertial>
         <mass value="40"/>

Commit message: update distance base visual and collision

File: urdf/base_v2/base.urdf.xacro (robot description, xacro)
@@ -11,5 +11,5 @@
             <mesh filename="package://sara_description/meshes/base.STL" scale="0.001 0.001 0.001"/>
          </geometry>
-         <origin xyz="0 0 0" rpy="-1.57 0 1.57"/>
+         <origin xyz="0.025 0 0" rpy="-1.57 0 1.57"/>
          <material name="black">
                <color rgba="0.12 0.12 0.12 1"/>
@@ -20,5 +20,5 @@
             <mesh filename="package://sara_description/meshes/base.STL" scale="0.001 0.001 0.001"/>
          </geometry>
-         <origin xyz="0 0 0" rpy="-1.57 0 1.57"/>
+         <origin xyz="0.025 0 0" rpy="-1.57 0 1.57"/>
       </collision>
       <inertial>
