Commit message: reformate l'urdf. le met à jours

File: urdf/base_v2/base.gazebo.xacro (robot description, xacro)
@@ -1,16 +1,13 @@
 <?xml version="1.0"?>
-<robot xmlns:xacro="http://ros.org/wiki/xacro">
-   <xacro:macro name="sara_base_gazebo_v2">
-       <gazebo reference="base_link">
-         <turnGravityOff>false</turnGravityOff>
-          <selfCollide>true</selfCollide>
-      </gazebo>
+<robot xmlns:xacro="http://www.ros.org/wiki/xacro">
+   <xacro:macro name="omni_steering" params="">
       <gazebo>
-         <plugin name="object_controller" filename="libgazebo_ros_planar_move.so">
+         <plugin name="omni_steering" filename="libgazebo_ros_planar_move.so">
             <commandTopic>/cmd_vel</commandTopic>
             <odometryTopic>/odom</odometryTopic>
             <odometryFrame>odom</odometryFrame>
-            <odometryRate>20.0</odometryRate>
+            <odometryRate>50.0</odometryRate>
             <robotBaseFrame>base_link</robotBaseFrame>
+            <publishTF>false</publishTF>
          </plugin>
       </gazebo>

File: urdf/base_v2/base.urdf.xacro (robot description, xacro)
@@ -1,18 +1,23 @@
 <?xml version="1.0"?>
 <robot xmlns:xacro="http://ros.org/wiki/xacro" >
-  <xacro:macro name="sara_base_v2" params="sim">
-      <xacro:if value="${sim}">
-          <xacro:include filename="$(find sara_description)/urdf/base_v2/base.gazebo.xacro"/>
-          <xacro:sara_base_gazebo_v2/>
-      </xacro:if>
-    <link name="base_link">
+  <xacro:macro name="sara_base" params="sim">
+      <xacro:include filename="$(find sara_description)/urdf/base_v2/base.gazebo.xacro"/>
+      <xacro:property name="PI" value="3.1415926535897931"/>
+      <link name="base_link">
+      <inertial>
+          <mass value="125.0" />
+          <origin xyz="0 0 0" />
+          <inertia  ixx="1.391" ixy="0.004"  ixz="0.0"
+                    iyy="6.853"  iyz="0.0"
+                    izz="6.125" />
+      </inertial>
       <visual>
-         <geometry>
-            <mesh filename="package://sara_description/meshes/base.STL" scale="0.001 0.001 0.001"/>
-         </geometry>
-         <origin xyz="0.025 0 0" rpy="-1.57 0 1.57"/>
-         <material name="black">
-               <color rgba="0 0.1 0.6 1"/>
-         </material>
+          <geometry>
+              <mesh filename="package://sara_description/meshes/base.STL" scale="0.001 0.001 0.001"/>
+          </geometry>
+          <origin xyz="0 0 0" rpy="${-PI/2} 0 ${PI/2}" />
+          <material name="darkgrey">
+              <color rgba="0.1 0.1 0.1 1"/>
+          </material>
       </visual>
       <collision>
@@ -20,13 +25,6 @@
             <mesh filename="package://sara_description/meshes/base.STL" scale="0.001 0.001 0.001"/>
          </geometry>
-         <origin xyz="0.025 0 0" rpy="-1.57 0 1.57"/>
+         <origin xyz="0.0 0 0" rpy="${-PI/2} 0 ${PI/2}"/>
       </collision>
-      <inertial>
-        <mass value="40"/>
-          <origin xyz="-0.055 0 0.227" rpy="-1.57 0 1.57"/>
-          <inertia ixx = "9.68458021" ixy = "2.23668848" ixz = "0.79348736"
-                   iyy = "2.66882541" iyz = "2.88061613"
-                   izz = "9.25217984"/>
-      </inertial>
     </link>
     </xacro:macro>

File: urdf/head_v1/head.gazebo.xacro (robot description, xacro)
@@ -1,8 +1,8 @@
 <?xml version="1.0"?>
-<robot xmlns:xacro="http://ros.org/wiki/xacro">
-   <xacro:macro name="sara_head_gazebo_v1">
+<robot xmlns:xacro="http://www.ros.org/wiki/xacro">
+   <xacro:macro name="sara_head_gazebo">
       <gazebo reference="head_link">
          <turnGravityOff>false</turnGravityOff>
-         <selfCollide>true</selfCollide>
+         <selfCollide>false</selfCollide>
       </gazebo>
    </xacro:macro>

File: urdf/head_v1/head.urdf.xacro (robot description, xacro)
@@ -1,11 +1,9 @@
 <?xml version="1.0"?>
-<robot xmlns:xacro="http://ros.org/wiki/xacro" >
-    <xacro:macro name="sara_head_v1" params="parent *origin sim">
+<robot xmlns:xacro="http://www.ros.org/wiki/xacro">
+    <xacro:macro name="sara_head" params="parent *origin sim">
         <xacro:if value="${sim}">
-            <xacro:include filename="$(find sara_description)/urdf/head_v1/head.gazebo.xacro" />
-            <xacro:sara_head_gazebo_v1/>
+            <xacro:include filename="$(find sara_description)/urdf/head_v1/head.gazebo.xacro"/>
+            <xacro:sara_head_gazebo/>
         </xacro:if>
-        <xacro:include filename="$(find sara_description)/urdf/head_v1/head.transmission.xacro" />
-        <xacro:sara_head_pitch_transmission_v1/>
         <joint name="head_pitch_joint" type="revolute">
             <parent link="${parent}_link"/>
@@ -13,30 +11,30 @@
             <limit effort="1000.0" lower="-1.3" upper="1.3" velocity="0.5"/>
             <xacro:insert_block name="origin"/>
-            <axis xyz="0 0 1" />
+            <axis xyz="0 0 1"/>
         </joint>
         <link name="head_link">
             <visual>
                 <geometry>
-                    <mesh filename="package://sara_description/meshes/tete.STL" scale="0.001 0.001 0.001" />
+                    <mesh filename="package://sara_description/meshes/tete.STL" scale="0.001 0.001 0.001"/>
                 </geometry>
-                <origin xyz="0 0 0" rpy="1.5708 -1.5708 1.5708" />
+                <origin xyz="0 0 0" rpy="1.5708 -1.5708 1.5708"/>
                 <material name="blue">
                     <color rgba="0.06 0.06 1 1"/>
-            </material>
-         </visual>
-         <collision>
-            <geometry>
-               <mesh filename="package://sara_description/meshes/tete.STL" scale="0.001 0.001 0.001" />
-            </geometry>
-            <origin xyz="0 0 0" rpy="1.5708 -1.5708 1.5708" />
-         </collision>
-         <inertial>
-            <mass value="2.60401968" />
-            <origin xyz="0 0 0" rpy="1.5708 0 1.5708" />
-            <inertia ixx = "0.02722768" ixy = "0.00015673" ixz = "0.0000148"
-                     iyy = "0.02716685" iyz = "0.00524002"
-                     izz = "0.04109802" />
-         </inertial>
-      </link>
-   </xacro:macro>
+                </material>
+            </visual>
+            <collision>
+                <geometry>
+                    <mesh filename="package://sara_description/meshes/tete.STL" scale="0.001 0.001 0.001"/>
+                </geometry>
+                <origin xyz="0 0 0" rpy="1.5708 -1.5708 1.5708"/>
+            </collision>
+            <inertial>
+                <mass value="2.60401968"/>
+                <origin xyz="0 0 0" rpy="1.5708 0 1.5708"/>
+                <inertia ixx="0.02722768" ixy="0.00015673" ixz="0.0000148"
+                         iyy="0.02716685" iyz="0.00524002"
+                         izz="0.04109802"/>
+            </inertial>
+        </link>
+    </xacro:macro>
 </robot>

File: urdf/head_xtion/head_xtion.urdf.xacro (robot description, xacro)
@@ -1,28 +1,28 @@
 <?xml version="1.0"?>
-<robot xmlns:xacro="http://ros.org/wiki/xacro">
-    <xacro:property name="M_PI" value="3.1415926535897931" />
+<robot xmlns:xacro="http://www.ros.org/wiki/xacro">
+    <xacro:property name="M_PI" value="3.1415926535897931"/>
     <xacro:macro name="asus_head_xtion" params="prefix parent *origin sim">
         <xacro:if value="${sim}">
-            <xacro:include filename="$(find sara_description)/urdf/head_xtion/head_xtion.gazebo.xacro" />
+            <xacro:include filename="$(find sara_description)/urdf/head_xtion/head_xtion.gazebo.xacro"/>
             <xacro:xtion_gazebo prefix="${prefix}"/>
         </xacro:if>
-      <joint name="${prefix}xtion_joint" type="fixed">
-        <xacro:insert_block name="origin" />
-        <parent link="${parent}_link"/>
-        <child link="${prefix}xtion_link"/>
-      </joint>
-      <link name="${prefix}xtion_link">
-        <inertial>
-          <mass value="0.200" />
-          <origin xyz="0 0 0" rpy="0 0 0" />
-          <inertia ixx="5.8083e-4" ixy="0" ixz="0" iyy="3.0833e-5" iyz="0" izz="5.9083e-4" />
-        </inertial>
-        <visual>
-          <origin xyz="0 0 0" rpy="0 0 0" />
-          <geometry>
-              <mesh filename="package://sara_description/meshes/head_xtion.STL" scale="0.001 0.001 0.001"/>
-          </geometry>
-        </visual>
-      </link>
+        <joint name="${prefix}xtion_joint" type="fixed">
+            <xacro:insert_block name="origin"/>
+            <parent link="${parent}_link"/>
+            <child link="${prefix}xtion_link"/>
+        </joint>
+        <link name="${prefix}xtion_link">
+            <inertial>
+                <mass value="0.200"/>
+                <origin xyz="0 0 0" rpy="0 0 0"/>
+                <inertia ixx="5.8083e-4" ixy="0" ixz="0" iyy="3.0833e-5" iyz="0" izz="5.9083e-4"/>
+            </inertial>
+            <visual>
+                <origin xyz="0 0 0" rpy="0 0 0"/>
+                <geometry>
+                    <mesh filename="package://sara_description/meshes/head_xtion.STL" scale="0.001 0.001 0.001"/>
+                </geometry>
+            </visual>
+        </link>
     </xacro:macro>
-  </robot>
+</robot>

File: urdf/hokuyo/hokuyo.gazebo.xacro (robot description, xacro)
@@ -1,4 +1,4 @@
 <?xml version="1.0"?>
-<robot xmlns:xacro="http://ros.org/wiki/xacro">
+<robot xmlns:xacro="http://www.ros.org/wiki/xacro">
     <xacro:macro name="hokuyo_gazebo" params="prefix">
         <!-- hokuyo -->
@@ -14,11 +14,11 @@
                             <samples>720</samples>
                             <resolution>1</resolution>
-                            <min_angle>-1.57</min_angle>
-                            <max_angle>1.57</max_angle>
+                            <min_angle>-2.35619449</min_angle>
+                            <max_angle>2.35619449</max_angle>
                         </horizontal>
                     </scan>
                     <range>
-                        <min>0.10</min>
-                        <max>30.0</max>
+                        <min>0.40</min>
+                        <max>10.0</max>
                         <resolution>0.01</resolution>
                     </range>
@@ -29,10 +29,10 @@
                                             stddev of 0.01m will put 99.7% of samples within 0.03m of the true
                                             reading. -->
-                        <mean>0.0</mean>
+                        <mean>0.01</mean>
                         <stddev>0.01</stddev>
                     </noise>
                 </ray>
                 <plugin name="gazebo_ros_${prefix}_hokuyo_controller" filename="libgazebo_ros_laser.so">
-                    <topicName>/hokuo/scan</topicName>
+                    <topicName>/scan</topicName>
                     <frameName>${prefix}hokuyo_link</frameName>
                 </plugin>

File: urdf/hokuyo/hokuyo.urdf.xacro (robot description, xacro)
@@ -1,4 +1,4 @@
 <?xml version="1.0"?>
-<robot xmlns:xacro="http://ros.org/wiki/xacro" >
+<robot xmlns:xacro="http://www.ros.org/wiki/xacro">
     <xacro:macro name="hokuyo" params="prefix parent *origin sim">
         <xacro:if value="${sim}">
@@ -21,10 +21,4 @@
                 </material>
             </visual>
-            <collision>
-                <geometry>
-                    <cylinder length="0.085" radius="0.03"/>
-                </geometry>
-                <origin xyz="0 0 0" rpy="0 0 0"/>
-            </collision>
             <inertial>
                 <mass value="0.5"/>

File: urdf/linear_actuator_v1/actuator.gazebo.xacro (robot description, xacro)
@@ -1,9 +1,9 @@
 <?xml version="1.0"?>
-<robot xmlns:xacro="http://ros.org/wiki/xacro">
-  <xacro:macro name="sara_linear_actuator_v1" params="prefix">
-    <gazebo reference="${prefix}actuator_link">
-        <turnGravityOff>false</turnGravityOff>
-      <selfCollide>true</selfCollide>
-    </gazebo>
-  </xacro:macro>
+<robot xmlns:xacro="http://www.ros.org/wiki/xacro">
+    <xacro:macro name="sara_linear_actuator_gazebo" params="prefix">
+        <gazebo reference="${prefix}actuator_link">
+            <turnGravityOff>false</turnGravityOff>
+            <selfCollide>true</selfCollide>
+        </gazebo>
+    </xacro:macro>
 </robot>

File: urdf/linear_actuator_v1/actuator.urdf.xacro (robot description, xacro)
@@ -1,23 +1,23 @@
 <?xml version="1.0"?>
-<robot xmlns:xacro="http://ros.org/wiki/xacro" >
-   <xacro:macro name="sara_linear_actuator_v1" params="parent *origin sim">
-       <xacro:if value="${sim}">
-           <xacro:include filename="$(find sara_description)/urdf/torso_v1/torso.gazebo.xacro" />
-           <xacro:sara_torso_gazebo_v1/>
-       </xacro:if>
-    <joint name="${parent}_actuator_joint" type="prismatic">
+<robot xmlns:xacro="http://www.ros.org/wiki/xacro">
+    <xacro:macro name="sara_linear_actuator" params="prefix parent *origin sim">
+        <xacro:if value="${sim}">
+            <xacro:include filename="$(find sara_description)/urdf/linear_actuator_v1/actuator.gazebo.xacro"/>
+            <xacro:sara_linear_actuator_gazebo prefix="${prefix}"/>
+        </xacro:if>
+        <joint name="${parent}_actuator_joint" type="prismatic">
             <parent link="${parent}_link"/>
             <child link="actuator_link"/>
             <xacro:insert_block name="origin"/>
             <limit effort="1000.0" lower="0" upper="0.675" velocity="0.02"/>
-            <axis xyz="0 0 1" />
-    </joint>
+            <axis xyz="0 0 1"/>
+        </joint>
         <link name="actuator_link">
             <inertial>
-      <origin rpy="0 0 0" xyz="-0.0013 -0.0009 0.3935" />
-      <mass value="10.7796" />
-      <inertia ixx="0.3354" ixy="0.0" ixz="-0.0162" iyy="0.3354" iyz="-0.0006" izz="0.0954" />
-    </inertial>
+                <origin rpy="0 0 0" xyz="-0.0013 -0.0009 0.3935"/>
+                <mass value="10.7796"/>
+                <inertia ixx="0.3354" ixy="0.0" ixz="-0.0162" iyy="0.3354" iyz="-0.0006" izz="0.0954"/>
+            </inertial>
         </link>
-   </xacro:macro>
+    </xacro:macro>
 </robot>

File: urdf/neck_v1/neck.gazebo.xacro (robot description, xacro)
@@ -1,8 +1,8 @@
 <?xml version="1.0"?>
-<robot xmlns:xacro="http://ros.org/wiki/xacro">
-   <xacro:macro name="sara_neck_gazebo_v1">
+<robot xmlns:xacro="http://www.ros.org/wiki/xacro">
+   <xacro:macro name="sara_neck_gazebo">
       <gazebo reference="neck_link">
          <turnGravityOff>false</turnGravityOff>
-         <selfCollide>true</selfCollide>
+         <selfCollide>false</selfCollide>
       </gazebo>
    </xacro:macro>

File: urdf/neck_v1/neck.urdf.xacro (robot description, xacro)
@@ -1,42 +1,40 @@
 <?xml version="1.0"?>
-<robot xmlns:xacro="http://ros.org/wiki/xacro" >
-   <xacro:macro name="sara_neck_v1" params="parent *origin sim">
-       <xacro:if value="${sim}">
-           <xacro:include filename="$(find sara_description)/urdf/neck_v1/neck.gazebo.xacro" />
-           <xacro:sara_neck_gazebo_v1/>
-       </xacro:if>
-       <xacro:include filename="$(find sara_description)/urdf/neck_v1/neck.transmission.xacro" />
-       <xacro:sara_head_yaw_transmission_v1/>
-       <joint name="head_yaw_joint" type="revolute">
-           <parent link="${parent}_link"/>
-           <child link="neck_link"/>
-           <limit effort="1000.0" lower="-1.5" upper="1.5" velocity="0.5"/>
-           <xacro:insert_block name="origin"/>
-           <axis xyz="0 0 1"/>
-       </joint>
-       <link name="neck_link">
-           <visual>
-               <geometry>
-                   <mesh filename="package://sara_description/meshes/couV2.STL" scale="0.001 0.001 0.001"/>
-               </geometry>
-               <origin xyz="0 0 0" rpy="1.5708 0 1.5708"/>
-               <material name="blue">
-                   <color rgba="0.06 0.06 1 1"/>
-               </material>
-             </visual>
-             <collision>
+<robot xmlns:xacro="http://www.ros.org/wiki/xacro">
+    <xacro:macro name="sara_neck" params="parent *origin sim">
+        <xacro:if value="${sim}">
+            <xacro:include filename="$(find sara_description)/urdf/neck_v1/neck.gazebo.xacro"/>
+            <xacro:sara_neck_gazebo/>
+        </xacro:if>
+        <joint name="head_yaw_joint" type="revolute">
+            <parent link="${parent}_link"/>
+            <child link="neck_link"/>
+            <limit effort="1000.0" lower="-1.5" upper="1.5" velocity="0.5"/>
+            <xacro:insert_block name="origin"/>
+            <axis xyz="0 0 1"/>
+        </joint>
+        <link name="neck_link">
+            <visual>
                 <geometry>
-                   <mesh filename="package://sara_description/meshes/couV2.STL" scale="0.001 0.001 0.001"/>
+                    <mesh filename="package://sara_description/meshes/couV2.STL" scale="0.001 0.001 0.001"/>
                 </geometry>
                 <origin xyz="0 0 0" rpy="1.5708 0 1.5708"/>
-             </collision>
-             <inertial>
+                <material name="blue">
+                    <color rgba="0.06 0.06 1 1"/>
+                </material>
+            </visual>
+            <collision>
+                <geometry>
+                    <mesh filename="package://sara_description/meshes/couV2.STL" scale="0.001 0.001 0.001"/>
+                </geometry>
+                <origin xyz="0 0 0" rpy="1.5708 0 1.5708"/>
+            </collision>
+            <inertial>
                 <mass value="2"/>
                 <origin xyz="0 0 0" rpy="1.5708 0 1.5708"/>
-                <inertia ixx = "0.00438238" ixy = "0.0" ixz = "0.0"
-                         iyy = "0.0040183" iyz = "0.0"
-                         izz = "0.00585293"/>
-             </inertial>
-       </link>
-   </xacro:macro>
+                <inertia ixx="0.00438238" ixy="0.0" ixz="0.0"
+                         iyy="0.0040183" iyz="0.0"
+                         izz="0.00585293"/>
+            </inertial>
+        </link>
+    </xacro:macro>
 </robot>

File: urdf/torso_v1/torso.gazebo.xacro (robot description, xacro)
@@ -1,5 +1,5 @@
 <?xml version="1.0"?>
-<robot xmlns:xacro="http://ros.org/wiki/xacro">
-   <xacro:macro name="sara_torso_gazebo_v1">
+<robot xmlns:xacro="http://www.ros.org/wiki/xacro">
+   <xacro:macro name="sara_torso_gazebo">
       <gazebo reference="torso_link">
          <turnGravityOff>false</turnGravityOff>

File: urdf/torso_v1/torso.urdf.xacro (robot description, xacro)
@@ -1,40 +1,38 @@
 <?xml version="1.0"?>
-<robot xmlns:xacro="http://ros.org/wiki/xacro" >
-   <xacro:macro name="sara_torso_v1" params="parent *origin sim">
-       <xacro:if value="${sim}">
-           <xacro:include filename="$(find sara_description)/urdf/torso_v1/torso.gazebo.xacro" />
-           <xacro:sara_torso_gazebo_v1/>
-       </xacro:if>
-       <joint name="${parent}_torso_joint" type="fixed">
-           <parent link="${parent}_link"/>
-           <child link="torso_link"/>
-           <limit effort="1000.0" lower="0" upper="0.5" velocity="0.2"/>
-           <xacro:insert_block name="origin"/>
-           <axis xyz="0 0 1" />
-       </joint>
-       <link name="torso_link">
-         <visual>
-            <geometry>
-               <mesh filename="package://sara_description/meshes/torse.STL" scale="0.001 0.001 0.001"/>
-            </geometry>
-            <origin xyz="0 0 0" rpy="0 0 0"/>
-            <material name="black">
-               <color rgba="0.12 0.12 0.12 1"/>
-            </material>
-         </visual>
-         <collision>
-            <geometry>
-               <mesh filename="package://sara_description/meshes/torse.STL" scale="0.001 0.001 0.001"/>
-            </geometry>
-            <origin xyz="0 0 0" rpy="0 0 0"/>
-         </collision>
-         <inertial>
-            <mass value="4.17008957"/>
-            <origin xyz="-0.14427 -0.197233 0" rpy="1.5708 0 1.5708"/>
-            <inertia ixx = "0.03994446" ixy = "0.00064933" ixz = "0.00005666"
-                     iyy = "0.04946667" iyz = "0.00660833"
-                     izz = "0.05202654"/>
-         </inertial>
-     </link>
-  </xacro:macro>
+<robot xmlns:xacro="http://www.ros.org/wiki/xacro">
+    <xacro:macro name="sara_torso" params="parent *origin sim">
+        <xacro:if value="${sim}">
+            <xacro:include filename="$(find sara_description)/urdf/torso_v1/torso.gazebo.xacro"/>
+            <xacro:sara_torso_gazebo/>
+        </xacro:if>
+        <joint name="${parent}_torso_joint" type="fixed">
+            <parent link="${parent}_link"/>
+            <child link="torso_link"/>
+            <xacro:insert_block name="origin"/>
+        </joint>
+        <link name="torso_link">
+            <visual>
+                <geometry>
+                    <mesh filename="package://sara_description/meshes/torse.STL" scale="0.001 0.001 0.001"/>
+                </geometry>
+                <origin xyz="0 0 0" rpy="0 0 0"/>
+                <material name="black">
+                    <color rgba="0.12 0.12 0.12 1"/>
+                </material>
+            </visual>
+            <collision>
+                <geometry>
+                    <mesh filename="package://sara_description/meshes/torse.STL" scale="0.001 0.001 0.001"/>
+                </geometry>
+                <origin xyz="0 0 0" rpy="0 0 0"/>
+            </collision>
+            <inertial>
+                <mass value="4.17008957"/>
+                <origin xyz="-0.14427 -0.197233 0" rpy="1.5708 0 1.5708"/>
+                <inertia ixx="0.03994446" ixy="0.00064933" ixz="0.00005666"
+                         iyy="0.04946667" iyz="0.00660833"
+                         izz="0.05202654"/>
+            </inertial>
+        </link>
+    </xacro:macro>
 </robot>
