Commit message: Utilise un force based planar movement pour controller les mouvements du robot

File: urdf/base_v2/base.gazebo.xacro (robot description, xacro)
@@ -1,15 +1,8 @@
 <?xml version="1.0"?>
 <robot xmlns:xacro="http://www.ros.org/wiki/xacro">
-   <xacro:macro name="omni_steering" params="">
-      <gazebo>
-         <plugin name="omni_steering" filename="libgazebo_ros_planar_move.so">
-            <commandTopic>/cmd_vel</commandTopic>
-            <odometryTopic>/odom</odometryTopic>
-            <odometryFrame>odom</odometryFrame>
-            <odometryRate>50.0</odometryRate>
-            <robotBaseFrame>base_link</robotBaseFrame>
-            <publishTF>false</publishTF>
-         </plugin>
-      </gazebo>
-   </xacro:macro>
+   <gazebo reference="chassis">
+      <material>Gazebo/DarkGrey</material>
+      <mu1>0.0</mu1>
+      <mu2>0.0</mu2>
+   </gazebo>
 </robot>

File: urdf/base_v2/base.urdf.xacro (robot description, xacro)
@@ -1,8 +1,12 @@
 <?xml version="1.0"?>
 <robot xmlns:xacro="http://ros.org/wiki/xacro" >
-  <xacro:macro name="sara_base" params="sim">
+  <xacro:macro name="sara_base" params="parent">
       <xacro:include filename="$(find sara_description)/urdf/base_v2/base.gazebo.xacro"/>
       <xacro:property name="PI" value="3.1415926535897931"/>
-      <link name="base_link">
+      <joint name="base_to_chassis" type="fixed">
+          <parent link="${parent}_link"/>
+          <child link="chassis"/>
+      </joint>
+      <link name="chassis">
       <inertial>
           <mass value="125.0" />

File: urdf/sara.gazebo.xacro (robot description, xacro)
@@ -1,10 +1,25 @@
 <?xml version="1.0"?>
-<robot xmlns:xacro="http://ros.org/wiki/xacro">
-   <xacro:macro name="sara_gazebo">
+<robot>
       <gazebo>
+         <static>false</static>
          <plugin name="gazebo_ros_control" filename="libgazebo_ros_control.so">
+            <robotNamespace>/sara_simulation</robotNamespace>
+            <robotSimType>gazebo_ros_control/DefaultRobotHWSim</robotSimType>
+            <legacyModeNS>false</legacyModeNS>
+         </plugin>
+         <plugin name="ridgeback_ros_force_based_move" filename="libridgeback_ros_force_based_move.so">
             <robotNamespace>/</robotNamespace>
+            <commandTopic>cmd_vel</commandTopic>
+            <odometryTopic>odom</odometryTopic>
+            <odometryFrame>odom</odometryFrame>
+            <odometryRate>25.0</odometryRate>
+            <robotBaseFrame>base_link</robotBaseFrame>
+            <cmdVelTimeOut>0.25</cmdVelTimeOut>
+            <!-- Don't publish a transform: the controller does it. -->
+            <publishOdometryTf>0</publishOdometryTf>
+            <yaw_velocity_p_gain>500.0</yaw_velocity_p_gain>
+            <x_velocity_p_gain>10000.0</x_velocity_p_gain>
+            <y_velocity_p_gain>10000.0</y_velocity_p_gain>
          </plugin>
       </gazebo>
-   </xacro:macro>
 </robot>

File: urdf/sara.urdf.xacro (robot description, xacro)
@@ -1,7 +1,7 @@
 <?xml version="1.0"?>
-<robot xmlns:xacro="http://ros.org/wiki/xacro" name="sara" >
+<robot name="sara" xmlns:xacro="http://ros.org/wiki/xacro">
+    <xacro:property name="PI" value="3.1415926535897931" />
     <xacro:arg name="sim" default="true"/>
     <xacro:property name="sim" value="$(arg sim)"/>
-    <!-- Inclure tous les autres urdf.xacros ici -->
     <xacro:include filename="$(find sara_description)/urdf/linear_actuator_v1/actuator.urdf.xacro"/>
     <xacro:include filename="$(find sara_description)/urdf/torso_v1/torso.urdf.xacro"/>
@@ -12,34 +12,19 @@
     <xacro:include filename="$(find sara_description)/urdf/base_v2/base.urdf.xacro"/>
     <xacro:include filename="$(find sara_description)/urdf/hokuyo/hokuyo.urdf.xacro"/>
-    <xacro:include filename="$(find sara_description)/urdf/mecanum_wheel/mecanum_wheel.urdf.xacro"/>
-    <xacro:include filename="$(find robotiq_140_description)/urdf/robotiq_arg2f_140_model_macro.xacro" />
-    <xacro:if value="${sim}">
-        <xacro:include filename="$(find sara_description)/urdf/sara.gazebo.xacro" />
-        <xacro:sara_gazebo/>
-    </xacro:if>
+    <link name="base_link"></link>
     <!-- Base -->
-    <xacro:sara_base_v2 sim="${sim}"/>
-    <!-- hokuyo -->
-    <xacro:hokuyo prefix="front_" parent="base" sim="${sim}">
-        <origin xyz="0.2516879 0 0" rpy="0 0 0" />
-    </xacro:hokuyo>
-    <!-- Wheels -->
-    <xacro:four_mecanum_wheels parent="base" x_center="0.22735" y_center="0.23" sim="${sim}"/>
-    <!-- Linear Actuator -->
-    <xacro:sara_linear_actuator_v1 parent="base" sim="${sim}">
-        <origin xyz="0 0 0.1" rpy="0 0 0" />
-    </xacro:sara_linear_actuator_v1>
+    <xacro:sara_base parent="base"/>
     <!-- Torso -->
-    <xacro:sara_torso_v1 parent="actuator" sim="${sim}">
-        <origin xyz="0.1999806 0 0.61595" rpy="0 0 0" />
-    </xacro:sara_torso_v1>
+    <xacro:sara_torso parent="base" sim="${sim}">
+        <origin xyz="0.1999806 0 1.189" rpy="0 0 0" />
+    </xacro:sara_torso>
     <!-- Neck -->
-    <xacro:sara_neck_v1 parent="torso" sim="${sim}">
+    <xacro:sara_neck parent="torso" sim="${sim}">
         <origin xyz="0.032295 0 0.10036" rpy="0 0 0"/>
-    </xacro:sara_neck_v1>
+    </xacro:sara_neck>
     <!-- Head -->
-    <xacro:sara_head_v1 parent="neck" sim="${sim}">
-        <origin xyz="0 0 0.1214" rpy="-1.57 0 0"/>
-    </xacro:sara_head_v1>
+    <xacro:sara_head parent="neck" sim="${sim}">
+        <origin xyz="0 0 0.0927" rpy="-1.57 0 0"/>
+    </xacro:sara_head>
     <!-- Head Xtion -->
     <xacro:asus_head_xtion prefix="head_" parent="head" sim="${sim}">
@@ -47,18 +32,8 @@
     </xacro:asus_head_xtion>
     <!-- Arm -->
-    <xacro:sara_arm_v2 prefix="right_" parent="torso" sim="${sim}">
+    <xacro:sara_arm prefix="right_" parent="torso" sim="${sim}">
         <origin xyz="0 -0.1437625 0.01166" rpy="0 -1.57 0"/>
-    </xacro:sara_arm_v2>
-    <!-- End Effector -->
-    <!-- Gripper 85 (round base)
-    <xacro:include filename="$(find robotiq_85_description)/urdf/robotiq_85_gripper.urdf.xacro"/>
-    <xacro:robotiq_85_gripper prefix="right_" parent="right_socket_link">
-        <origin xyz="0 0 -0.02989" rpy="0 1.5708 0"/>
-    </xacro:robotiq_85_gripper>-->
-    <!-- Gripper C2 (old model)
-    <xacro:include filename="$(find robotiq_c2_description)/urdf/robotiq_c2_model_macro.xacro"/>
-    <xacro:robotiq_c2_model prefix="right_" parent="right_socket_link">
-        <origin xyz="0 0 -0.02989" rpy="0 1.5708 0"/>
-    </xacro:robotiq_c2_model>-->
-    <xacro:robotiq_arg2f_140 prefix="right_"/>
+    </xacro:sara_arm>
+    <!-- Bring in simulation data for Gazebo. -->
+    <xacro:include filename="$(find sara_description)/urdf/sara.gazebo.xacro" />
 </robot>
