Commit message: base xtion ready to work

File: urdf/base_xtion/base_xtion.urdf.xacro (robot description, xacro)
@@ -43,5 +43,5 @@
           <dynamics damping="0.1"/>
           <limit effort="10000.0" lower="-1.5708" upper="1.5708" velocity="0.5"/>
-          <origin xyz="0.0115 0.035 0" rpy="1.5708 0 3.14" />
+          <origin xyz="0.035 0 0.0115" rpy="0 0 0" />
           <axis xyz="0 0 1" />
         </joint>

File: urdf/sara.urdf.xacro (robot description, xacro)
@@ -58,5 +58,5 @@
     <!-- Base xtion -->
     <xacro:asus_base_xtion prefix="base_" parent="base" sim="${sim}">
-        <origin xyz="0.2603774 0 0.9846921" rpy="0 0 0" />
+        <origin xyz="0.2003774 0 0.9846921" rpy="0 0 0" />
     </xacro:asus_base_xtion>
     <!-- End Effector -->

Commit message: changed orientation for base xtion pi / 4 to map

File: urdf/base_xtion/base_xtion.urdf.xacro (robot description, xacro)
@@ -43,5 +43,5 @@
           <dynamics damping="0.1"/>
           <limit effort="10000.0" lower="-1.5708" upper="1.5708" velocity="0.5"/>
-          <origin xyz="0.035 0 0.0115" rpy="0 0 0" />
+          <origin xyz="0.035 0 0.0115" rpy="0 0.78539816339 0" />
           <axis xyz="0 0 1" />
         </joint>
