Commit message: Update urdf with actuator

File: urdf/linear_actuator_v1/actuator.urdf.xacro (robot description, xacro)
@@ -9,18 +9,14 @@
             <parent link="${parent}_link"/>
             <child link="actuator_link"/>
-            <limit effort="1000.0" lower="-0.38" upper="0" velocity="0.5"/>
-            <origin rpy="0 0 0" xyz="0 0 0"/>
+            <xacro:insert_block name="origin"/>
+            <limit effort="1000.0" lower="0" upper="0.675" velocity="1"/>
             <axis xyz="0 0 1" />
     </joint>
         <link name="actuator_link">
-                 <visual>
-                    <geometry>
-                       <box size="1 1 1" />
-                    </geometry>
-                    <origin xyz="0 0 0" rpy="0 0 0"/>
-                    <material name="black">
-                       <color rgba="0.12 0.12 0.12 1"/>
-                    </material>
-                 </visual>
+            <inertial>
+      <origin rpy="0 0 0" xyz="-0.0013 -0.0009 0.2935" />
+      <mass value="10.7796" />
+      <inertia ixx="0.3354" ixy="0.0" ixz="-0.0162" iyy="0.3354" iyz="-0.0006" izz="0.0954" />
+    </inertial>
         </link>
    </xacro:macro>

Commit message: ajuste l'urdf pour accomoder la colone

File: urdf/linear_actuator_v1/actuator.urdf.xacro (robot description, xacro)
@@ -3,5 +3,5 @@
    <xacro:macro name="sara_linear_actuator_v1" params="parent *origin sim">
        <xacro:if value="${sim}">
-           <xacro:include filename="$(find sara_description)/urdf/linear_actuator_v1/torso.gazebo.xacro" />
+           <xacro:include filename="$(find sara_description)/urdf/torso_v1/torso.gazebo.xacro" />
            <xacro:sara_torso_gazebo_v1/>
        </xacro:if>
@@ -10,5 +10,5 @@
             <child link="actuator_link"/>
             <xacro:insert_block name="origin"/>
-            <limit effort="1000.0" lower="0" upper="0.675" velocity="1"/>
+            <limit effort="1000.0" lower="0" upper="0.675" velocity="0.02"/>
             <axis xyz="0 0 1" />
     </joint>
