Commit message: ajustements des limites des joints

File: urdf/head_v1/head.urdf.xacro (robot description, xacro)
@@ -11,5 +11,5 @@
             <parent link="${parent}_link"/>
             <child link="head_link"/>
-            <limit effort="1000.0" lower="-0.8" upper="0.8" velocity="0.5"/>
+            <limit effort="1000.0" lower="-0.9" upper="0.9" velocity="0.5"/>
             <xacro:insert_block name="origin"/>
             <axis xyz="0 0 1" />

File: urdf/linear_actuator_v1/actuator.urdf.xacro (robot description, xacro)
@@ -15,5 +15,5 @@
         <link name="actuator_link">
             <inertial>
-      <origin rpy="0 0 0" xyz="-0.0013 -0.0009 0.2935" />
+      <origin rpy="0 0 0" xyz="-0.0013 -0.0009 0.3935" />
       <mass value="10.7796" />
       <inertia ixx="0.3354" ixy="0.0" ixz="-0.0162" iyy="0.3354" iyz="-0.0006" izz="0.0954" />

File: urdf/sara.urdf.xacro (robot description, xacro)
@@ -28,5 +28,5 @@
     <!-- Linear Actuator -->
     <xacro:sara_linear_actuator_v1 parent="base" sim="${sim}">
-        <origin xyz="0 0 0" rpy="0 0 0" />
+        <origin xyz="0 0 0.1" rpy="0 0 0" />
     </xacro:sara_linear_actuator_v1>
     <!-- Torso -->
