Commit message: Updated with new neck geometry.

File: urdf/neck_v1/neck.urdf.xacro (robot description, xacro)
@@ -18,5 +18,5 @@
            <visual>
                <geometry>
-                   <mesh filename="package://sara_description/meshes/cou.STL" scale="0.001 0.001 0.001"/>
+                   <mesh filename="package://sara_description/meshes/couV2.STL" scale="0.001 0.001 0.001"/>
                </geometry>
                <origin xyz="0 0 0" rpy="1.5708 0 1.5708"/>
@@ -27,5 +27,5 @@
              <collision>
                 <geometry>
-                   <mesh filename="package://sara_description/meshes/cou.STL" scale="0.001 0.001 0.001"/>
+                   <mesh filename="package://sara_description/meshes/couV2.STL" scale="0.001 0.001 0.001"/>
                 </geometry>
                 <origin xyz="0 0 0" rpy="1.5708 0 1.5708"/>

File: urdf/sara.urdf.xacro (robot description, xacro)
@@ -40,5 +40,5 @@
     <!-- Head -->
     <xacro:sara_head_v1 parent="neck" sim="${sim}">
-        <origin xyz="0 0 0.0927" rpy="-1.57 0 0"/>
+        <origin xyz="0 0 0.1214" rpy="-1.57 0 0"/>
     </xacro:sara_head_v1>
     <!-- Head Xtion -->
