Commit message: Adding transmission files, renaming link and joints, adding modularity, working xtion simulation.

File: urdf/arm_v2/arm.urdf.xacro (robot description, xacro)
@@ -1,29 +1,33 @@
 <?xml version="1.0"?>
 <robot xmlns:xacro="http://ros.org/wiki/xacro" >
-   <xacro:include filename="$(find sara_description)/urdf/arm_v1/arm.gazebo.xacro" />
-   <xacro:macro name="sara_arm_v1" params="name parent">
-     <xacro:sara_arm_gazebo_v1 name="${name}" parent="${parent}"/>
-     <joint name="${parent}_${name}_joint" type="revolute">
+   <xacro:macro name="sara_arm_v2" params="prefix parent *origin sim">
+     <xacro:if value="${sim}">
+       <xacro:include filename="$(find sara_description)/urdf/arm_v2/arm.gazebo.xacro" />
+       <xacro:sara_arm_gazebo_v2 prefix="${prefix}"/>
+     </xacro:if>
+     <xacro:include filename="$(find sara_description)/urdf/arm_v2/arm.transmission.xacro" />
+     <xacro:sara_arm_transmission_v2 prefix="${prefix}"/>
+     <joint name="${prefix}shoulder_roll_joint" type="revolute">
        <parent link="${parent}_link"/>
-       <child link="${name}_clavicular_link"/>
+       <child link="${prefix}clavicular_link"/>
        <limit effort="1000.0" lower="-1.6" upper="1.4" velocity="0.5"/>
-       <origin xyz="0 -0.145 0.189" rpy="0 -1.57 0"/>
-       <axis xyz="0 0 1" />
-     </joint>
-     <link name="${name}_clavicular_link">
-       <visual>
-         <geometry>
-           <mesh filename="package://sara_description/meshes/epaule.STL" scale="0.001 0.001 0.001"/>
-           </geometry>
+       <xacro:insert_block name="origin"/>
+       <axis xyz="0 0 1" />
+     </joint>
+     <link name="${prefix}clavicular_link">
+       <visual>
+         <geometry>
+           <mesh filename="package://sara_description/meshes/epaule.STL" scale="0.001 0.001 0.001"/>
+         </geometry>
+         <origin xyz="0 0 0" rpy="0 3.1416 0"/>
+         <material name="black">
+           <color rgba="0.12 0.12 0.12 1"/>
+         </material>
+       </visual>
+       <collision>
+         <geometry>
+           <mesh filename="package://sara_description/meshes/epaule.STL" scale="0.001 0.001 0.001"/>
+         </geometry>
            <origin xyz="0 0 0" rpy="0 3.1416 0"/>
-           <material name="black">
-             <color rgba="0.12 0.12 0.12 1"/>
-           </material>
-       </visual>
-       <collision>
-         <geometry>
-           <mesh filename="package://sara_description/meshes/epaule.STL" scale="0.001 0.001 0.001"/>
-         </geometry>
-           <origin xyz="0 0 0" rpy="0 3.1416 0"/>
        </collision>
        <inertial>
@@ -33,12 +37,12 @@
        </inertial>
      </link>
-     <joint name="${name}_shoulder_joint" type="revolute">
-       <parent link="${name}_clavicular_link"/>
-       <child link="${name}_fix_upper_link"/>
+     <joint name="${prefix}shoulder_pitch_joint" type="revolute">
+       <parent link="${prefix}clavicular_link"/>
+       <child link="${prefix}upper_arm_upper_link"/>
        <limit effort="1000.0" lower="-4.7124" upper="1.5708" velocity="0.5"/>
        <origin xyz="0 -0.085 0" rpy="-1.57 0 0" />
        <axis xyz="0 0 1" />
      </joint>
-     <link name="${name}_fix_upper_link">
+     <link name="${prefix}upper_arm_upper_link">
        <visual>
          <geometry>
@@ -62,12 +66,12 @@
          </inertial>
      </link>
-     <joint name="${name}_rot_elbow_joint" type="revolute">
-       <parent link="${name}_fix_upper_link"/>
-       <child link="${name}_rot_upper_link"/>
+     <joint name="${prefix}shoulder_yaw_joint" type="revolute">
+       <parent link="${prefix}upper_arm_upper_link"/>
+       <child link="${prefix}upper_arm_lower_link"/>
        <limit effort="1000.0" lower="-3.1416" upper="3.1416" velocity="0.5"/>
        <origin xyz="-0.085 0 0" rpy="1.5708 0 1.5708" />
        <axis xyz="0 0 1" />
      </joint>
-     <link name="${name}_rot_upper_link">
+     <link name="${prefix}upper_arm_lower_link">
        <visual>
          <geometry>
@@ -91,12 +95,12 @@
        </inertial>
      </link>
-      <joint name="${name}_elbow_joint" type="revolute">
-        <parent link="${name}_rot_upper_link"/>
-        <child link="${name}_fix_lower_link"/>
+      <joint name="${prefix}elbow_pitch_joint" type="revolute">
+        <parent link="${prefix}upper_arm_lower_link"/>
+        <child link="${prefix}forearm_upper_link"/>
         <limit effort="1000.0" lower="-2.20" upper="1.90" velocity="0.5"/>
         <origin xyz="0 0 -0.31" rpy="-1.5708 0 0" />
         <axis xyz="0 0 1" />
       </joint>
-      <link name="${name}_fix_lower_link">
+      <link name="${prefix}forearm_upper_link">
         <visual>
           <geometry>
@@ -120,12 +124,12 @@
         </inertial>
       </link>
-     <joint name="${name}_rot_wrist_joint" type="revolute">
-       <parent link="${name}_fix_lower_link"/>
-       <child link="${name}_rot_lower_link"/>
+     <joint name="${prefix}elbow_yaw_joint" type="revolute">
+       <parent link="${prefix}forearm_upper_link"/>
+       <child link="${prefix}forearm_lower_link"/>
        <limit effort="1000.0" lower="-3.1416" upper="3.1416" velocity="0.5"/>
        <origin xyz="0 0.0945 0" rpy="1.5708 -1.5708 0" />
        <axis xyz="0 0 1" />
      </joint>
-     <link name="${name}_rot_lower_link">
+     <link name="${prefix}forearm_lower_link">
        <visual>
          <geometry>
@@ -149,12 +153,12 @@
        </inertial>
      </link>
-     <joint name="${name}_forarm_wrist_joint" type="fixed">
-       <parent link="${name}_rot_lower_link"/>
-       <child link="${name}_high_wrist_link"/>
+     <joint name="${prefix}wrist_joint" type="fixed">
+       <parent link="${prefix}forearm_lower_link"/>
+       <child link="${prefix}upper_wrist_link"/>
        <limit effort="1000.0" lower="-3.1416" upper="3.1416" velocity="0.5"/>
        <origin xyz="0 0 -0.11184" rpy="1.5708 -1.5708 0" />
        <axis xyz="0 1 0" />
      </joint>
-     <link name="${name}_high_wrist_link">
+     <link name="${prefix}upper_wrist_link">
        <visual>
          <geometry>
@@ -178,12 +182,12 @@
        </inertial>
      </link>
-     <joint name="${name}_high_low_wrist_joint" type="revolute">
-       <parent link="${name}_high_wrist_link"/>
-       <child link="${name}_low_wrist_link"/>
+     <joint name="${prefix}wrist_pitch_joint" type="revolute">
+       <parent link="${prefix}upper_wrist_link"/>
+       <child link="${prefix}lower_wrist_link"/>
        <limit effort="1000.0" lower="-1.5708" upper="1.5708" velocity="0.5"/>
        <origin xyz="0 0 0" rpy="1.5708 -1.5708 0" />
        <axis xyz="0 0 1" />
      </joint>
-     <link name="${name}_low_wrist_link">
+     <link name="${prefix}lower_wrist_link">
        <visual>
          <geometry>
@@ -207,12 +211,12 @@
        </inertial>
      </link>
-     <joint name="${name}_low_wrist_grasp_socket_joint" type="revolute">
-       <parent link="${name}_low_wrist_link"/>
-       <child link="${name}_socket_link"/>
+     <joint name="${prefix}wrist_yaw_joint" type="revolute">
+       <parent link="${prefix}lower_wrist_link"/>
+       <child link="${prefix}socket_link"/>
        <limit effort="1000.0" lower="-1.49" upper="1.49" velocity="0.5"/>
        <origin xyz="0 0.084375 0" rpy="1.5708 0 0" />
        <axis xyz="1 0 0" />
      </joint>
-     <link name="${name}_socket_link">
+     <link name="${prefix}socket_link">
        <visual>
          <geometry>

File: urdf/base_v2/base.urdf.xacro (robot description, xacro)
@@ -1,8 +1,10 @@
 <?xml version="1.0"?>
 <robot xmlns:xacro="http://ros.org/wiki/xacro" >
-  <xacro:include filename="$(find sara_description)/urdf/base_v1/base.gazebo.xacro"/>
-  <xacro:macro name="sara_base_v1" params="name parent">
-    <xacro:sara_base_gazebo_v1 name="${name}" parent="${parent}"/>
-    <link name="${name}_link">
+  <xacro:macro name="sara_base_v2" params="sim">
+      <xacro:if value="${sim}">
+          <xacro:include filename="$(find sara_description)/urdf/base_v2/base.gazebo.xacro"/>
+          <xacro:sara_base_gazebo_v2/>
+      </xacro:if>
+    <link name="base_link">
       <visual>
          <geometry>
@@ -50,32 +52,4 @@
       </inertial>
     </link>
-    <!-- Lidar -->
-    <link name="lidar_link">
-      <visual>
-        <geometry>
-          <cylinder length="0.085" radius="0.03"/>
-        </geometry>
-        <origin xyz="0 0 0" rpy="0 0 0"/>
-        <material name="orange">
-          <color rgba="1 0.5 0 1"/>
-        </material>
-      </visual>
-      <collision>
-        <geometry>
-          <cylinder length="0.085" radius="0.03"/>
-        </geometry>
-        <origin xyz="0 0 0" rpy="0 0 0"/>
-      </collision>
-      <inertial>
-        <mass value="0.5"/>
-        <origin xyz="0 0 0" rpy="0 0 0"/>
-        <inertia ixx="0.001" ixy="0" ixz="0" iyy="0.001" iyz="0" izz="0.001"/>
-      </inertial>
-    </link>
-    <joint name="laser_joint" type="fixed">
-      <parent link="base_link"/>
-      <child link="lidar_link"/>
-      <origin xyz="0.2516879 0 0" rpy="0 0 0" />
-    </joint>
     </xacro:macro>
   </robot>

File: urdf/head_v1/head.gazebo.xacro (robot description, xacro)
@@ -1,49 +1,8 @@
 <?xml version="1.0"?>
 <robot xmlns:xacro="http://ros.org/wiki/xacro">
-   <xacro:macro name="sara_head_gazebo_v1" params="name parent">
-      <gazebo reference="neck_dynamixel_link">
-         <turnGravityOff>false</turnGravityOff>
-      </gazebo>
+   <xacro:macro name="sara_head_gazebo_v1">
       <gazebo reference="head_link">
          <turnGravityOff>false</turnGravityOff>
-      </gazebo>
-      <gazebo reference="camera_link">
-         <turnGravityOff>false</turnGravityOff>
-         <sensor type="depth" name="camera">
-            <visualize>true</visualize>
-            <pose>0 0 0 0 0 0</pose>
-            <always_on>true</always_on>
-            <update_rate>20.0</update_rate>
-            <camera>
-               <horizontal_fov>1.3962634</horizontal_fov>
-               <image>
-                  <format>R8G8B8</format>
-                  <width>640</width>
-                  <height>480</height>
-               </image>
-               <clip>
-                  <near>0.05</near>
-                  <far>8.0</far>
-               </clip>
-            </camera>
-            <plugin name="kinect_camera_controller" filename="libgazebo_ros_openni_kinect.so">
-               <cameraName>camera</cameraName>
-               <alwaysOn>true</alwaysOn>
-               <updateRate>5</updateRate>
-               <imageTopicName>rgb/image_raw</imageTopicName>
-               <depthImageTopicName>depth/image_raw</depthImageTopicName>
-               <pointCloudTopicName>depth/points</pointCloudTopicName>
-               <cameraInfoTopicName>rgb/camera_info</cameraInfoTopicName>
-               <depthImageCameraInfoTopicName>depth/camera_info</depthImageCameraInfoTopicName>
-               <frameName>camera/camera_rgb_optical_frame</frameName>
-               <baseline>0.1</baseline>
-               <distortion_k1>0.0</distortion_k1>
-               <distortion_k2>0.0</distortion_k2>
-               <distortion_k3>0.0</distortion_k3>
-               <distortion_t1>0.0</distortion_t1>
-               <distortion_t2>0.0</distortion_t2>
-               <pointCloudCutoff>0.4</pointCloudCutoff>
-            </plugin>
-         </sensor>
+         <selfCollide>true</selfCollide>
       </gazebo>
    </xacro:macro>

File: urdf/head_v1/head.urdf.xacro (robot description, xacro)
@@ -1,15 +1,26 @@
 <?xml version="1.0"?>
 <robot xmlns:xacro="http://ros.org/wiki/xacro" >
-   <xacro:include filename="$(find sara_description)/urdf/head_v1/head.gazebo.xacro" />
-   <xacro:macro name="sara_head_v1" params="name parent">
-     <xacro:sara_head_gazebo_v1 name="${name}" parent="${parent}"/>
-     <link name="${name}_link">
-         <visual>
-            <geometry>
-               <mesh filename="package://sara_description/meshes/tete.STL" scale="0.001 0.001 0.001" />
-            </geometry>
-            <origin xyz="0 0 0" rpy="1.5708 -1.5708 1.5708" />
-            <material name="blue">
-                <color rgba="0.06 0.06 1 1"/>
+    <xacro:macro name="sara_head_v1" params="parent *origin sim">
+        <xacro:if value="${sim}">
+            <xacro:include filename="$(find sara_description)/urdf/head_v1/head.gazebo.xacro" />
+            <xacro:sara_head_gazebo_v1/>
+        </xacro:if>
+        <xacro:include filename="$(find sara_description)/urdf/head_v1/head.transmission.xacro" />
+        <xacro:sara_head_pitch_transmission_v1/>
+        <joint name="head_pitch_joint" type="revolute">
+            <parent link="${parent}_link"/>
+            <child link="head_link"/>
+            <limit effort="1000.0" lower="-0.40" upper="1.04" velocity="0.5"/>
+            <xacro:insert_block name="origin"/>
+            <axis xyz="0 0 1" />
+        </joint>
+        <link name="head_link">
+            <visual>
+                <geometry>
+                    <mesh filename="package://sara_description/meshes/tete.STL" scale="0.001 0.001 0.001" />
+                </geometry>
+                <origin xyz="0 0 0" rpy="1.5708 -1.5708 1.5708" />
+                <material name="blue">
+                    <color rgba="0.06 0.06 1 1"/>
             </material>
          </visual>
@@ -26,61 +37,4 @@
          </inertial>
       </link>
-      <link name="${name}_dynamixel_link">
-         <visual>
-            <geometry>
-               <cylinder length="0.015" radius="0.02"/>
-            </geometry>
-            <origin xyz="0 0 0.018" rpy="0 0 0"/>
-            <material name="blue">
-               <color rgba="0 0 1 1"/>
-            </material>
-        </visual>
-        <inertial>
-            <mass value="5" />
-            <origin xyz="0 0 0.018" rpy="0 0 0" />
-            <inertia ixx="0.001" ixy="0" ixz="0" iyy="0.001" iyz="0" izz="0.001" />
-         </inertial>
-      </link>
-      <joint name="${name}_dynamixel_joint" type="revolute">
-         <parent link="${name}_link"/>
-         <child link="${name}_dynamixel_link"/>
-         <limit effort="1000.0" lower="-1.5" upper="1.5" velocity="0.5"/>
-         <origin xyz="0 -0.054 0" rpy="3.1416 0 0"/>
-         <axis xyz="0 0 1"/>
-      </joint>
-      <joint name="${parent}_${name}_joint" type="revolute">
-         <parent link="${parent}_link"/>
-         <child link="${name}_link"/>
-         <limit effort="1000.0" lower="-0.40" upper="1.04" velocity="0.5"/>
-         <origin xyz="0 0 0.0927" rpy="-1.57 0 0"/>
-         <axis xyz="0 0 1" />
-      </joint>
-      <!-- xtion -->
-      <link name="camera_link">
-         <visual>
-            <geometry>
-               <mesh filename="package://sara_description/meshes/xtion.STL" scale="0.001 0.001 0.001"/>
-            </geometry>
-            <origin xyz="0 0 0" rpy="1.5708 0 1.5708"/>
-            <material name="black"/>
-         </visual>
-         <collision>
-            <geometry>
-               <mesh filename="package://sara_description/meshes/xtion.STL" scale="0.001 0.001 0.001"/>
-            </geometry>
-            <origin xyz="0 0 0" rpy="1.5708 0 1.5708"/>
-         </collision>
-         <inertial>
-            <mass value="0.5"/>
-            <origin xyz="0 0 0" rpy="1.5708 0 1.5708"/>
-            <inertia ixx="0.001" ixy="0" ixz="0" iyy="0.001" iyz="0" izz="0.001"/>
-         </inertial>
-      </link>
-      <joint name="camera_joint" type="fixed">
-         <parent link="${name}_link"/>
-         <child link="camera_link"/>
-         <origin xyz="0.0776104 -0.13 0" rpy="1.57 0 0" />
-         <axis xyz="0 1 0" />
-      </joint>
    </xacro:macro>
 </robot>

File: urdf/kinect2/kinect2.gazebo.xacro (robot description, xacro)
@@ -4,4 +4,5 @@
       <gazebo reference="${name}_link">
          <turnGravityOff>false</turnGravityOff>
+         <selfCollide>true</selfCollide>
       </gazebo>
    </xacro:macro>

File: urdf/kinect2/kinect2.urdf.xacro (robot description, xacro)
@@ -1,8 +1,17 @@
 <?xml version="1.0"?>
 <robot xmlns:xacro="http://ros.org/wiki/xacro" >
-  <xacro:include filename="$(find sara_description)/urdf/kinect_v1/kinect.gazebo.xacro" />
-  <xacro:macro name="kinect2" params="name parent">
-      <xacro:kinect2_gazebo name="${name}" parent="${parent}"/>
-      <link name="${name}_link">
+  <xacro:macro name="kinect2" params="prefix parent *origin sim">
+      <xacro:if value="${sim}">
+          <xacro:include filename="$(find sara_description)/urdf/kinect2/kinect2.gazebo.xacro" />
+          <xacro:kinect2_gazebo name="kinect2" parent="${parent}"/>
+      </xacro:if>
+      <joint name="${parent}_kinect2_joint" type="fixed">
+          <parent link="${parent}_link"/>
+          <child link="kinect2_link"/>
+          <limit effort="1000.0" lower="0" upper="0.5" velocity="0.2"/>
+          <xacro:insert_block name="origin" />
+          <axis xyz="0 0 1" />
+      </joint>
+      <link name="kinect2_link">
         <visual>
            <geometry>
@@ -26,11 +35,4 @@
         </inertial>
     </link>
-    <joint name="${parent}_${name}_joint" type="fixed">
-        <parent link="${parent}_link"/>
-        <child link="${name}_link"/>
-        <limit effort="1000.0" lower="0" upper="0.5" velocity="0.2"/>
-        <origin xyz="0.177374 0 0.65676" rpy="-1.5708 0 -1.5708" />
-        <axis xyz="0 0 1" />
-   </joint>
  </xacro:macro>
 </robot>

File: urdf/mecanum_wheel/mecanum_wheel.gazebo.xacro (robot description, xacro)
@@ -1,6 +1,6 @@
 <?xml version="1.0"?>
 <robot xmlns:xacro="http://ros.org/wiki/xacro">
-   <xacro:macro name="sara_wheels_gazebo_v1" params="name parent">
-      <gazebo reference="${name}_link">
+   <xacro:macro name="mecanum_wheel_gazebo" params="position">
+      <gazebo reference="${position}_mecanum_wheel_link">
         <mu1 value="0"/>
         <mu2 value="0"/>

File: urdf/neck_v1/neck.gazebo.xacro (robot description, xacro)
@@ -1,7 +1,8 @@
 <?xml version="1.0"?>
 <robot xmlns:xacro="http://ros.org/wiki/xacro">
-   <xacro:macro name="sara_neck_gazebo_v1" params="name parent">
-      <gazebo reference="${name}_link">
+   <xacro:macro name="sara_neck_gazebo_v1">
+      <gazebo reference="neck_link">
          <turnGravityOff>false</turnGravityOff>
+         <selfCollide>true</selfCollide>
       </gazebo>
    </xacro:macro>

File: urdf/neck_v1/neck.urdf.xacro (robot description, xacro)
@@ -1,37 +1,40 @@
 <?xml version="1.0"?>
 <robot xmlns:xacro="http://ros.org/wiki/xacro" >
-   <xacro:include filename="$(find sara_description)/urdf/neck_v1/neck.gazebo.xacro" />
-   <xacro:macro name="sara_neck_v1" params="name parent">
-     <xacro:sara_neck_gazebo_v1 name="${name}" parent="${parent}"/>
-     <link name="${name}_link">
-         <visual>
-            <geometry>
-               <mesh filename="package://sara_description/meshes/cou.STL" scale="0.001 0.001 0.001"/>
-            </geometry>
-            <origin xyz="0 0 0" rpy="1.5708 0 1.5708"/>
-            <material name="blue">
-                <color rgba="0.06 0.06 1 1"/>
-            </material>
-         </visual>
-         <collision>
-            <geometry>
-               <mesh filename="package://sara_description/meshes/cou.STL" scale="0.001 0.001 0.001"/>
-            </geometry>
-            <origin xyz="0 0 0" rpy="1.5708 0 1.5708"/>
-         </collision>
-         <inertial>
-            <mass value="2"/>
-            <origin xyz="0 0 0" rpy="1.5708 0 1.5708"/>
-            <inertia ixx="0.001" ixy="0" ixz="0" iyy="0.001" iyz="0" izz="0.001"/>
-         </inertial>
-      </link>
-      <joint name="${parent}_${name}_joint" type="revolute">
-         <parent link="${parent}_link"/>
-         <child link="${name}_link"/>
-         <limit effort="1000.0" lower="-1.22173" upper="1.22173" velocity="0.5"/>
-         <!-- 1mm ajoute en z (collision) -->
-         <origin xyz="0.032295 0 0.2777" rpy="0 0 0"/>
-         <axis xyz="0 0 1"/>
-      </joint>
+   <xacro:macro name="sara_neck_v1" params="parent *origin sim">
+       <xacro:if value="${sim}">
+           <xacro:include filename="$(find sara_description)/urdf/neck_v1/neck.gazebo.xacro" />
+           <xacro:sara_neck_gazebo_v1/>
+       </xacro:if>
+       <xacro:include filename="$(find sara_description)/urdf/neck_v1/neck.transmission.xacro" />
+       <xacro:sara_head_yaw_transmission_v1/>
+       <joint name="head_yaw_joint" type="revolute">
+           <parent link="${parent}_link"/>
+           <child link="neck_link"/>
+           <limit effort="1000.0" lower="-1.22173" upper="1.22173" velocity="0.5"/>
+           <xacro:insert_block name="origin"/>
+           <axis xyz="0 0 1"/>
+       </joint>
+       <link name="neck_link">
+           <visual>
+               <geometry>
+                   <mesh filename="package://sara_description/meshes/cou.STL" scale="0.001 0.001 0.001"/>
+               </geometry>
+               <origin xyz="0 0 0" rpy="1.5708 0 1.5708"/>
+               <material name="blue">
+                   <color rgba="0.06 0.06 1 1"/>
+               </material>
+             </visual>
+             <collision>
+                <geometry>
+                   <mesh filename="package://sara_description/meshes/cou.STL" scale="0.001 0.001 0.001"/>
+                </geometry>
+                <origin xyz="0 0 0" rpy="1.5708 0 1.5708"/>
+             </collision>
+             <inertial>
+                <mass value="2"/>
+                <origin xyz="0 0 0" rpy="1.5708 0 1.5708"/>
+                <inertia ixx="0.001" ixy="0" ixz="0" iyy="0.001" iyz="0" izz="0.001"/>
+             </inertial>
+       </link>
    </xacro:macro>
 </robot>
