Commit message: Adding transmission files, renaming link and joints, adding modularity, working xtion simulation.

File: urdf/sara.urdf.xacro (robot description, xacro)
@@ -1,36 +1,66 @@
 <?xml version="1.0"?>
 <robot xmlns:xacro="http://ros.org/wiki/xacro" name="sara" >
+    <xacro:property name="sim" value="$(arg sim)"/>
+    <xacro:property name="end_effector" value="$(arg end_effector)"/>
     <!-- Inclure tous les autres urdf.xacros ici -->
     <xacro:include filename="$(find sara_description)/urdf/torso_v1/torso.urdf.xacro"/>
     <xacro:include filename="$(find sara_description)/urdf/neck_v1/neck.urdf.xacro"/>
-    <xacro:include filename="$(find sara_description)/urdf/kinect_v1/kinect.urdf.xacro"/>
+    <xacro:include filename="$(find sara_description)/urdf/kinect2/kinect2.urdf.xacro"/>
+    <xacro:include filename="$(find sara_description)/urdf/xtion/xtion.urdf.xacro"/>
     <xacro:include filename="$(find sara_description)/urdf/head_v1/head.urdf.xacro"/>
-    <xacro:include filename="$(find sara_description)/urdf/arm_v1/arm.urdf.xacro"/>
-    <xacro:include filename="$(find sara_description)/urdf/base_v1/base.urdf.xacro"/>
-    <xacro:include filename="$(find sara_description)/urdf/wheels_v1/wheels.urdf.xacro"/>
-    <xacro:include filename="$(find robotiq_85_description)/urdf/robotiq_85_gripper.urdf.xacro"/>
-    <xacro:include filename="$(find robotiq_c2_model_visualization)/urdf/robotiq_c2_model_macro.xacro"/>
+    <xacro:include filename="$(find sara_description)/urdf/arm_v2/arm.urdf.xacro"/>
+    <xacro:include filename="$(find sara_description)/urdf/base_v2/base.urdf.xacro"/>
+    <xacro:include filename="$(find sara_description)/urdf/hokuyo/hokuyo.urdf.xacro"/>
+    <xacro:include filename="$(find sara_description)/urdf/mecanum_wheel/mecanum_wheel.urdf.xacro"/>
+    <xacro:if value="${sim}">
+        <xacro:include filename="$(find sara_description)/urdf/sara.gazebo.xacro" />
+        <xacro:sara_gazebo/>
+    </xacro:if>
     <!-- Base -->
-    <xacro:sara_base_v1 name="base" parent=""/>
+    <xacro:sara_base_v2 sim="${sim}"/>
+    <!-- hokuyo -->
+    <xacro:hokuyo prefix="front_" parent="base" sim="${sim}">
+        <origin xyz="0.2516879 0 0" rpy="0 0 0" />
+    </xacro:hokuyo>
     <!-- Wheels -->
-    <xacro:sara_wheels_v1 name="wheels" parent="base"/>
-    <!-- Kinect -->
-    <xacro:kinect2 name="kinect" parent="base"/>
+    <xacro:four_mecanum_wheels parent="base" x_center="0.22735" y_center="0.2056310" sim="${sim}"/>
     <!-- Torso -->
-    <xacro:sara_torso_v1 name="torso" parent="base"/>
+    <xacro:sara_torso_v1 parent="base" sim="${sim}">
+        <origin xyz="0.177374 0 0.70531" rpy="0 0 0" />
+    </xacro:sara_torso_v1>
+    <!-- Torso Kinect -->
+    <xacro:kinect2 prefix="torso_" parent="base" sim="${sim}">
+        <origin xyz="0.177374 0 0.65676" rpy="-1.5708 0 -1.5708" />
+    </xacro:kinect2>
     <!-- Neck -->
-    <xacro:sara_neck_v1 name="neck" parent="torso"/>
+    <xacro:sara_neck_v1 parent="torso" sim="${sim}">
+        <origin xyz="0.032295 0 0.2447" rpy="0 0 0"/>
+    </xacro:sara_neck_v1>
     <!-- Head -->
-    <xacro:sara_head_v1 name="head" parent="neck"/>
+    <xacro:sara_head_v1 parent="neck" sim="${sim}">
+        <origin xyz="0 0 0.0927" rpy="-1.57 0 0"/>
+    </xacro:sara_head_v1>
+    <!-- Head Xtion -->
+    <xacro:asus_xtion prefix="head_" parent="head" sim="${sim}">
+        <origin xyz="0.0776104 -0.13 0" rpy="1.57 0 0" />
+    </xacro:asus_xtion>
     <!-- Arm -->
-    <xacro:sara_arm_v1 name="arm" parent="torso"/>
-    <!-- Gripper 85 (new)
-    <xacro:robotiq_85_gripper prefix="" parent="arm_socket_link">
-      <origin xyz="0 0 -0.02989" rpy="0 1.5708 0"/>
-    </xacro:robotiq_85_gripper>
-    -->
-    <!-- Gripper C2 (old)-->
-    <xacro:robotiq_c2_model prefix="" parent="arm_socket_link">
-      <origin xyz="0 0 -0.02989" rpy="0 1.5708 0"/>
-    </xacro:robotiq_c2_model>
+    <xacro:sara_arm_v2 prefix="right_" parent="torso" sim="${sim}">
+        <origin xyz="0 -0.145 0.189" rpy="0 -1.57 0"/>
+    </xacro:sara_arm_v2>
+    <!-- End Effector -->
+    <xacro:if value="${end_effector == 85}">
+        <!-- Gripper 85 (round base) -->
+        <xacro:include filename="$(find robotiq_85_description)/urdf/robotiq_85_gripper.urdf.xacro"/>
+        <xacro:robotiq_85_gripper prefix="right_" parent="right_socket_link">
+            <origin xyz="0 0 -0.02989" rpy="0 1.5708 0"/>
+        </xacro:robotiq_85_gripper>
+    </xacro:if>
+    <xacro:if value="${end_effector == 'C2'}">
+        <!-- Gripper C2 (old model)-->
+        <xacro:include filename="$(find robotiq_c2_model_visualization)/urdf/robotiq_c2_model_macro.xacro"/>
+        <xacro:robotiq_c2_model prefix="right_" parent="right_socket_link">
+            <origin xyz="0 0 -0.02989" rpy="0 1.5708 0"/>
+        </xacro:robotiq_c2_model>
+    </xacro:if>
 </robot>

File: urdf/torso_v1/torso.gazebo.xacro (robot description, xacro)
@@ -1,7 +1,8 @@
 <?xml version="1.0"?>
 <robot xmlns:xacro="http://ros.org/wiki/xacro">
-   <xacro:macro name="sara_torso_gazebo_v1" params="name parent">
-      <gazebo reference="${name}_link">
+   <xacro:macro name="sara_torso_gazebo_v1">
+      <gazebo reference="torso_link">
          <turnGravityOff>false</turnGravityOff>
+         <selfCollide>true</selfCollide>
       </gazebo>
    </xacro:macro>

File: urdf/torso_v1/torso.urdf.xacro (robot description, xacro)
@@ -1,8 +1,17 @@
 <?xml version="1.0"?>
 <robot xmlns:xacro="http://ros.org/wiki/xacro" >
-   <xacro:include filename="$(find sara_description)/urdf/torso_v1/torso.gazebo.xacro" />
-   <xacro:macro name="sara_torso_v1" params="name parent">
-       <xacro:sara_torso_gazebo_v1 name="${name}" parent="${parent}"/>
-       <link name="${name}_link">
+   <xacro:macro name="sara_torso_v1" params="parent *origin sim">
+       <xacro:if value="${sim}">
+           <xacro:include filename="$(find sara_description)/urdf/torso_v1/torso.gazebo.xacro" />
+           <xacro:sara_torso_gazebo_v1/>
+       </xacro:if>
+       <joint name="${parent}_torso_joint" type="fixed">
+           <parent link="${parent}_link"/>
+           <child link="torso_link"/>
+           <limit effort="1000.0" lower="0" upper="0.5" velocity="0.2"/>
+           <xacro:insert_block name="origin"/>
+           <axis xyz="0 0 1" />
+       </joint>
+       <link name="torso_link">
          <visual>
             <geometry>
@@ -26,11 +35,4 @@
          </inertial>
      </link>
-     <joint name="${parent}_${name}_joint" type="fixed">
-         <parent link="${parent}_link"/>
-         <child link="${name}_link"/>
-         <limit effort="1000.0" lower="0" upper="0.5" velocity="0.2"/>
-         <origin xyz="0.177374 0 0.70531" rpy="0 0 0" />
-         <axis xyz="0 0 1" />
-    </joint>
   </xacro:macro>
 </robot>

Commit message: New inercia matrix

File: urdf/arm_v2/arm.urdf.xacro (robot description, xacro)
@@ -34,5 +34,7 @@
          <mass value="1" />
          <origin xyz="0 0 0" rpy="0 3.1416 0" />
-         <inertia ixx="0.001" ixy="0" ixz="0" iyy="0.001" iyz="0" izz="0.001" />
+         <inertia ixx="0.0012247" ixy="0.0" ixz="0.0"
+                  iyy="0.00049634" iyz="0.0002987"
+                  izz="0.00131941" />
        </inertial>
      </link>
@@ -62,5 +64,5 @@
          <inertial>
            <mass value="1" />
-           <origin xyz="0 0 0" rpy="3.1416 0 1.5708" />
+           <origin xyz="0 0 0" rpy="3.1416 0 1.5708"/>
            <inertia ixx="0.001" ixy="0" ixz="0" iyy="0.001" iyz="0" izz="0.001" />
          </inertial>
@@ -91,6 +93,8 @@
        <inertial>
          <mass value="1" />
-         <origin xyz="0 0 0" rpy="1.5708 3.1416 3.1416" />
-         <inertia ixx="0.001" ixy="0" ixz="0" iyy="0.001" iyz="0" izz="0.001" />
+         <origin xyz="0 0 0" rpy="1.5708 3.1416 3.1416"/>
+         <inertia ixx = "0.02042044" ixy="-0.00028692" ixz="-0.00000813"
+                  iyy="0.00056723" iyz="0.00027077"
+                  izz="0.02071076" />
        </inertial>
      </link>
@@ -120,6 +124,8 @@
         <inertial>
           <mass value="1" />
-          <origin xyz="0 0 0" rpy="0 3.1416 0" />
-          <inertia ixx="0.001" ixy="0" ixz="0" iyy="0.001" iyz="0" izz="0.001" />
+          <origin xyz="0 0 -0.0005" rpy="3.1416 0 0"/>
+          <inertia ixx="0.00124099" ixy="0.0" ixz="0.0"
+                   iyy="0.00037378" iyz="0.00026280"
+                   izz="0.00135553" />
         </inertial>
       </link>
@@ -149,6 +155,8 @@
        <inertial>
          <mass value="1" />
-         <origin xyz="-0.0676 0.0676 0" rpy="-1.5708 0 -1.5708" />
-         <inertia ixx="0.001" ixy="0" ixz="0" iyy="0.001" iyz="0" izz="0.001" />
+         <origin xyz="-0.0338 0.0338 0" rpy="-1.5708 0 -1.5708" />
+         <inertia ixx="0.00037838" ixy="0.00014913" ixz="0.00014658"
+                  iyy="0.00040127" iyz="0.00015139"
+                  izz="0.00041573" />
        </inertial>
      </link>
@@ -178,6 +186,8 @@
        <inertial>
          <mass value="1" />
-         <origin xyz="-0.0676 0.0676 0" rpy="-1.5708 0 -1.5708" />
-         <inertia ixx="0.001" ixy="0" ixz="0" iyy="0.001" iyz="0" izz="0.001" />
+         <origin xyz="0.0706 0.0283 -0.030" rpy="1.5708 -1.5708 0" />
+         <inertia ixx = "0.00015783" ixy = "0.00005533" ixz = "0.00005899"
+                  iyy = "0.00016618" iyz = "0.00005219"
+                  izz = "0.00016459" />
        </inertial>
      </link>
@@ -207,6 +217,8 @@
        <inertial>
          <mass value="1" />
-         <origin xyz="-0.0676 0.0676 0" rpy="-1.5708 0 -1.5708" />
-         <inertia ixx="0.001" ixy="0" ixz="0" iyy="0.001" iyz="0" izz="0.001" />
+         <origin xyz="-0.02575  -0.01375 0.0305448" rpy="0 1.5708 0" />
+         <inertia ixx="0.00039755" ixy="0.00015393" ixz="0.0000828"
+                  iyy="0.00022585" iyz="0.00013002"
+                  izz="0.00044072" />
        </inertial>
      </link>
@@ -236,6 +248,8 @@
        <inertial>
          <mass value="1" />
-         <origin xyz="-0.0676 0.0676 0" rpy="-1.5708 0 -1.5708" />
-         <inertia ixx="0.001" ixy="0" ixz="0" iyy="0.001" iyz="0" izz="0.001" />
+         <origin xyz="0.028925 -0.025 -0.0362070" rpy="0 0 1.5708" />
+         <inertia ixx="0.00006064" ixy="0.00002022" ixz="0.00001417"
+                  iyy="0.00003787" iyz="0.0000164"
+                  izz="0.00006587" />
        </inertial>
      </link>

File: urdf/base_v2/base.urdf.xacro (robot description, xacro)
@@ -38,16 +38,9 @@
       </collision>
       <inertial>
-        <mass value="100"/>
-        <origin xyz="-0.055 0 0.227" rpy="0 0 0"/>
-        <inertia ixx="0.1" ixy="0.1" ixz="0.1"
-                 iyy="0.1" iyz="0.1"
-                 izz="0.1"/>
-      </inertial>
-      <inertial>
-        <mass value="30"/>
-        <origin xyz="0 0 0" rpy="0 0 0"/>
-        <inertia ixx="0.1" ixy="0.1" ixz="0.1"
-                 iyy="0.1" iyz="0.1"
-                 izz="0.1"/>
+        <mass value="230"/>
+          <origin xyz="-0.055 0 0.227" rpy="0 0 1.57"/>
+          <inertia ixx = "9.68458021" ixy = "2.23668848" ixz = "0.79348736"
+                   iyy = "2.66882541" iyz = "2.88061613"
+                   izz = "9.25217984"/>
       </inertial>
     </link>

File: urdf/head_v1/head.urdf.xacro (robot description, xacro)
@@ -34,5 +34,7 @@
             <mass value="5" />
             <origin xyz="0 0 0" rpy="1.5708 0 1.5708" />
-            <inertia ixx="0.001" ixy="0" ixz="0" iyy="0.001" iyz="0" izz="0.001" />
+            <inertia ixx = "0.02722768" ixy = "0.00015673" ixz = "0.0000148"
+                     iyy = "0.02716685" iyz = "0.00524002"
+                     izz = "0.04109802" />
          </inertial>
       </link>

File: urdf/neck_v1/neck.urdf.xacro (robot description, xacro)
@@ -34,5 +34,7 @@
                 <mass value="2"/>
                 <origin xyz="0 0 0" rpy="1.5708 0 1.5708"/>
-                <inertia ixx="0.001" ixy="0" ixz="0" iyy="0.001" iyz="0" izz="0.001"/>
+                <inertia ixx = "0.00438238" ixy = "0.0" ixz = "0.0"
+                         iyy = "0.0040183" iyz = "0.0"
+                         izz = "0.00585293"/>
              </inertial>
        </link>

File: urdf/sara.urdf.xacro (robot description, xacro)
@@ -56,5 +56,5 @@
     </xacro:robotiq_85_gripper>-->
     <!-- Gripper C2 (old model)-->
-    <xacro:include filename="$(find robotiq_c2_model_visualization)/urdf/robotiq_c2_model_macro.xacro"/>
+    <xacro:include filename="$(find robotiq_c2_description)/urdf/robotiq_c2_model_macro.xacro"/>
     <xacro:robotiq_c2_model prefix="right_" parent="right_socket_link">
         <origin xyz="0 0 -0.02989" rpy="0 1.5708 0"/>

File: urdf/torso_v1/torso.urdf.xacro (robot description, xacro)
@@ -32,5 +32,7 @@
             <mass value="10"/>
             <origin xyz="-0.14427 -0.197233 0" rpy="1.5708 0 1.5708"/>
-            <inertia ixx="0.001" ixy="0" ixz="0" iyy="0.001" iyz="0" izz="0.001"/>
+            <inertia ixx = "0.03994446" ixy = "0.00064933" ixz = "0.00005666"
+                     iyy = "0.04946667" iyz = "0.00660833"
+                     izz = "0.05202654"/>
          </inertial>
      </link>

Commit message: Good origins on mesh files | updated arm.urdf.xacro

File: urdf/arm_v2/arm.urdf.xacro (robot description, xacro)
@@ -142,5 +142,5 @@
            <mesh filename="package://sara_description/meshes/avant-bras.STL" scale="0.001 0.001 0.001"/>
          </geometry>
-         <origin xyz="-0.0338 0.0338 0" rpy="-1.5708 0 -1.5708" />
+         <origin xyz="0 0 0" rpy="-1.5708 0 -1.5708" />
            <material name="black">
              <color rgba="0.12 0.12 0.12 1"/>
@@ -151,5 +151,5 @@
            <mesh filename="package://sara_description/meshes/avant-bras.STL" scale="0.001 0.001 0.001"/>
          </geometry>
-           <origin xyz="-0.0338 0.0338 0" rpy="-1.5708 0 -1.5708" />
+           <origin xyz="0 0 0" rpy="-1.5708 0 -1.5708" />
        </collision>
        <inertial>
@@ -165,5 +165,5 @@
        <child link="${prefix}wrist_upper_link"/>
        <limit effort="1000.0" lower="-3.1416" upper="3.1416" velocity="0.5"/>
-       <origin xyz="0 0 -0.11184" rpy="1.5708 -1.5708 0" />
+       <origin xyz="0 0 -0.05124" rpy="1.5708 -1.5708 0" />
        <axis xyz="0 1 0" />
      </joint>
@@ -173,7 +173,7 @@
            <mesh filename="package://sara_description/meshes/poignet_haut.STL" scale="0.001 0.001 0.001"/>
          </geometry>
-         <origin xyz="0.0706 0.0283 -0.030" rpy="1.5708 -1.5708 0"/>
-         <material name="blue">
-           <color rgba="0 0 1 .06"/>
+         <origin xyz="0 0 0" rpy="1.5708 -1.5708 0"/>
+         <material name="black">
+           <color rgba="0.12 0.12 0.12 1"/>
          </material>
        </visual>
@@ -182,5 +182,5 @@
            <mesh filename="package://sara_description/meshes/poignet_haut.STL" scale="0.001 0.001 0.001"/>
          </geometry>
-         <origin xyz="0.0706 0.0283 -0.030" rpy="1.5708 -1.5708 0"/>
+         <origin xyz="0 0 0" rpy="1.5708 -1.5708 0"/>
        </collision>
        <inertial>
@@ -196,5 +196,5 @@
        <child link="${prefix}wrist_lower_link"/>
        <limit effort="1000.0" lower="-1.5708" upper="1.5708" velocity="0.5"/>
-       <origin xyz="0 0 0" rpy="1.5708 -1.5708 0" />
+       <origin xyz="-0.0606 0 0" rpy="1.5708 -1.5708 0" />
        <axis xyz="0 0 1" />
      </joint>
@@ -204,5 +204,5 @@
            <mesh filename="package://sara_description/meshes/poignet_bas.STL" scale="0.001 0.001 0.001"/>
          </geometry>
-         <origin xyz="-0.02575  -0.01375 0.0305448" rpy=" 0 1.5708 0"/>
+         <origin xyz="0 0 0" rpy=" 0 1.5708 0"/>
          <material name="black">
            <color rgba="0.12 0.12 0.12 1"/>
@@ -213,5 +213,5 @@
            <mesh filename="package://sara_description/meshes/poignet_bas.STL" scale="0.001 0.001 0.001"/>
          </geometry>
-         <origin xyz="-0.02575  -0.01375 0.0305448" rpy=" 0 1.5708 0"/>
+         <origin xyz="0 0 0" rpy=" 0 1.5708 0"/>
        </collision>
        <inertial>
@@ -233,14 +233,14 @@
        <visual>
          <geometry>
-           <mesh filename="package://sara_description/meshes/attache-pince.STL" scale="0.001 0.001 0.001"/>
-         </geometry>
-         <origin xyz="0.028925 -0.025 -0.0362070" rpy="0 0 1.5708"/>
-         <material name="black">
-           <color rgba="0.12 0.12 0.12 1"/>
-         </material>
-       </visual>
-       <collision>
-         <geometry>
-           <mesh filename="package://sara_description/meshes/attache-pince.STL" scale="0.001 0.001 0.001"/>
+           <mesh filename="package://sara_description/meshes/attache_pince.STL" scale="0.001 0.001 0.001"/>
+         </geometry>
+         <origin xyz="0 0 0" rpy="0 0 1.5708"/>
+         <material name="black">
+           <color rgba="0.12 0.12 0.12 1"/>
+         </material>
+       </visual>
+       <collision>
+         <geometry>
+           <mesh filename="package://sara_description/meshes/attache_pince.STL" scale="0.001 0.001 0.001"/>
          </geometry>
          <origin xyz="0.028925 -0.025 -0.0362070" rpy="0 0 1.5708"/>

Commit message: Corrected center of mass in wrist and forarm

File: urdf/arm_v2/arm.urdf.xacro (robot description, xacro)
@@ -33,8 +33,8 @@
        <inertial>
          <mass value="1" />
-         <origin xyz="0 0 0" rpy="0 3.1416 0" />
-         <inertia ixx="0.0012247" ixy="0.0" ixz="0.0"
-                  iyy="0.00049634" iyz="0.0002987"
-                  izz="0.00131941" />
+         <origin xyz="0 -0.05029668 0.01842530" rpy="0 3.1416 0" />
+         <inertia ixx = "0.00040675" ixy="0.0" ixz="0.0"
+                  iyy = "0.00039956" iyz = "0.00003451"
+                  izz = "0.00059825" />
        </inertial>
      </link>
@@ -155,8 +155,8 @@
        <inertial>
          <mass value="1" />
-         <origin xyz="-0.0338 0.0338 0" rpy="-1.5708 0 -1.5708" />
-         <inertia ixx="0.00037838" ixy="0.00014913" ixz="0.00014658"
-                  iyy="0.00040127" iyz="0.00015139"
-                  izz="0.00041573" />
+         <origin xyz="-0.00000184 0.03625492 0.0" rpy="-1.5708 0 -1.5708" />
+         <inertia ixx = "0.00007571" ixy = "0.0" ixz = "0.0"
+                  iyy = "0.00010905" iyz = "0.0"
+                  izz = "0.00011768" />
        </inertial>
      </link>
@@ -186,8 +186,8 @@
        <inertial>
          <mass value="1" />
-         <origin xyz="0.0706 0.0283 -0.030" rpy="1.5708 -1.5708 0" />
-         <inertia ixx = "0.00015783" ixy = "0.00005533" ixz = "0.00005899"
-                  iyy = "0.00016618" iyz = "0.00005219"
-                  izz = "0.00016459" />
+         <origin xyz="0.00000283 0.03890077 0.00017201" rpy="1.5708 -1.5708 0"/>
+         <inertia ixx = "0.00013274" ixy = "0.0" ixz = "0.0"
+                  iyy = "0.00007056" iyz = "0.00000150"
+                  izz = "0.00011649" />
        </inertial>
      </link>
@@ -217,8 +217,8 @@
        <inertial>
          <mass value="1" />
-         <origin xyz="-0.02575  -0.01375 0.0305448" rpy="0 1.5708 0" />
-         <inertia ixx="0.00039755" ixy="0.00015393" ixz="0.0000828"
-                  iyy="0.00022585" iyz="0.00013002"
-                  izz="0.00044072" />
+         <origin xyz="0.0 0.06377326 -0.000001541" rpy=" 0 1.5708 0"/>
+         <inertia ixx = "0.00009654" ixy = "0.0" ixz = "0.0"
+                  iyy = "0.00004298" iyz = "0.00000061"
+                  izz = "0.00009099" />
        </inertial>
      </link>
@@ -248,8 +248,8 @@
        <inertial>
          <mass value="1" />
-         <origin xyz="0.028925 -0.025 -0.0362070" rpy="0 0 1.5708" />
-         <inertia ixx="0.00006064" ixy="0.00002022" ixz="0.00001417"
-                  iyy="0.00003787" iyz="0.0000164"
-                  izz="0.00006587" />
+         <origin xyz="0.0157046 0.0 0.0" rpy="0 0 1.5708"/>
+         <inertia ixx = "0.00000933" ixy = "0.0" ixz = "0.0"
+                  iyy = "0.00000332" iyz = "0.0"
+                  izz = "0.00000955" />
        </inertial>
      </link>
