Commit message: New origins on all parts

File: urdf/arm_v2/arm.urdf.xacro (robot description, xacro)
@@ -18,14 +18,14 @@
        <visual>
          <geometry>
-           <mesh filename="package://sara_description/meshes/epaule.STL" scale="0.001 0.001 0.001"/>
-         </geometry>
-         <origin xyz="0 0 0" rpy="0 3.1416 0"/>
-         <material name="black">
-           <color rgba="0.12 0.12 0.12 1"/>
-         </material>
-       </visual>
-       <collision>
-         <geometry>
-           <mesh filename="package://sara_description/meshes/epaule.STL" scale="0.001 0.001 0.001"/>
+           <mesh filename="package://sara_description/meshes/epaule1.STL" scale="0.001 0.001 0.001"/>
+         </geometry>
+         <origin xyz="0 0 0" rpy="0 0 0"/>
+         <material name="black">
+           <color rgba="0.12 0.12 0.12 1"/>
+         </material>
+       </visual>
+       <collision>
+         <geometry>
+           <mesh filename="package://sara_description/meshes/epaule1.STL" scale="0.001 0.001 0.001"/>
          </geometry>
            <origin xyz="0 0 0" rpy="0 3.1416 0"/>
@@ -49,7 +49,7 @@
        <visual>
          <geometry>
-           <mesh filename="package://sara_description/meshes/epaule.STL" scale="0.001 0.001 0.001"/>
-         </geometry>
-           <origin xyz="0 0 0" rpy="3.1416 0 1.5708"/>
+           <mesh filename="package://sara_description/meshes/epaule2.STL" scale="0.001 0.001 0.001"/>
+         </geometry>
+           <origin xyz="0 0 0" rpy="0 0 0"/>
            <material name="black">
              <color rgba="0.12 0.12 0.12 1"/>
@@ -58,7 +58,7 @@
        <collision>
          <geometry>
-           <mesh filename="package://sara_description/meshes/epaule.STL" scale="0.001 0.001 0.001"/>
-         </geometry>
-           <origin xyz="0 0 0" rpy="3.1416 0 1.5708"/>
+           <mesh filename="package://sara_description/meshes/epaule2.STL" scale="0.001 0.001 0.001"/>
+         </geometry>
+           <origin xyz="0 0 0" rpy="0 0 0"/>
          </collision>
          <inertial>
@@ -80,5 +80,5 @@
            <mesh filename="package://sara_description/meshes/bras_haut.STL" scale="0.001 0.001 0.001"/>
          </geometry>
-         <origin xyz="0 0 0" rpy="1.5708 3.1416 3.1416"/>
+         <origin xyz="0 0 0" rpy="0 0 0"/>
          <material name="black">
            <color rgba="0.12 0.12 0.12 1"/>
@@ -111,5 +111,5 @@
             <mesh filename="package://sara_description/meshes/coude.STL" scale="0.001 0.001 0.001"/>
           </geometry>
-            <origin xyz="0 0 -0.0005" rpy="3.1416 0 0"/>
+            <origin xyz="0 0 -0.0005" rpy="0 0 0"/>
             <material name="black">
               <color rgba="0.12 0.12 0.12 1"/>
@@ -140,7 +140,7 @@
        <visual>
          <geometry>
-           <mesh filename="package://sara_description/meshes/avant-bras.STL" scale="0.001 0.001 0.001"/>
-         </geometry>
-         <origin xyz="0 0 0" rpy="-1.5708 0 -1.5708" />
+           <mesh filename="package://sara_description/meshes/avant_bras.STL" scale="0.001 0.001 0.001"/>
+         </geometry>
+         <origin xyz="0 0 0" rpy="0 0 0" />
            <material name="black">
              <color rgba="0.12 0.12 0.12 1"/>
@@ -149,5 +149,5 @@
        <collision>
          <geometry>
-           <mesh filename="package://sara_description/meshes/avant-bras.STL" scale="0.001 0.001 0.001"/>
+           <mesh filename="package://sara_description/meshes/avant_bras.STL" scale="0.001 0.001 0.001"/>
          </geometry>
            <origin xyz="0 0 0" rpy="-1.5708 0 -1.5708" />
@@ -173,5 +173,5 @@
            <mesh filename="package://sara_description/meshes/poignet_haut.STL" scale="0.001 0.001 0.001"/>
          </geometry>
-         <origin xyz="0 0 0" rpy="1.5708 -1.5708 0"/>
+         <origin xyz="0 0 0" rpy="0 0 0"/>
          <material name="black">
            <color rgba="0.12 0.12 0.12 1"/>
@@ -204,5 +204,5 @@
            <mesh filename="package://sara_description/meshes/poignet_bas.STL" scale="0.001 0.001 0.001"/>
          </geometry>
-         <origin xyz="0 0 0" rpy=" 0 1.5708 0"/>
+         <origin xyz="0 0 0" rpy=" 0 0 0"/>
          <material name="black">
            <color rgba="0.12 0.12 0.12 1"/>
@@ -235,5 +235,5 @@
            <mesh filename="package://sara_description/meshes/attache_pince.STL" scale="0.001 0.001 0.001"/>
          </geometry>
-         <origin xyz="0 0 0" rpy="0 0 1.5708"/>
+         <origin xyz="0 0 0" rpy="0 0 0"/>
          <material name="black">
            <color rgba="0.12 0.12 0.12 1"/>

Commit message: It works! arm.urdf.xacro new inertias

File: urdf/arm_v2/arm.urdf.xacro (robot description, xacro)
@@ -29,11 +29,11 @@
            <mesh filename="package://sara_description/meshes/epaule1.STL" scale="0.001 0.001 0.001"/>
          </geometry>
-           <origin xyz="0 0 0" rpy="0 3.1416 0"/>
-       </collision>
-       <inertial>
-         <mass value="1" />
-         <origin xyz="0 -0.05029668 0.01842530" rpy="0 3.1416 0" />
-         <inertia ixx = "0.00040675" ixy="0.0" ixz="0.0"
-                  iyy = "0.00039956" iyz = "0.00003451"
+           <origin xyz="0 0 0" rpy="0 0 0"/>
+       </collision>
+       <inertial>
+         <mass value="0.28506911" />
+         <origin xyz="0.0 -0.03225261 -0.01842117" rpy="0 0 0" />
+         <inertia ixx = "0.00040678" ixy="0.0" ixz = "-0.00000004"
+                  iyy = "0.00039958" iyz = "-0.00003453"
                   izz = "0.00059825" />
        </inertial>
@@ -63,7 +63,7 @@
          </collision>
          <inertial>
-           <mass value="1" />
-           <origin xyz="0 0 0" rpy="3.1416 0 1.5708"/>
-           <inertia ixx="0.001" ixy="0" ixz="0" iyy="0.001" iyz="0" izz="0.001" />
+           <mass value="0.28506911" />
+           <origin xyz="-0.03225261 0 -0.01842117" rpy="0 0 0"/>
+           <inertia ixx = "0.00039958" ixy="0" ixz = "-0.00003453" iyy = "0.00040678" iyz = "0.00000004" izz = "0.00059825" />
          </inertial>
      </link>
@@ -89,12 +89,12 @@
            <mesh filename="package://sara_description/meshes/bras_haut.STL" scale="0.001 0.001 0.001"/>
          </geometry>
-         <origin xyz="0 0 0" rpy="1.5708 3.1416 3.1416"/>
-       </collision>
-       <inertial>
-         <mass value="1" />
-         <origin xyz="0 0 0" rpy="1.5708 3.1416 3.1416"/>
-         <inertia ixx = "0.02042044" ixy="-0.00028692" ixz="-0.00000813"
-                  iyy="0.00056723" iyz="0.00027077"
-                  izz="0.02071076" />
+         <origin xyz="0 0 0" rpy="0 0 0"/>
+       </collision>
+       <inertial>
+         <mass value="0.85240803" />
+         <origin xyz="-0.00168302 0.00155140 -0.13913505" rpy="0 0 0"/>
+         <inertia ixx = "0.00538199" ixy = "-0.00000635" ixz = "0.00012863"
+                  iyy = "0.00562525" iyz = "-0.00012986"
+                  izz = "0.00050159" />
        </inertial>
      </link>
@@ -120,12 +120,12 @@
             <mesh filename="package://sara_description/meshes/coude.STL" scale="0.001 0.001 0.001"/>
           </geometry>
-          <origin xyz="0 0 -0.0005" rpy="3.1416 0 0"/>
+          <origin xyz="0 0 0" rpy="0 0 0"/>
         </collision>
         <inertial>
-          <mass value="1" />
-          <origin xyz="0 0 -0.0005" rpy="3.1416 0 0"/>
-          <inertia ixx="0.00124099" ixy="0.0" ixz="0.0"
-                   iyy="0.00037378" iyz="0.00026280"
-                   izz="0.00135553" />
+          <mass value="0.28300045" />
+          <origin xyz="0.00000207 0.03922132 -0.01628605" rpy="0 0 0"/>
+          <inertia ixx = "0.00036109" ixy = "0.0" ixz = "-0.00000002"
+                   iyy = "0.00029872" iyz = "0.00001701"
+                   izz = "0.00055069" />
         </inertial>
       </link>
@@ -151,12 +151,12 @@
            <mesh filename="package://sara_description/meshes/avant_bras.STL" scale="0.001 0.001 0.001"/>
          </geometry>
-           <origin xyz="0 0 0" rpy="-1.5708 0 -1.5708" />
-       </collision>
-       <inertial>
-         <mass value="1" />
-         <origin xyz="-0.00000184 0.03625492 0.0" rpy="-1.5708 0 -1.5708" />
-         <inertia ixx = "0.00007571" ixy = "0.0" ixz = "0.0"
-                  iyy = "0.00010905" iyz = "0.0"
-                  izz = "0.00011768" />
+           <origin xyz="0 0 0" rpy="0 0 0"/>
+       </collision>
+       <inertial>
+         <mass value="0.1177" />
+         <origin xyz="0.0 -0.00000184 -0.03625492" rpy="0 0 0" />
+         <inertia ixx = "0.54274952" ixy = "0.0" ixz = "0.0"
+                  iyy = "1.03078569" iyz = "0.0"
+                  izz = "0.00010905" />
        </inertial>
      </link>
@@ -182,12 +182,12 @@
            <mesh filename="package://sara_description/meshes/poignet_haut.STL" scale="0.001 0.001 0.001"/>
          </geometry>
-         <origin xyz="0 0 0" rpy="1.5708 -1.5708 0"/>
-       </collision>
-       <inertial>
-         <mass value="1" />
-         <origin xyz="0.00000283 0.03890077 0.00017201" rpy="1.5708 -1.5708 0"/>
-         <inertia ixx = "0.00013274" ixy = "0.0" ixz = "0.0"
-                  iyy = "0.00007056" iyz = "0.00000150"
-                  izz = "0.00011649" />
+         <origin xyz="0 0 0" rpy="0 0 0"/>
+       </collision>
+       <inertial>
+         <mass value="0.1956991" />
+         <origin xyz="-0.03893593 0.00017228 -0.00000284" rpy="0 0 0"/>
+         <inertia ixx = "0.00007035" ixy = "-0.00000150" ixz = "0.0"
+                  iyy = "0.00011510" iyz = "0.0"
+                  izz = "0.00013235" />
        </inertial>
      </link>
@@ -213,12 +213,12 @@
            <mesh filename="package://sara_description/meshes/poignet_bas.STL" scale="0.001 0.001 0.001"/>
          </geometry>
-         <origin xyz="0 0 0" rpy=" 0 1.5708 0"/>
-       </collision>
-       <inertial>
-         <mass value="1" />
-         <origin xyz="0.0 0.06377326 -0.000001541" rpy=" 0 1.5708 0"/>
-         <inertia ixx = "0.00009654" ixy = "0.0" ixz = "0.0"
-                  iyy = "0.00004298" iyz = "0.00000061"
-                  izz = "0.00009099" />
+         <origin xyz="0 0 0" rpy="0 0 0"/>
+       </collision>
+       <inertial>
+         <mass value="0.18747684" />
+         <origin xyz="0.00001243 0.05721169 0.0" rpy=" 0 0 0"/>
+         <inertia ixx = "0.00015391" ixy = "-0.00000060" ixz = "0.0"
+                  iyy = "0.00006260" iyz = "0.0"
+                  izz = "0.00015218" />
        </inertial>
      </link>
@@ -244,12 +244,12 @@
            <mesh filename="package://sara_description/meshes/attache_pince.STL" scale="0.001 0.001 0.001"/>
          </geometry>
-         <origin xyz="0.028925 -0.025 -0.0362070" rpy="0 0 1.5708"/>
-       </collision>
-       <inertial>
-         <mass value="1" />
-         <origin xyz="0.0157046 0.0 0.0" rpy="0 0 1.5708"/>
-         <inertia ixx = "0.00000933" ixy = "0.0" ixz = "0.0"
-                  iyy = "0.00000332" iyz = "0.0"
-                  izz = "0.00000955" />
+         <origin xyz="0 0 0" rpy="0 0 0"/>
+       </collision>
+       <inertial>
+         <mass value="0.02796" />
+         <origin xyz="0.0 0.0 -0.01570460" rpy="0 0 0"/>
+         <inertia ixx = "0.00000889" ixy = "0.0" ixz = "0.0"
+                  iyy= "0.00002569" iyz = "0.0"
+                  izz = "0.00002493" />
        </inertial>
      </link>

Commit message: Added new mass taken frome solidwork

File: urdf/arm_v2/arm.urdf.xacro (robot description, xacro)
@@ -11,5 +11,6 @@
        <parent link="${parent}_link"/>
        <child link="${prefix}clavicular_link"/>
-       <limit effort="1000.0" lower="-1.6" upper="1.4" velocity="0.5"/>
+       <dynamics damping="0.1"/>
+       <limit effort="10000.0" lower="-1.6" upper="1.4" velocity="0.5"/>
        <xacro:insert_block name="origin"/>
        <axis xyz="0 0 1" />
@@ -42,5 +43,6 @@
        <parent link="${prefix}clavicular_link"/>
        <child link="${prefix}upper_arm_upper_link"/>
-       <limit effort="1000.0" lower="-4.7124" upper="1.5708" velocity="0.5"/>
+       <dynamics damping="0.1"/>
+       <limit effort="10000.0" lower="-4.7124" upper="1.5708" velocity="0.5"/>
        <origin xyz="0 -0.085 0" rpy="-1.57 0 0" />
        <axis xyz="0 0 1" />
@@ -71,5 +73,6 @@
        <parent link="${prefix}upper_arm_upper_link"/>
        <child link="${prefix}upper_arm_lower_link"/>
-       <limit effort="1000.0" lower="-3.1416" upper="3.1416" velocity="0.5"/>
+       <dynamics damping="0.1"/>
+       <limit effort="10000.0" lower="-3.1416" upper="3.1416" velocity="0.5"/>
        <origin xyz="-0.085 0 0" rpy="1.5708 0 1.5708" />
        <axis xyz="0 0 1" />
@@ -102,5 +105,6 @@
         <parent link="${prefix}upper_arm_lower_link"/>
         <child link="${prefix}forearm_upper_link"/>
-        <limit effort="1000.0" lower="-2.20" upper="1.90" velocity="0.5"/>
+        <dynamics damping="0.1"/>
+        <limit effort="10000.0" lower="-2.20" upper="1.90" velocity="0.5"/>
         <origin xyz="0 0 -0.31" rpy="-1.5708 0 0" />
         <axis xyz="0 0 1" />
@@ -133,5 +137,6 @@
        <parent link="${prefix}forearm_upper_link"/>
        <child link="${prefix}forearm_lower_link"/>
-       <limit effort="1000.0" lower="-3.1416" upper="3.1416" velocity="0.5"/>
+       <dynamics damping="0.1"/>
+       <limit effort="10000.0" lower="-3.1416" upper="3.1416" velocity="0.5"/>
        <origin xyz="0 0.0945 0" rpy="1.5708 -1.5708 0" />
        <axis xyz="0 0 1" />
@@ -164,5 +169,5 @@
        <parent link="${prefix}forearm_lower_link"/>
        <child link="${prefix}wrist_upper_link"/>
-       <limit effort="1000.0" lower="-3.1416" upper="3.1416" velocity="0.5"/>
+       <limit effort="10000.0" lower="-3.1416" upper="3.1416" velocity="0.5"/>
        <origin xyz="0 0 -0.05124" rpy="1.5708 -1.5708 0" />
        <axis xyz="0 1 0" />
@@ -195,5 +200,6 @@
        <parent link="${prefix}wrist_upper_link"/>
        <child link="${prefix}wrist_lower_link"/>
-       <limit effort="1000.0" lower="-1.5708" upper="1.5708" velocity="0.5"/>
+       <dynamics damping="0.1"/>
+       <limit effort="10000.0" lower="-1.5708" upper="1.5708" velocity="0.5"/>
        <origin xyz="-0.0606 0 0" rpy="1.5708 -1.5708 0" />
        <axis xyz="0 0 1" />
@@ -226,5 +232,6 @@
        <parent link="${prefix}wrist_lower_link"/>
        <child link="${prefix}socket_link"/>
-       <limit effort="1000.0" lower="-1.49" upper="1.49" velocity="0.5"/>
+       <dynamics damping="0.1"/>
+       <limit effort="10000.0" lower="-1.49" upper="1.49" velocity="0.5"/>
        <origin xyz="0 0.084375 0" rpy="1.5708 0 0" />
        <axis xyz="1 0 0" />

File: urdf/base_v2/base.urdf.xacro (robot description, xacro)
@@ -38,6 +38,6 @@
       </collision>
       <inertial>
-        <mass value="230"/>
-          <origin xyz="-0.055 0 0.227" rpy="0 0 1.57"/>
+        <mass value="40"/>
+          <origin xyz="-0.055 0 0.227" rpy="-1.57 0 1.57"/>
           <inertia ixx = "9.68458021" ixy = "2.23668848" ixz = "0.79348736"
                    iyy = "2.66882541" iyz = "2.88061613"

File: urdf/head_v1/head.urdf.xacro (robot description, xacro)
@@ -32,5 +32,5 @@
          </collision>
          <inertial>
-            <mass value="5" />
+            <mass value="2.60401968" />
             <origin xyz="0 0 0" rpy="1.5708 0 1.5708" />
             <inertia ixx = "0.02722768" ixy = "0.00015673" ixz = "0.0000148"

File: urdf/torso_v1/torso.urdf.xacro (robot description, xacro)
@@ -30,5 +30,5 @@
          </collision>
          <inertial>
-            <mass value="10"/>
+            <mass value="4.17008957"/>
             <origin xyz="-0.14427 -0.197233 0" rpy="1.5708 0 1.5708"/>
             <inertia ixx = "0.03994446" ixy = "0.00064933" ixz = "0.00005666"

File: urdf/xtion/xtion.urdf.xacro (robot description, xacro)
@@ -24,10 +24,4 @@
           </geometry>
         </visual>
-        <collision>
-          <origin xyz="0 0 0" rpy="1.5708 0 1.5708" />
-          <geometry>
-            <box size="0.035 0.185 0.025"/>
-          </geometry>
-        </collision>
       </link>
     </xacro:macro>

Commit message: Modified links

File: urdf/arm_v2/arm.urdf.xacro (robot description, xacro)
@@ -197,4 +197,67 @@
        </inertial>
      </link>
+     <joint name="${prefix}support_xtion_joint" type="fixed">
+       <parent link="${prefix}wrist_upper_link"/>
+       <child link="${prefix}xtion_support_link"/>
+       <limit effort="10000.0" lower="-3.1416" upper="3.1416" velocity="0.5"/>
+       <origin xyz="0 0.0216704 0" rpy="0 0 0" />
+       <axis xyz="0 1 0" />
+     </joint>
+     <link name="${prefix}xtion_support_link">
+       <visual>
+         <geometry>
+           <mesh filename="package://sara_description/meshes/support_poignet.STL" scale="0.001 0.001 0.001"/>
+         </geometry>
+         <origin xyz="0 0 0" rpy="0 0 0"/>
+         <material name="black">
+           <color rgba="0.12 0.12 0.12 1"/>
+         </material>
+       </visual>
+       <collision>
+         <geometry>
+           <mesh filename="package://sara_description/meshes/support_poignet.STL" scale="0.001 0.001 0.001"/>
+         </geometry>
+         <origin xyz="0 0 0" rpy="0 0 0"/>
+       </collision>
+       <inertial>
+         <mass value="0" />
+         <origin xyz="0 0 0" rpy="0 0 0"/>
+         <inertia ixx = "0" ixy = "0" ixz = "0"
+                  iyy = "0" iyz = "0"
+                  izz = "0" />
+       </inertial>
+     </link>
+     <joint name="xtion_joint" type="fixed">
+       <parent link="${prefix}xtion_support_link"/>
+       <child link="${prefix}xtion_link"/>
+       <dynamics damping="0.1"/>
+       <limit effort="10000.0" lower="-1.5708" upper="1.5708" velocity="0.5"/>
+       <origin xyz="0.0115 0.035 0" rpy="0 0 0" />
+       <axis xyz="0 0 1" />
+     </joint>
+     <link name="${prefix}xtion_link">
+       <visual>
+         <geometry>
+           <mesh filename="package://sara_description/meshes/xtion_bras.STL" scale="0.001 0.001 0.001"/>
+         </geometry>
+         <origin xyz="0 0 0" rpy="0 0 0"/>
+         <material name="black">
+           <color rgba="0.12 0.12 0.12 1"/>
+         </material>
+       </visual>
+       <collision>
+         <geometry>
+           <mesh filename="package://sara_description/meshes/xtion_bras.STL" scale="0.001 0.001 0.001"/>
+         </geometry>
+         <origin xyz="0 0 0" rpy="0 0 0"/>
+       </collision>
+       <inertial>
+         <mass value="0" />
+         <origin xyz="0 0 0" rpy="0 0 0"/>
+         <inertia ixx = "0" ixy = "0" ixz = "0"
+                  iyy = "0" iyz = "0"
+                  izz = "0" />
+       </inertial>
+     </link>
      <joint name="${prefix}wrist_pitch_joint" type="revolute">
        <parent link="${prefix}wrist_upper_link"/>

File: urdf/base_v2/base.urdf.xacro (robot description, xacro)
@@ -11,14 +11,5 @@
             <mesh filename="package://sara_description/meshes/base.STL" scale="0.001 0.001 0.001"/>
          </geometry>
-         <origin xyz="0.295 -0.250 0.85635" rpy="-1.57 0 1.57"/>
-         <material name="black">
-               <color rgba="0.12 0.12 0.12 1"/>
-         </material>
-      </visual>
-      <visual>
-         <geometry>
-              <box size="0.4 0.35635 0.454"/>
-         </geometry>
-         <origin xyz="-0.055 0 0.227" rpy="0 0 0"/>
+         <origin xyz="0 0 0" rpy="-1.57 0 1.57"/>
          <material name="black">
                <color rgba="0.12 0.12 0.12 1"/>
@@ -29,5 +20,5 @@
             <mesh filename="package://sara_description/meshes/base.STL" scale="0.001 0.001 0.001"/>
          </geometry>
-         <origin xyz="0.295 -0.250 0.85635" rpy="-1.57 0 1.57"/>
+         <origin xyz="0 0 0" rpy="-1.57 0 1.57"/>
       </collision>
       <collision>

File: urdf/sara.urdf.xacro (robot description, xacro)
@@ -27,13 +27,13 @@
     <!-- Torso -->
     <xacro:sara_torso_v1 parent="base" sim="${sim}">
-        <origin xyz="0.177374 0 0.70531" rpy="0 0 0" />
+        <origin xyz="0.1749806 0 1.189" rpy="0 0 0" />
     </xacro:sara_torso_v1>
     <!-- Torso Kinect -->
     <xacro:kinect2 prefix="torso_" parent="base" sim="${sim}">
-        <origin xyz="0.177374 0 0.65676" rpy="-1.5708 0 -1.5708" />
+        <origin xyz="0 0 0" rpy="-1.5708 0 -1.5708" />
     </xacro:kinect2>
     <!-- Neck -->
     <xacro:sara_neck_v1 parent="torso" sim="${sim}">
-        <origin xyz="0.032295 0 0.2777" rpy="0 0 0"/>
+        <origin xyz="0 0 0.10036" rpy="0 0 0"/>
     </xacro:sara_neck_v1>
     <!-- Head -->
@@ -43,9 +43,9 @@
     <!-- Head Xtion -->
     <xacro:asus_xtion prefix="head_" parent="head" sim="${sim}">
-        <origin xyz="0.0776104 -0.13 0" rpy="1.57 0 0" />
+        <origin xyz="0.1008657 0 0.10601" rpy="1.57 0 0" />
     </xacro:asus_xtion>
     <!-- Arm -->
     <xacro:sara_arm_v2 prefix="right_" parent="torso" sim="${sim}">
-        <origin xyz="0 -0.145 0.189" rpy="0 -1.57 0"/>
+        <origin xyz="0 -0.1437625 0.01166" rpy="0 -1.57 0"/>
     </xacro:sara_arm_v2>
     <!-- End Effector -->

File: urdf/torso_v1/torso.urdf.xacro (robot description, xacro)
@@ -18,5 +18,5 @@
                <mesh filename="package://sara_description/meshes/torse.STL" scale="0.001 0.001 0.001"/>
             </geometry>
-            <origin xyz="-0.14427 -0.197233 0" rpy="1.5708 0 1.5708"/>
+            <origin xyz="0 0 0" rpy="0 0 0"/>
             <material name="black">
                <color rgba="0.12 0.12 0.12 1"/>

Commit message: updated tf for arm_xtion

File: urdf/arm_v2/arm.urdf.xacro (robot description, xacro)
@@ -233,5 +233,5 @@
        <dynamics damping="0.1"/>
        <limit effort="10000.0" lower="-1.5708" upper="1.5708" velocity="0.5"/>
-       <origin xyz="0.0115 0.035 0" rpy="0 0 0" />
+       <origin xyz="0.0115 0.035 0" rpy="1.5708 0 3.14" />
        <axis xyz="0 0 1" />
      </joint>
