Commit message: functional plugin for arm_xtion need to set the right orientation for the referentials

File: urdf/arm_v2/arm.urdf.xacro (robot description, xacro)
@@ -197,67 +197,4 @@
        </inertial>
      </link>
-     <joint name="${prefix}support_xtion_joint" type="fixed">
-       <parent link="${prefix}wrist_upper_link"/>
-       <child link="${prefix}xtion_support_link"/>
-       <limit effort="10000.0" lower="-3.1416" upper="3.1416" velocity="0.5"/>
-       <origin xyz="0 0.0216704 0" rpy="0 0 0" />
-       <axis xyz="0 1 0" />
-     </joint>
-     <link name="${prefix}xtion_support_link">
-       <visual>
-         <geometry>
-           <mesh filename="package://sara_description/meshes/support_poignet.STL" scale="0.001 0.001 0.001"/>
-         </geometry>
-         <origin xyz="0 0 0" rpy="0 0 0"/>
-         <material name="black">
-           <color rgba="0.12 0.12 0.12 1"/>
-         </material>
-       </visual>
-       <collision>
-         <geometry>
-           <mesh filename="package://sara_description/meshes/support_poignet.STL" scale="0.001 0.001 0.001"/>
-         </geometry>
-         <origin xyz="0 0 0" rpy="0 0 0"/>
-       </collision>
-       <inertial>
-         <mass value="0" />
-         <origin xyz="0 0 0" rpy="0 0 0"/>
-         <inertia ixx = "0" ixy = "0" ixz = "0"
-                  iyy = "0" iyz = "0"
-                  izz = "0" />
-       </inertial>
-     </link>
-     <joint name="xtion_joint" type="fixed">
-       <parent link="${prefix}xtion_support_link"/>
-       <child link="${prefix}xtion_link"/>
-       <dynamics damping="0.1"/>
-       <limit effort="10000.0" lower="-1.5708" upper="1.5708" velocity="0.5"/>
-       <origin xyz="0.0115 0.035 0" rpy="1.5708 0 3.14" />
-       <axis xyz="0 0 1" />
-     </joint>
-     <link name="${prefix}xtion_link">
-       <visual>
-         <geometry>
-           <mesh filename="package://sara_description/meshes/xtion_bras.STL" scale="0.001 0.001 0.001"/>
-         </geometry>
-         <origin xyz="0 0 0" rpy="0 0 0"/>
-         <material name="black">
-           <color rgba="0.12 0.12 0.12 1"/>
-         </material>
-       </visual>
-       <collision>
-         <geometry>
-           <mesh filename="package://sara_description/meshes/xtion_bras.STL" scale="0.001 0.001 0.001"/>
-         </geometry>
-         <origin xyz="0 0 0" rpy="0 0 0"/>
-       </collision>
-       <inertial>
-         <mass value="0" />
-         <origin xyz="0 0 0" rpy="0 0 0"/>
-         <inertia ixx = "0" ixy = "0" ixz = "0"
-                  iyy = "0" iyz = "0"
-                  izz = "0" />
-       </inertial>
-     </link>
      <joint name="${prefix}wrist_pitch_joint" type="revolute">
        <parent link="${prefix}wrist_upper_link"/>

File: urdf/head_xtion/head_xtion.urdf.xacro (robot description, xacro)
@@ -2,5 +2,5 @@
 <robot xmlns:xacro="http://ros.org/wiki/xacro">
     <xacro:property name="M_PI" value="3.1415926535897931" />
-    <xacro:macro name="asus_xtion" params="prefix parent *origin sim">
+    <xacro:macro name="asus_head_xtion" params="prefix parent *origin sim">
         <xacro:if value="${sim}">
             <xacro:include filename="$(find sara_description)/urdf/head_xtion/head_xtion.gazebo.xacro" />

File: urdf/sara.urdf.xacro (robot description, xacro)
@@ -13,4 +13,5 @@
     <xacro:include filename="$(find sara_description)/urdf/hokuyo/hokuyo.urdf.xacro"/>
     <xacro:include filename="$(find sara_description)/urdf/mecanum_wheel/mecanum_wheel.urdf.xacro"/>
+    <xacro:include filename="$(find sara_description)/urdf/arm_xtion/arm_xtion.urdf.xacro"/>
     <xacro:if value="${sim}">
         <xacro:include filename="$(find sara_description)/urdf/sara.gazebo.xacro" />
@@ -42,11 +43,15 @@
     </xacro:sara_head_v1>
     <!-- Head Xtion -->
-    <xacro:asus_xtion prefix="head_" parent="head" sim="${sim}">
+    <xacro:asus_head_xtion prefix="head_" parent="head" sim="${sim}">
         <origin xyz="0.0776104 -0.13 0" rpy="1.57 0 0" />0.1008657
-    </xacro:asus_xtion>
+    </xacro:asus_head_xtion>
     <!-- Arm -->
     <xacro:sara_arm_v2 prefix="right_" parent="torso" sim="${sim}">
         <origin xyz="0 -0.1437625 0.01166" rpy="0 -1.57 0"/>
     </xacro:sara_arm_v2>
+    <!-- Arm xtion -->
+    <xacro:asus_arm_xtion prefix="right_" parent="right_wrist_upper_link" sim="${sim}">
+        <origin xyz="0 0.0216704 0" rpy="0 0 0" />0.1008657
+    </xacro:asus_arm_xtion>
     <!-- End Effector -->
     <!-- Gripper 85 (round base)

Commit message: New gripper. Have to fix TF problem

File: urdf/arm_v2/arm.urdf.xacro (robot description, xacro)
@@ -261,4 +261,12 @@
        </inertial>
      </link>
+     <joint name="${prefix}gripper_joint" type="fixed">
+       <parent link="${prefix}socket_link"/>
+       <child link="${prefix}robotiq_arg2f_base_link"/>
+       <dynamics damping="0.1"/>
+       <limit effort="10000.0" lower="-1.49" upper="1.49" velocity="0.5"/>
+       <origin xyz="0 0 0" rpy="0 0 0" />
+        <axis xyz="0 1 0" />
+     </joint>
    </xacro:macro>
 </robot>

File: urdf/sara.urdf.xacro (robot description, xacro)
@@ -14,4 +14,5 @@
     <xacro:include filename="$(find sara_description)/urdf/mecanum_wheel/mecanum_wheel.urdf.xacro"/>
     <xacro:include filename="$(find sara_description)/urdf/arm_xtion/arm_xtion.urdf.xacro"/>
+    <xacro:include filename="$(find robotiq_140_description)/urdf/robotiq_arg2f_140_model_macro.xacro" />
     <xacro:if value="${sim}">
         <xacro:include filename="$(find sara_description)/urdf/sara.gazebo.xacro" />
@@ -60,8 +61,10 @@
         <origin xyz="0 0 -0.02989" rpy="0 1.5708 0"/>
     </xacro:robotiq_85_gripper>-->
-    <!-- Gripper C2 (old model)-->
+    <!-- Gripper C2 (old model)
     <xacro:include filename="$(find robotiq_c2_description)/urdf/robotiq_c2_model_macro.xacro"/>
     <xacro:robotiq_c2_model prefix="right_" parent="right_socket_link">
         <origin xyz="0 0 -0.02989" rpy="0 1.5708 0"/>
-    </xacro:robotiq_c2_model>
+    </xacro:robotiq_c2_model>-->
+    <xacro:robotiq_arg2f_140 prefix="right_"/>
+  -->
 </robot>

Commit message: Gripper at good position. Need to change orientation

File: urdf/arm_v2/arm.urdf.xacro (robot description, xacro)
@@ -263,5 +263,5 @@
      <joint name="${prefix}gripper_joint" type="fixed">
        <parent link="${prefix}socket_link"/>
-       <child link="${prefix}robotiq_arg2f_base_link"/>
+       <child link="robotiq_arg2f_link"/>
        <dynamics damping="0.1"/>
        <limit effort="10000.0" lower="-1.49" upper="1.49" velocity="0.5"/>

File: urdf/sara.urdf.xacro (robot description, xacro)
@@ -66,5 +66,4 @@
         <origin xyz="0 0 -0.02989" rpy="0 1.5708 0"/>
     </xacro:robotiq_c2_model>-->
-    <xacro:robotiq_arg2f_140 prefix="right_"/>
-  -->
+    <xacro:robotiq_arg2f_140 prefix=""/>
 </robot>

Commit message: good orientation of the gripper and it's TF

File: urdf/arm_v2/arm.urdf.xacro (robot description, xacro)
@@ -266,5 +266,5 @@
        <dynamics damping="0.1"/>
        <limit effort="10000.0" lower="-1.49" upper="1.49" velocity="0.5"/>
-       <origin xyz="0 0 0" rpy="0 0 0" />
+       <origin xyz="0 0 0" rpy="0 3.14 0" />
         <axis xyz="0 1 0" />
      </joint>

Commit message: changed orientation of gripper

File: urdf/arm_v2/arm.urdf.xacro (robot description, xacro)
@@ -266,5 +266,5 @@
        <dynamics damping="0.1"/>
        <limit effort="10000.0" lower="-1.49" upper="1.49" velocity="0.5"/>
-       <origin xyz="0 0 0" rpy="0 3.14 0" />
+       <origin xyz="0 0 0" rpy="0 3.14 1.57" />
         <axis xyz="0 1 0" />
      </joint>

Commit message: Good offset on the gripper

File: urdf/arm_v2/arm.urdf.xacro (robot description, xacro)
@@ -266,5 +266,5 @@
        <dynamics damping="0.1"/>
        <limit effort="10000.0" lower="-1.49" upper="1.49" velocity="0.5"/>
-       <origin xyz="0 0 0" rpy="0 3.14 1.57" />
+       <origin xyz="0 0 -0.0360875" rpy="0 3.14 1.570796" />
         <axis xyz="0 1 0" />
      </joint>

Commit message: Fixed collisions

File: urdf/arm_v2/arm.urdf.xacro (robot description, xacro)
@@ -115,5 +115,5 @@
             <mesh filename="package://sara_description/meshes/coude.STL" scale="0.001 0.001 0.001"/>
           </geometry>
-            <origin xyz="0 0 -0.0005" rpy="0 0 0"/>
+            <origin xyz="0 0 0" rpy="0 0 0"/>
             <material name="black">
               <color rgba="0.12 0.12 0.12 1"/>

File: urdf/base_xtion/base_xtion.urdf.xacro (robot description, xacro)
@@ -4,5 +4,5 @@
     <xacro:macro name="asus_base_xtion" params="prefix parent *origin sim">
         <xacro:if value="${sim}">
-            <xacro:include filename="$(find sara_description)/urdf/arm_xtion/arm_xtion.gazebo.xacro" />
+            <xacro:include filename="$(find sara_description)/urdf/base_xtion/base_xtion.gazebo.xacro" />
             <xacro:xtion_gazebo prefix="${prefix}"/>
         </xacro:if>

File: urdf/torso_v1/torso.urdf.xacro (robot description, xacro)
@@ -27,5 +27,5 @@
                <mesh filename="package://sara_description/meshes/torse.STL" scale="0.001 0.001 0.001"/>
             </geometry>
-            <origin xyz="-0.14427 -0.197233 0" rpy="1.5708 0 1.5708"/>
+            <origin xyz="0 0 0" rpy="0 0 0"/>
          </collision>
          <inertial>

Commit message: fixed bug in gripper

File: urdf/arm_v2/arm.urdf.xacro (robot description, xacro)
@@ -263,5 +263,5 @@
      <joint name="${prefix}gripper_joint" type="fixed">
        <parent link="${prefix}socket_link"/>
-       <child link="robotiq_arg2f_link"/>
+       <child link="${prefix}robotiq_arg2f_link"/>
        <dynamics damping="0.1"/>
        <limit effort="10000.0" lower="-1.49" upper="1.49" velocity="0.5"/>

File: urdf/sara.urdf.xacro (robot description, xacro)
@@ -71,4 +71,4 @@
         <origin xyz="0 0 -0.02989" rpy="0 1.5708 0"/>
     </xacro:robotiq_c2_model>-->
-    <xacro:robotiq_arg2f_140 prefix=""/>
+    <xacro:robotiq_arg2f_140 prefix="right_"/>
 </robot>

Commit message: changed orientation of arm

File: urdf/arm_v2/arm.urdf.xacro (robot description, xacro)
@@ -107,5 +107,5 @@
         <dynamics damping="0.1"/>
         <limit effort="10000.0" lower="-2.20" upper="1.90" velocity="0.5"/>
-        <origin xyz="0 0 -0.31" rpy="-1.5708 0 0" />
+        <origin xyz="0 0 -0.31" rpy="-1.5708 -1.5708 0" />
         <axis xyz="0 0 1" />
       </joint>

Commit message: met des limites de joints plus raisonables.

File: urdf/arm_v2/arm.urdf.xacro (robot description, xacro)
@@ -12,5 +12,5 @@
        <child link="${prefix}clavicular_link"/>
        <dynamics damping="0.1"/>
-       <limit effort="10000.0" lower="-1.6" upper="1.4" velocity="0.5"/>
+       <limit effort="10000.0" lower="-1" upper="1" velocity="0.5"/>
        <xacro:insert_block name="origin"/>
        <axis xyz="0 0 1" />
@@ -44,5 +44,5 @@
        <child link="${prefix}upper_arm_upper_link"/>
        <dynamics damping="0.1"/>
-       <limit effort="10000.0" lower="-4.7124" upper="1.5708" velocity="0.5"/>
+       <limit effort="10000.0" lower="-1.9" upper="0.6" velocity="0.5"/>
        <origin xyz="0 -0.085 0" rpy="-1.57 0 0" />
        <axis xyz="0 0 1" />
@@ -74,5 +74,5 @@
        <child link="${prefix}upper_arm_lower_link"/>
        <dynamics damping="0.1"/>
-       <limit effort="10000.0" lower="-3.1416" upper="3.1416" velocity="0.5"/>
+       <limit effort="10000.0" lower="-1.5" upper="1.3" velocity="0.5"/>
        <origin xyz="-0.085 0 0" rpy="1.5708 0 1.5708" />
        <axis xyz="0 0 1" />
@@ -106,5 +106,5 @@
         <child link="${prefix}forearm_upper_link"/>
         <dynamics damping="0.1"/>
-        <limit effort="10000.0" lower="-2.20" upper="1.90" velocity="0.5"/>
+        <limit effort="10000.0" lower="-0.5" upper="1.40" velocity="0.5"/>
         <origin xyz="0 0 -0.31" rpy="-1.5708 -1.5708 0" />
         <axis xyz="0 0 1" />
@@ -138,5 +138,5 @@
        <child link="${prefix}forearm_lower_link"/>
        <dynamics damping="0.1"/>
-       <limit effort="10000.0" lower="-3.1416" upper="3.1416" velocity="0.5"/>
+       <limit effort="10000.0" lower="-1.5" upper="1.5" velocity="0.5"/>
        <origin xyz="0 0.0945 0" rpy="1.5708 -1.5708 0" />
        <axis xyz="0 0 1" />
@@ -201,5 +201,5 @@
        <child link="${prefix}wrist_lower_link"/>
        <dynamics damping="0.1"/>
-       <limit effort="10000.0" lower="-1.5708" upper="1.5708" velocity="0.5"/>
+       <limit effort="10000.0" lower="-1.5" upper="1.5" velocity="0.5"/>
        <origin xyz="-0.0606 0 0" rpy="1.5708 -1.5708 0" />
        <axis xyz="0 0 1" />
@@ -233,5 +233,5 @@
        <child link="${prefix}socket_link"/>
        <dynamics damping="0.1"/>
-       <limit effort="10000.0" lower="-1.49" upper="1.49" velocity="0.5"/>
+       <limit effort="10000.0" lower="-1.5" upper="1.5" velocity="0.5"/>
        <origin xyz="0 0.084375 0" rpy="1.5708 0 0" />
        <axis xyz="1 0 0" />

File: urdf/head_v1/head.urdf.xacro (robot description, xacro)
@@ -11,5 +11,5 @@
             <parent link="${parent}_link"/>
             <child link="head_link"/>
-            <limit effort="1000.0" lower="-0.40" upper="1.04" velocity="0.5"/>
+            <limit effort="1000.0" lower="-0.8" upper="0.8" velocity="0.5"/>
             <xacro:insert_block name="origin"/>
             <axis xyz="0 0 1" />

File: urdf/neck_v1/neck.urdf.xacro (robot description, xacro)
@@ -11,5 +11,5 @@
            <parent link="${parent}_link"/>
            <child link="neck_link"/>
-           <limit effort="1000.0" lower="-1.22173" upper="1.22173" velocity="0.5"/>
+           <limit effort="1000.0" lower="-1.5" upper="1.5" velocity="0.5"/>
            <xacro:insert_block name="origin"/>
            <axis xyz="0 0 1"/>

Commit message: ajste les limites pour les rendres plus permissives.

File: urdf/arm_v2/arm.urdf.xacro (robot description, xacro)
@@ -12,5 +12,5 @@
        <child link="${prefix}clavicular_link"/>
        <dynamics damping="0.1"/>
-       <limit effort="10000.0" lower="-1" upper="1" velocity="0.5"/>
+       <limit effort="10000.0" lower="-1.57" upper="1.5" velocity="0.57"/>
        <xacro:insert_block name="origin"/>
        <axis xyz="0 0 1" />
@@ -44,5 +44,5 @@
        <child link="${prefix}upper_arm_upper_link"/>
        <dynamics damping="0.1"/>
-       <limit effort="10000.0" lower="-1.9" upper="0.6" velocity="0.5"/>
+       <limit effort="10000.0" lower="-1.9" upper="0.6" velocity="1"/>
        <origin xyz="0 -0.085 0" rpy="-1.57 0 0" />
        <axis xyz="0 0 1" />
@@ -74,5 +74,5 @@
        <child link="${prefix}upper_arm_lower_link"/>
        <dynamics damping="0.1"/>
-       <limit effort="10000.0" lower="-1.5" upper="1.3" velocity="0.5"/>
+       <limit effort="10000.0" lower="-1.5" upper="1.3" velocity="1"/>
        <origin xyz="-0.085 0 0" rpy="1.5708 0 1.5708" />
        <axis xyz="0 0 1" />
@@ -106,5 +106,5 @@
         <child link="${prefix}forearm_upper_link"/>
         <dynamics damping="0.1"/>
-        <limit effort="10000.0" lower="-0.5" upper="1.40" velocity="0.5"/>
+        <limit effort="10000.0" lower="-0.75" upper="1.40" velocity="1"/>
         <origin xyz="0 0 -0.31" rpy="-1.5708 -1.5708 0" />
         <axis xyz="0 0 1" />
@@ -138,5 +138,5 @@
        <child link="${prefix}forearm_lower_link"/>
        <dynamics damping="0.1"/>
-       <limit effort="10000.0" lower="-1.5" upper="1.5" velocity="0.5"/>
+       <limit effort="10000.0" lower="-0.5" upper="3.0" velocity="1"/>
        <origin xyz="0 0.0945 0" rpy="1.5708 -1.5708 0" />
        <axis xyz="0 0 1" />
@@ -169,5 +169,5 @@
        <parent link="${prefix}forearm_lower_link"/>
        <child link="${prefix}wrist_upper_link"/>
-       <limit effort="10000.0" lower="-3.1416" upper="3.1416" velocity="0.5"/>
+       <limit effort="10000.0" lower="-3.1416" upper="3.1416" velocity="1"/>
        <origin xyz="0 0 -0.05124" rpy="1.5708 -1.5708 0" />
        <axis xyz="0 1 0" />
@@ -201,5 +201,5 @@
        <child link="${prefix}wrist_lower_link"/>
        <dynamics damping="0.1"/>
-       <limit effort="10000.0" lower="-1.5" upper="1.5" velocity="0.5"/>
+       <limit effort="10000.0" lower="-1.5" upper="1.5" velocity="1"/>
        <origin xyz="-0.0606 0 0" rpy="1.5708 -1.5708 0" />
        <axis xyz="0 0 1" />
@@ -233,5 +233,5 @@
        <child link="${prefix}socket_link"/>
        <dynamics damping="0.1"/>
-       <limit effort="10000.0" lower="-1.5" upper="1.5" velocity="0.5"/>
+       <limit effort="10000.0" lower="-1.5" upper="1.5" velocity="1"/>
        <origin xyz="0 0.084375 0" rpy="1.5708 0 0" />
        <axis xyz="1 0 0" />
@@ -265,5 +265,5 @@
        <child link="${prefix}robotiq_arg2f_link"/>
        <dynamics damping="0.1"/>
-       <limit effort="10000.0" lower="-1.49" upper="1.49" velocity="0.5"/>
+       <limit effort="10000.0" lower="-1.49" upper="1.49" velocity="1"/>
        <origin xyz="0 0 -0.0360875" rpy="0 3.14 1.570796" />
         <axis xyz="0 1 0" />

Commit message: add an offset to the elbow yaw joint to take the offset of the gripper into account.

File: urdf/arm_v2/arm.urdf.xacro (robot description, xacro)
@@ -139,5 +139,5 @@
        <dynamics damping="0.1"/>
        <limit effort="10000.0" lower="-0.5" upper="3.0" velocity="1"/>
-       <origin xyz="0 0.0945 0" rpy="1.5708 -1.5708 0" />
+       <origin xyz="0 0.0945 0" rpy="1.5708 3.14159 0" />
        <axis xyz="0 0 1" />
      </joint>

Commit message: ajuste mieux les limites et met la bonne orientation au poignet

File: urdf/arm_v2/arm.urdf.xacro (robot description, xacro)
@@ -138,6 +138,6 @@
        <child link="${prefix}forearm_lower_link"/>
        <dynamics damping="0.1"/>
-       <limit effort="10000.0" lower="-0.5" upper="3.0" velocity="1"/>
-       <origin xyz="0 0.0945 0" rpy="1.5708 3.14159 0" />
+       <limit effort="10000.0" lower="-3" upper="3" velocity="1"/>
+       <origin xyz="0 0.0945 0" rpy="1.5708 -3.14159 0" />
        <axis xyz="0 0 1" />
      </joint>

Commit message: added new joint and link

File: urdf/arm_v2/arm.urdf.xacro (robot description, xacro)
@@ -264,4 +264,5 @@
        <parent link="${prefix}socket_link"/>
        <child link="${prefix}robotiq_arg2f_link"/>
+       <child link="${prefix}_effector"/>
        <dynamics damping="0.1"/>
        <limit effort="10000.0" lower="-1.49" upper="1.49" velocity="1"/>
@@ -269,4 +270,14 @@
         <axis xyz="0 1 0" />
      </joint>
+     <joint name="${prefix}_effector" type="fixed">
+       <parent link="${prefix}socket_link"/>
+       <child link="${prefix}_dummy"/>
+       <dynamics damping="0.1"/>
+       <limit effort="10000.0" lower="-1.49" upper="1.49" velocity="1"/>
+       <origin xyz="0 0 0" rpy="1.57 1.57 0" />
+        <axis xyz="0 1 0" />
+     </joint>
+     <link name="${prefix}_dummy">
+     </link>
    </xacro:macro>
 </robot>

Commit message: added shift for dummy link

File: urdf/arm_v2/arm.urdf.xacro (robot description, xacro)
@@ -275,5 +275,5 @@
        <dynamics damping="0.1"/>
        <limit effort="10000.0" lower="-1.49" upper="1.49" velocity="1"/>
-       <origin xyz="0 0 0" rpy="1.57 1.57 0" />
+       <origin xyz="0 0 -0.2" rpy="1.57 1.57 0" />
         <axis xyz="0 1 0" />
      </joint>
