Commit message: Mise à jour pour le nouveau poignet

File: urdf/arm_v2/arm.urdf.xacro (robot description, xacro)
@@ -143,26 +143,4 @@
      </joint>
      <link name="${prefix}forearm_lower_link">
-       <visual>
-         <geometry>
-           <mesh filename="package://sara_description/meshes/avant_bras.STL" scale="0.001 0.001 0.001"/>
-         </geometry>
-         <origin xyz="0 0 0" rpy="0 0 0" />
-           <material name="black">
-             <color rgba="0.12 0.12 0.12 1"/>
-           </material>
-       </visual>
-       <collision>
-         <geometry>
-           <mesh filename="package://sara_description/meshes/avant_bras.STL" scale="0.001 0.001 0.001"/>
-         </geometry>
-           <origin xyz="0 0 0" rpy="0 0 0"/>
-       </collision>
-       <inertial>
-         <mass value="0.1177" />
-         <origin xyz="0.0 -0.00000184 -0.03625492" rpy="0 0 0" />
-         <inertia ixx = "0.54274952" ixy = "0.0" ixz = "0.0"
-                  iyy = "1.03078569" iyz = "0.0"
-                  izz = "0.00010905" />
-       </inertial>
      </link>
      <joint name="${prefix}wrist_joint" type="fixed">
@@ -170,5 +148,5 @@
        <child link="${prefix}wrist_upper_link"/>
        <limit effort="10000.0" lower="-3.1416" upper="3.1416" velocity="1"/>
-       <origin xyz="0 0 -0.05124" rpy="1.5708 -1.5708 0" />
+       <origin xyz="0 0 0" rpy="1.5708 -1.5708 0" />
        <axis xyz="0 1 0" />
      </joint>
@@ -176,14 +154,14 @@
        <visual>
          <geometry>
-           <mesh filename="package://sara_description/meshes/poignet_haut.STL" scale="0.001 0.001 0.001"/>
-         </geometry>
-         <origin xyz="0 0 0" rpy="0 0 0"/>
-         <material name="black">
-           <color rgba="0.12 0.12 0.12 1"/>
-         </material>
-       </visual>
-       <collision>
-         <geometry>
-           <mesh filename="package://sara_description/meshes/poignet_haut.STL" scale="0.001 0.001 0.001"/>
+           <mesh filename="package://sara_description/meshes/saraRightArm_wrist1.STL" scale="0.001 0.001 0.001"/>
+         </geometry>
+         <origin xyz="0 0 0" rpy="0 0 3.141592"/>
+         <material name="black">
+           <color rgba="0.12 0.12 0.12 1"/>
+         </material>
+       </visual>
+       <collision>
+         <geometry>
+           <mesh filename="package://sara_description/meshes/saraRightArm_wrist1.STL" scale="0.001 0.001 0.001"/>
          </geometry>
          <origin xyz="0 0 0" rpy="0 0 0"/>
@@ -202,5 +180,5 @@
        <dynamics damping="0.1"/>
        <limit effort="10000.0" lower="-1.5" upper="1.5" velocity="1"/>
-       <origin xyz="-0.0606 0 0" rpy="1.5708 -1.5708 0" />
+       <origin xyz="-0.17755 0 0" rpy="0 0 1.5708" />
        <axis xyz="0 0 1" />
      </joint>
@@ -208,14 +186,14 @@
        <visual>
          <geometry>
-           <mesh filename="package://sara_description/meshes/poignet_bas.STL" scale="0.001 0.001 0.001"/>
-         </geometry>
-         <origin xyz="0 0 0" rpy=" 0 0 0"/>
-         <material name="black">
-           <color rgba="0.12 0.12 0.12 1"/>
-         </material>
-       </visual>
-       <collision>
-         <geometry>
-           <mesh filename="package://sara_description/meshes/poignet_bas.STL" scale="0.001 0.001 0.001"/>
+           <mesh filename="package://sara_description/meshes/saraRightArm_wrist2.STL" scale="0.001 0.001 0.001"/>
+         </geometry>
+         <origin xyz="0.0 -0.039925 0.0" rpy=" 0 1.5708 0"/>
+         <material name="black">
+           <color rgba="0.12 0.12 0.12 1"/>
+         </material>
+       </visual>
+       <collision>
+         <geometry>
+           <mesh filename="package://sara_description/meshes/saraRightArm_wrist2.STL" scale="0.001 0.001 0.001"/>
          </geometry>
          <origin xyz="0 0 0" rpy="0 0 0"/>
@@ -234,5 +212,5 @@
        <dynamics damping="0.1"/>
        <limit effort="10000.0" lower="-1.5" upper="1.5" velocity="1"/>
-       <origin xyz="0 0.084375 0" rpy="1.5708 0 0" />
+       <origin xyz="0 0.027475 0" rpy="1.5708 0 0" />
        <axis xyz="1 0 0" />
      </joint>
@@ -267,5 +245,5 @@
        <dynamics damping="0.1"/>
        <limit effort="10000.0" lower="-1.49" upper="1.49" velocity="1"/>
-       <origin xyz="0 0 -0.0360875" rpy="0 3.14 1.570796" />
+       <origin xyz="0 0 -0.0360875" rpy="0 3.14 0.0" />
         <axis xyz="0 1 0" />
      </joint>

Commit message: change mass to make admittance working

File: urdf/arm_v2/arm.urdf.xacro (robot description, xacro)
@@ -143,4 +143,26 @@
      </joint>
      <link name="${prefix}forearm_lower_link">
+        <visual>
+          <geometry>
+            <mesh filename="package://sara_description/meshes/coude.STL" scale="0.001 0.001 0.001"/>
+          </geometry>
+            <origin xyz="0 0 0" rpy="0 0 0"/>
+            <material name="black">
+              <color rgba="0.12 0.12 0.12 1"/>
+            </material>
+        </visual>
+        <collision>
+          <geometry>
+            <mesh filename="package://sara_description/meshes/coude.STL" scale="0.001 0.001 0.001"/>
+          </geometry>
+          <origin xyz="0 0 0" rpy="0 0 0"/>
+        </collision>
+        <inertial>
+          <mass value="0.48300045" />
+          <origin xyz="0.00000207 0.03922132 -0.01628605" rpy="0 0 0"/>
+          <inertia ixx = "0.00036109" ixy = "0.0" ixz = "-0.00000002"
+                   iyy = "0.00029872" iyz = "0.00001701"
+                   izz = "0.00055069" />
+        </inertial>
      </link>
      <joint name="${prefix}wrist_joint" type="fixed">
@@ -168,5 +190,5 @@
        </collision>
        <inertial>
-         <mass value="0.1956991" />
+         <mass value="0.3956991" />
          <origin xyz="-0.03893593 0.00017228 -0.00000284" rpy="0 0 0"/>
          <inertia ixx = "0.00007035" ixy = "-0.00000150" ixz = "0.0"
@@ -200,5 +222,5 @@
        </collision>
        <inertial>
-         <mass value="0.18747684" />
+         <mass value="0.28747684" />
          <origin xyz="0.00001243 0.05721169 0.0" rpy=" 0 0 0"/>
          <inertia ixx = "0.00015391" ixy = "-0.00000060" ixz = "0.0"
@@ -232,5 +254,5 @@
        </collision>
        <inertial>
-         <mass value="0.02796" />
+         <mass value="1.82796" />
          <origin xyz="0.0 0.0 -0.01570460" rpy="0 0 0"/>
          <inertia ixx = "0.00000889" ixy = "0.0" ixz = "0.0"

Commit message: Updated wrist geometry to match current setup (with DYNAMIXEL XM540W270R) and removal of unused geometry files.

File: urdf/arm_v2/arm.urdf.xacro (robot description, xacro)
@@ -145,5 +145,5 @@
         <visual>
           <geometry>
-            <mesh filename="package://sara_description/meshes/coude.STL" scale="0.001 0.001 0.001"/>
+            <mesh filename="package://sara_description/meshes/coude.STL" scale="0.00001 0.00001 0.00001"/>
           </geometry>
             <origin xyz="0 0 0" rpy="0 0 0"/>
@@ -176,16 +176,16 @@
        <visual>
          <geometry>
-           <mesh filename="package://sara_description/meshes/saraRightArm_wrist1.STL" scale="0.001 0.001 0.001"/>
-         </geometry>
-         <origin xyz="0 0 0" rpy="0 0 3.141592"/>
-         <material name="black">
-           <color rgba="0.12 0.12 0.12 1"/>
-         </material>
-       </visual>
-       <collision>
-         <geometry>
-           <mesh filename="package://sara_description/meshes/saraRightArm_wrist1.STL" scale="0.001 0.001 0.001"/>
-         </geometry>
-         <origin xyz="0 0 0" rpy="0 0 0"/>
+           <mesh filename="package://sara_description/meshes/WRA-01.STL" scale="0.001 0.001 0.001"/>
+         </geometry>
+         <origin xyz="0 0 0" rpy="-1.5708 0 3.141592"/>
+         <material name="black">
+           <color rgba="0.12 0.12 0.12 1"/>
+         </material>
+       </visual>
+       <collision>
+         <geometry>
+           <mesh filename="package://sara_description/meshes/WRA-01.STL" scale="0.001 0.001 0.001"/>
+         </geometry>
+         <origin xyz="0 0 0" rpy="-1.5708 0 3.141592"/>
        </collision>
        <inertial>
@@ -201,6 +201,6 @@
        <child link="${prefix}wrist_lower_link"/>
        <dynamics damping="0.1"/>
-       <limit effort="10000.0" lower="-1.5" upper="1.5" velocity="1"/>
-       <origin xyz="-0.17755 0 0" rpy="0 0 1.5708" />
+       <limit effort="10000.0" lower="-1.57" upper="1.57" velocity="1"/>
+       <origin xyz="-0.10795 0 0" rpy="0 1.5708 1.5708" />
        <axis xyz="0 0 1" />
      </joint>
@@ -208,16 +208,16 @@
        <visual>
          <geometry>
-           <mesh filename="package://sara_description/meshes/saraRightArm_wrist2.STL" scale="0.001 0.001 0.001"/>
-         </geometry>
-         <origin xyz="0.0 -0.039925 0.0" rpy=" 0 1.5708 0"/>
-         <material name="black">
-           <color rgba="0.12 0.12 0.12 1"/>
-         </material>
-       </visual>
-       <collision>
-         <geometry>
-           <mesh filename="package://sara_description/meshes/saraRightArm_wrist2.STL" scale="0.001 0.001 0.001"/>
-         </geometry>
-         <origin xyz="0 0 0" rpy="0 0 0"/>
+           <mesh filename="package://sara_description/meshes/WRA-02.STL" scale="0.001 0.001 0.001"/>
+         </geometry>
+         <origin xyz="0.0 0 0.0" rpy=" 0 1.5708 0"/>
+         <material name="black">
+           <color rgba="0.12 0.12 0.12 1"/>
+         </material>
+       </visual>
+       <collision>
+         <geometry>
+           <mesh filename="package://sara_description/meshes/WRA-02.STL" scale="0.001 0.001 0.001"/>
+         </geometry>
+         <origin xyz="0 0 0" rpy=" 0 1.5708 0"/>
        </collision>
        <inertial>
@@ -234,5 +234,5 @@
        <dynamics damping="0.1"/>
        <limit effort="10000.0" lower="-1.5" upper="1.5" velocity="1"/>
-       <origin xyz="0 0.027475 0" rpy="1.5708 0 0" />
+       <origin xyz="0 0.0635 0" rpy="1.5708 0 0" />
        <axis xyz="1 0 0" />
      </joint>
@@ -240,16 +240,16 @@
        <visual>
          <geometry>
-           <mesh filename="package://sara_description/meshes/attache_pince.STL" scale="0.001 0.001 0.001"/>
-         </geometry>
-         <origin xyz="0 0 0" rpy="0 0 0"/>
-         <material name="black">
-           <color rgba="0.12 0.12 0.12 1"/>
-         </material>
-       </visual>
-       <collision>
-         <geometry>
-           <mesh filename="package://sara_description/meshes/attache_pince.STL" scale="0.001 0.001 0.001"/>
-         </geometry>
-         <origin xyz="0 0 0" rpy="0 0 0"/>
+           <mesh filename="package://sara_description/meshes/WRA-03.STL" scale="0.001 0.001 0.001"/>
+         </geometry>
+         <origin xyz="0 0 0" rpy="0 1.5708 -1.5708"/>
+         <material name="black">
+           <color rgba="0.12 0.12 0.12 1"/>
+         </material>
+       </visual>
+       <collision>
+         <geometry>
+           <mesh filename="package://sara_description/meshes/WRA-03.STL" scale="0.001 0.001 0.001"/>
+         </geometry>
+         <origin xyz="0 0 0" rpy="0 1.5708 -1.5708"/>
        </collision>
        <inertial>
@@ -267,5 +267,5 @@
        <dynamics damping="0.1"/>
        <limit effort="10000.0" lower="-1.49" upper="1.49" velocity="1"/>
-       <origin xyz="0 0 -0.0360875" rpy="0 3.14 0.0" />
+       <origin xyz="0 0 -0.057" rpy="0 3.14 1.5708" />
         <axis xyz="0 1 0" />
      </joint>

Commit message: ajuste les limites de joints

File: urdf/arm_v2/arm.urdf.xacro (robot description, xacro)
@@ -201,5 +201,5 @@
        <child link="${prefix}wrist_lower_link"/>
        <dynamics damping="0.1"/>
-       <limit effort="10000.0" lower="-1.57" upper="1.57" velocity="1"/>
+       <limit effort="10000.0" lower="-1.5" upper="1.5" velocity="1"/>
        <origin xyz="-0.10795 0 0" rpy="0 1.5708 1.5708" />
        <axis xyz="0 0 1" />
@@ -233,5 +233,5 @@
        <child link="${prefix}socket_link"/>
        <dynamics damping="0.1"/>
-       <limit effort="10000.0" lower="-1.5" upper="1.5" velocity="1"/>
+       <limit effort="10000.0" lower="-1.45" upper="1.45" velocity="1"/>
        <origin xyz="0 0.0635 0" rpy="1.5708 0 0" />
        <axis xyz="1 0 0" />

Commit message: ajuste les limites pour la tête et le poignet

File: urdf/arm_v2/arm.urdf.xacro (robot description, xacro)
@@ -12,5 +12,5 @@
        <child link="${prefix}clavicular_link"/>
        <dynamics damping="0.1"/>
-       <limit effort="10000.0" lower="-1.57" upper="1.5" velocity="0.57"/>
+       <limit effort="10000.0" lower="-0.3" upper="1.5" velocity="0.57"/>
        <xacro:insert_block name="origin"/>
        <axis xyz="0 0 1" />
@@ -275,5 +275,5 @@
        <dynamics damping="0.1"/>
        <limit effort="10000.0" lower="-1.49" upper="1.49" velocity="1"/>
-       <origin xyz="0 0 -0.2" rpy="1.57 1.57 0" />
+       <origin xyz="0 0 -0.24" rpy="1.57 1.57 3.141592" />
         <axis xyz="0 1 0" />
      </joint>

File: urdf/head_v1/head.urdf.xacro (robot description, xacro)
@@ -11,5 +11,5 @@
             <parent link="${parent}_link"/>
             <child link="head_link"/>
-            <limit effort="1000.0" lower="-0.9" upper="0.9" velocity="0.5"/>
+            <limit effort="1000.0" lower="-1.3" upper="1.3" velocity="0.5"/>
             <xacro:insert_block name="origin"/>
             <axis xyz="0 0 1" />
