Commit message: Fix xtion visual + fix rong joint name

File: urdf/arm_v2/arm.gazebo.xacro (robot description, xacro)
@@ -22,9 +22,9 @@
       <selfCollide>true</selfCollide>
     </gazebo>
-    <gazebo reference="${prefix}upper_wrist_link">
+    <gazebo reference="${prefix}wrist_upper_link">
       <turnGravityOff>false</turnGravityOff>
       <selfCollide>true</selfCollide>
     </gazebo>
-    <gazebo reference="${prefix}lower_wrist_link">
+    <gazebo reference="${prefix}wrist_lower_link">
       <turnGravityOff>false</turnGravityOff>
       <selfCollide>true</selfCollide>

File: urdf/arm_v2/arm.transmission.xacro (robot description, xacro)
@@ -56,10 +56,10 @@
       </joint>
     </transmission>
-    <transmission name="${prefix}wrist_yaw_trans" type="SimpleTransmission">
+    <transmission name="${prefix}wrist_roll_trans" type="SimpleTransmission">
       <type>transmission_interface/SimpleTransmission</type>
-      <actuator name="${prefix}wrist_yaw_motor">
+      <actuator name="${prefix}wrist_roll_motor">
       	 <mechanicalReduction>1</mechanicalReduction>
       </actuator>
-      <joint name="${prefix}wrist_yaw_joint">
+      <joint name="${prefix}wrist_roll_joint">
       	 <hardwareInterface>VelocityJointInterface</hardwareInterface>
       </joint>

File: urdf/arm_v2/arm.urdf.xacro (robot description, xacro)
@@ -155,10 +155,10 @@
      <joint name="${prefix}wrist_joint" type="fixed">
        <parent link="${prefix}forearm_lower_link"/>
-       <child link="${prefix}upper_wrist_link"/>
+       <child link="${prefix}wrist_upper_link"/>
        <limit effort="1000.0" lower="-3.1416" upper="3.1416" velocity="0.5"/>
        <origin xyz="0 0 -0.11184" rpy="1.5708 -1.5708 0" />
        <axis xyz="0 1 0" />
      </joint>
-     <link name="${prefix}upper_wrist_link">
+     <link name="${prefix}wrist_upper_link">
        <visual>
          <geometry>
@@ -183,11 +183,11 @@
      </link>
      <joint name="${prefix}wrist_pitch_joint" type="revolute">
-       <parent link="${prefix}upper_wrist_link"/>
-       <child link="${prefix}lower_wrist_link"/>
+       <parent link="${prefix}wrist_upper_link"/>
+       <child link="${prefix}wrist_lower_link"/>
        <limit effort="1000.0" lower="-1.5708" upper="1.5708" velocity="0.5"/>
        <origin xyz="0 0 0" rpy="1.5708 -1.5708 0" />
        <axis xyz="0 0 1" />
      </joint>
-     <link name="${prefix}lower_wrist_link">
+     <link name="${prefix}wrist_lower_link">
        <visual>
          <geometry>
@@ -211,6 +211,6 @@
        </inertial>
      </link>
-     <joint name="${prefix}wrist_yaw_joint" type="revolute">
-       <parent link="${prefix}lower_wrist_link"/>
+     <joint name="${prefix}wrist_roll_joint" type="revolute">
+       <parent link="${prefix}wrist_lower_link"/>
        <child link="${prefix}socket_link"/>
        <limit effort="1000.0" lower="-1.49" upper="1.49" velocity="0.5"/>

File: urdf/sara.urdf (robot description, URDF)
Before this commit: robot sara, 30 links, 29 joints
Links:
- removed link arm_clavicular_link
- removed link arm_fix_lower_link
- removed link arm_fix_upper_link
- removed link arm_high_wrist_link
- removed link arm_low_wrist_link
- removed link arm_rot_lower_link
- removed link arm_rot_upper_link
- removed link arm_socket_link
- removed link camera_link
- removed link front_left_wheel
- removed link front_right_wheel
- removed link grasp_link
- removed link head_dynamixel_link
- removed link kinect_link
- removed link lidar_link
- removed link rear_left_wheel
- removed link rear_right_wheel
- removed link robotiq_85_base_link
- removed link robotiq_85_left_finger_link
- removed link robotiq_85_left_finger_tip_link
- removed link robotiq_85_left_inner_knuckle_link
- removed link robotiq_85_left_knuckle_link
- removed link robotiq_85_right_finger_link
- removed link robotiq_85_right_finger_tip_link
- removed link robotiq_85_right_inner_knuckle_link
- removed link robotiq_85_right_knuckle_link
- added link front_hokuyo_link, mass 0.5; collision cylinder length=0.085 radius=0.03; visual cylinder length=0.085 radius=0.03
- added link front_left_mecanum_wheel_link
- added link front_right_mecanum_wheel_link
- added link head_xtion_depth_frame
- added link head_xtion_depth_optical_frame
- added link head_xtion_link, mass 0.200; collision box size=0.035 0.185 0.025; visual mesh filename=package://sara_description/meshes/xtion.STL scale=0.001 0.001 0.001
- added link head_xtion_rgb_frame
- added link head_xtion_rgb_optical_frame
- added link kinect2_link, mass 10; collision mesh filename=package://sara_description/meshes/kinect.STL scale=0.001 0.001 0.001; visual mesh filename=package://sara_description/meshes/kinect.STL scale=0.001 0.001 0.001
- added link rear_left_mecanum_wheel_link
- added link rear_right_mecanum_wheel_link
- added link right_clavicular_link, mass 1; collision mesh filename=package://sara_description/meshes/epaule.STL scale=0.001 0.001 0.001; visual mesh filename=package://sara_description/meshes/epaule.STL scale=0.001 0.001 0.001
- added link right_forearm_lower_link, mass 1; collision mesh filename=package://sara_description/meshes/avant-bras.STL scale=0.001 0.001 0.001; visual mesh filename=package://sara_description/meshes/avant-bras.STL scale=0.001 0.001 0.001
- added link right_forearm_upper_link, mass 1; collision mesh filename=package://sara_description/meshes/coude.STL scale=0.001 0.001 0.001; visual mesh filename=package://sara_description/meshes/coude.STL scale=0.001 0.001 0.001
- added link right_lower_wrist_link, mass 1; collision mesh filename=package://sara_description/meshes/poignet_bas.STL scale=0.001 0.001 0.001; visual mesh filename=package://sara_description/meshes/poignet_bas.STL scale=0.001 0.001 0.001
- added link right_robotiq_85_base_link, mass 0.636951; collision mesh filename=package://robotiq_c2_model_visualization/meshes/robotiq_c2/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; visual mesh filename=package://robotiq_c2_model_visualization/meshes/robotiq_c2/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
- added link right_robotiq_85_left_finger_link, mass 0.027309; collision mesh filename=package://robotiq_c2_model_visualization/meshes/robotiq_c2/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; visual mesh filename=package://robotiq_c2_model_visualization/meshes/robotiq_c2/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
- added link right_robotiq_85_left_finger_tip_link, mass 0.019555; collision mesh filename=package://robotiq_c2_model_visualization/meshes/robotiq_c2/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; visual mesh filename=package://robotiq_c2_model_visualization/meshes/robotiq_c2/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
- added link right_robotiq_85_left_inner_knuckle_link, mass 0.029951; collision mesh filename=package://robotiq_c2_model_visualization/meshes/robotiq_c2/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; visual mesh filename=package://robotiq_c2_model_visualization/meshes/robotiq_c2/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
- added link right_robotiq_85_left_knuckle_link, mass 0.018491; collision mesh filename=package://robotiq_c2_model_visualization/meshes/robotiq_c2/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; visual mesh filename=package://robotiq_c2_model_visualization/meshes/robotiq_c2/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
- added link right_robotiq_85_right_finger_link, mass 0.027309; collision mesh filename=package://robotiq_c2_model_visualization/meshes/robotiq_c2/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; visual mesh filename=package://robotiq_c2_model_visualization/meshes/robotiq_c2/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
- added link right_robotiq_85_right_finger_tip_link, mass 0.019555; collision mesh filename=package://robotiq_c2_model_visualization/meshes/robotiq_c2/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; visual mesh filename=package://robotiq_c2_model_visualization/meshes/robotiq_c2/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
- added link right_robotiq_85_right_inner_knuckle_link, mass 0.029951; collision mesh filename=package://robotiq_c2_model_visualization/meshes/robotiq_c2/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; visual mesh filename=package://robotiq_c2_model_visualization/meshes/robotiq_c2/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
- added link right_robotiq_85_right_knuckle_link, mass 0.018491; collision mesh filename=package://robotiq_c2_model_visualization/meshes/robotiq_c2/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; visual mesh filename=package://robotiq_c2_model_visualization/meshes/robotiq_c2/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
- added link right_socket_link, mass 1; collision mesh filename=package://sara_description/meshes/attache-pince.STL scale=0.001 0.001 0.001; visual mesh filename=package://sara_description/meshes/attache-pince.STL scale=0.001 0.001 0.001
- added link right_upper_arm_lower_link, mass 1; collision mesh filename=package://sara_description/meshes/bras_haut.STL scale=0.001 0.001 0.001; visual mesh filename=package://sara_description/meshes/bras_haut.STL scale=0.001 0.001 0.001
- added link right_upper_arm_upper_link, mass 1; collision mesh filename=package://sara_description/meshes/epaule.STL scale=0.001 0.001 0.001; visual mesh filename=package://sara_description/meshes/epaule.STL scale=0.001 0.001 0.001
- added link right_upper_wrist_link, mass 1; collision mesh filename=package://sara_description/meshes/poignet_haut.STL scale=0.001 0.001 0.001; visual mesh filename=package://sara_description/meshes/poignet_haut.STL scale=0.001 0.001 0.001
Joints:
- removed joint arm_elbow_joint
- removed joint arm_end_effector_joint
- removed joint arm_forarm_wrist_joint
- removed joint arm_high_low_wrist_joint
- removed joint arm_low_wrist_grasp_socket_joint
- removed joint arm_rot_elbow_joint
- removed joint arm_rot_wrist_joint
- removed joint arm_shoulder_joint
- removed joint base_kinect_joint
- removed joint base_to_front_left_wheel
- removed joint base_to_front_right_wheel
- removed joint base_to_rear_left_wheel
- removed joint base_to_rear_right_wheel
- removed joint camera_joint
- removed joint grasp_joint
- removed joint head_dynamixel_joint
- removed joint laser_joint
- removed joint neck_head_joint
- removed joint robotiq_85_left_finger_joint
- removed joint robotiq_85_left_finger_tip_joint
- removed joint robotiq_85_left_inner_knuckle_joint
- removed joint robotiq_85_left_knuckle_joint
- removed joint robotiq_85_right_finger_joint
- removed joint robotiq_85_right_finger_tip_joint
- removed joint robotiq_85_right_inner_knuckle_joint
- removed joint robotiq_85_right_knuckle_joint
- removed joint torso_arm_joint
- removed joint torso_neck_joint
- added joint base_kinect2_joint: type fixed, parent base_link, child kinect2_link, origin xyz=0.177374 0 0.65676 rpy=-1.5708 0 -1.5708, axis 0 0 1, limit lower=0 upper=0.5 effort=1000.0 velocity=0.2
- added joint front_hokuyo_joint: type fixed, parent base_link, child front_hokuyo_link, origin xyz=0.2516879 0 0 rpy=0 0 0
- added joint front_left_mecanum_wheel_joint: type continuous, parent base_link, child front_left_mecanum_wheel_link, origin xyz=0.205631 0.22735 -0.06 rpy= -1.57079632679 0 0, axis 0 0 1
- added joint front_right_mecanum_wheel_joint: type continuous, parent base_link, child front_right_mecanum_wheel_link, origin xyz=0.205631 -0.22735 -0.06 rpy= 1.57079632679 0 0, axis 0 0 1
- added joint head_pitch_joint: type revolute, parent neck_link, child head_link, origin xyz=0 0 0.0927 rpy=-1.57 0 0, axis 0 0 1, limit lower=-0.40 upper=1.04 effort=1000.0 velocity=0.5
- added joint head_xtion_depth_joint: type fixed, parent head_xtion_link, child head_xtion_depth_frame, origin xyz=0.0 0.049 0.0 rpy=0 0 0
- added joint head_xtion_depth_optical_joint: type fixed, parent head_xtion_depth_frame, child head_xtion_depth_optical_frame, origin xyz=0 0 0 rpy=-1.57079632679 0.0 -1.57079632679
- added joint head_xtion_joint: type fixed, parent head_link, child head_xtion_link, origin xyz=0.0776104 -0.13 0 rpy=1.57 0 0
- added joint head_xtion_rgb_joint: type fixed, parent head_xtion_link, child head_xtion_rgb_frame, origin xyz=0.0 0.022 0.0 rpy=0 0 0
- added joint head_xtion_rgb_optical_joint: type fixed, parent head_xtion_rgb_frame, child head_xtion_rgb_optical_frame, origin xyz=0 0 0 rpy=-1.57079632679 0.0 -1.57079632679
- added joint head_yaw_joint: type revolute, parent torso_link, child neck_link, origin xyz=0.032295 0 0.2777 rpy=0 0 0, axis 0 0 1, limit lower=-1.22173 upper=1.22173 effort=1000.0 velocity=0.5
- added joint rear_left_mecanum_wheel_joint: type continuous, parent base_link, child rear_left_mecanum_wheel_link, origin xyz=-0.205631 0.22735 -0.06 rpy= -1.57079632679 0 0, axis 0 0 1
- added joint rear_right_mecanum_wheel_joint: type continuous, parent base_link, child rear_right_mecanum_wheel_link, origin xyz=-0.205631 -0.22735 -0.06 rpy= 1.57079632679 0 0, axis 0 0 1
- added joint right_elbow_pitch_joint: type revolute, parent right_upper_arm_lower_link, child right_forearm_upper_link, origin xyz=0 0 -0.31 rpy=-1.5708 0 0, axis 0 0 1, limit lower=-2.20 upper=1.90 effort=1000.0 velocity=0.5
- added joint right_elbow_yaw_joint: type revolute, parent right_forearm_upper_link, child right_forearm_lower_link, origin xyz=0 0.0945 0 rpy=1.5708 -1.5708 0, axis 0 0 1, limit lower=-3.1416 upper=3.1416 effort=1000.0 velocity=0.5
- added joint right_robotiq_85_base_joint: type fixed, parent right_socket_link, child right_robotiq_85_base_link, origin xyz=0 0 -0.02989 rpy=0 1.5708 0, axis 1 0 0
- added joint right_robotiq_85_left_finger_joint: type fixed, parent right_robotiq_85_left_knuckle_link, child right_robotiq_85_left_finger_link, origin xyz=0 .00508 .03134 rpy=3.1415 0 0, axis 1 0 0, limit lower=0 upper=1.5707 effort=1000 velocity=2.0
- added joint right_robotiq_85_left_finger_tip_joint: type revolute, parent right_robotiq_85_left_inner_knuckle_link, child right_robotiq_85_left_finger_tip_link, origin xyz=0 .04196 -.0388 rpy=0 0 0, axis 1 0 0, limit lower=0 upper=1.5707 effort=1000 velocity=2.0, mimic joint=right_robotiq_85_left_knuckle_joint multiplier=-1
- added joint right_robotiq_85_left_inner_knuckle_joint: type revolute, parent right_robotiq_85_base_link, child right_robotiq_85_left_inner_knuckle_link, origin xyz=.04843 .0127 0 rpy=1.5707 1.5707 0, axis 1 0 0, limit lower=0 upper=1.5707 effort=1000 velocity=2.0, mimic joint=right_robotiq_85_left_knuckle_joint offset=0
- added joint right_robotiq_85_left_knuckle_joint: type revolute, parent right_robotiq_85_base_link, child right_robotiq_85_left_knuckle_link, origin xyz=.04191 .0306 0 rpy=-1.5707 1.5707 0, axis 1 0 0, limit lower=0 upper=.8575 effort=1000 velocity=2.0
- added joint right_robotiq_85_right_finger_joint: type fixed, parent right_robotiq_85_right_knuckle_link, child right_robotiq_85_right_finger_link, origin xyz=0 .00508 .03134 rpy=3.1415 0 0, axis 1 0 0, limit lower=0 upper=1.5707 effort=1000 velocity=2.0
- added joint right_robotiq_85_right_finger_tip_joint: type revolute, parent right_robotiq_85_right_inner_knuckle_link, child right_robotiq_85_right_finger_tip_link, origin xyz=0 .04196 -.0388 rpy=0 0 0, axis 1 0 0, limit lower=0 upper=1.5707 effort=1000 velocity=2.0, mimic joint=right_robotiq_85_left_knuckle_joint multiplier=-1
- added joint right_robotiq_85_right_inner_knuckle_joint: type revolute, parent right_robotiq_85_base_link, child right_robotiq_85_right_inner_knuckle_link, origin xyz=.04843 -.0127 0 rpy=-1.5707 -1.5707 0, axis 1 0 0, limit lower=0 upper=1.5707 effort=1000 velocity=2.0, mimic joint=right_robotiq_85_left_knuckle_joint offset=0
- added joint right_robotiq_85_right_knuckle_joint: type revolute, parent right_robotiq_85_base_link, child right_robotiq_85_right_knuckle_link, origin xyz=.04191 -.0306 0 rpy=1.5707 -1.5707 0, axis 1 0 0, limit lower=0 upper=1.5707 effort=1000 velocity=2.0, mimic joint=right_robotiq_85_left_knuckle_joint multiplier=1
- added joint right_shoulder_pitch_joint: type revolute, parent right_clavicular_link, child right_upper_arm_upper_link, origin xyz=0 -0.085 0 rpy=-1.57 0 0, axis 0 0 1, limit lower=-4.7124 upper=1.5708 effort=1000.0 velocity=0.5
- added joint right_shoulder_roll_joint: type revolute, parent torso_link, child right_clavicular_link, origin xyz=0 -0.145 0.189 rpy=0 -1.57 0, axis 0 0 1, limit lower=-1.6 upper=1.4 effort=1000.0 velocity=0.5
- added joint right_shoulder_yaw_joint: type revolute, parent right_upper_arm_upper_link, child right_upper_arm_lower_link, origin xyz=-0.085 0 0 rpy=1.5708 0 1.5708, axis 0 0 1, limit lower=-3.1416 upper=3.1416 effort=1000.0 velocity=0.5
- added joint right_wrist_joint: type fixed, parent right_forearm_lower_link, child right_upper_wrist_link, origin xyz=0 0 -0.11184 rpy=1.5708 -1.5708 0, axis 0 1 0, limit lower=-3.1416 upper=3.1416 effort=1000.0 velocity=0.5
- added joint right_wrist_pitch_joint: type revolute, parent right_upper_wrist_link, child right_lower_wrist_link, origin xyz=0 0 0 rpy=1.5708 -1.5708 0, axis 0 0 1, limit lower=-1.5708 upper=1.5708 effort=1000.0 velocity=0.5
- added joint right_wrist_yaw_joint: type revolute, parent right_lower_wrist_link, child right_socket_link, origin xyz=0 0.084375 0 rpy=1.5708 0 0, axis 1 0 0, limit lower=-1.49 upper=1.49 effort=1000.0 velocity=0.5

File: urdf/sara.urdf.xacro (robot description, xacro)
@@ -1,6 +1,6 @@
 <?xml version="1.0"?>
 <robot xmlns:xacro="http://ros.org/wiki/xacro" name="sara" >
+    <xacro:arg name="sim" default="true"/>
     <xacro:property name="sim" value="$(arg sim)"/>
-    <xacro:property name="end_effector" value="$(arg end_effector)"/>
     <!-- Inclure tous les autres urdf.xacros ici -->
     <xacro:include filename="$(find sara_description)/urdf/torso_v1/torso.urdf.xacro"/>
@@ -35,5 +35,5 @@
     <!-- Neck -->
     <xacro:sara_neck_v1 parent="torso" sim="${sim}">
-        <origin xyz="0.032295 0 0.2447" rpy="0 0 0"/>
+        <origin xyz="0.032295 0 0.2777" rpy="0 0 0"/>
     </xacro:sara_neck_v1>
     <!-- Head -->
@@ -50,17 +50,13 @@
     </xacro:sara_arm_v2>
     <!-- End Effector -->
-    <xacro:if value="${end_effector == 85}">
-        <!-- Gripper 85 (round base) -->
-        <xacro:include filename="$(find robotiq_85_description)/urdf/robotiq_85_gripper.urdf.xacro"/>
-        <xacro:robotiq_85_gripper prefix="right_" parent="right_socket_link">
-            <origin xyz="0 0 -0.02989" rpy="0 1.5708 0"/>
-        </xacro:robotiq_85_gripper>
-    </xacro:if>
-    <xacro:if value="${end_effector == 'C2'}">
-        <!-- Gripper C2 (old model)-->
-        <xacro:include filename="$(find robotiq_c2_model_visualization)/urdf/robotiq_c2_model_macro.xacro"/>
-        <xacro:robotiq_c2_model prefix="right_" parent="right_socket_link">
-            <origin xyz="0 0 -0.02989" rpy="0 1.5708 0"/>
-        </xacro:robotiq_c2_model>
-    </xacro:if>
+    <!-- Gripper 85 (round base)
+    <xacro:include filename="$(find robotiq_85_description)/urdf/robotiq_85_gripper.urdf.xacro"/>
+    <xacro:robotiq_85_gripper prefix="right_" parent="right_socket_link">
+        <origin xyz="0 0 -0.02989" rpy="0 1.5708 0"/>
+    </xacro:robotiq_85_gripper>-->
+    <!-- Gripper C2 (old model)-->
+    <xacro:include filename="$(find robotiq_c2_model_visualization)/urdf/robotiq_c2_model_macro.xacro"/>
+    <xacro:robotiq_c2_model prefix="right_" parent="right_socket_link">
+        <origin xyz="0 0 -0.02989" rpy="0 1.5708 0"/>
+    </xacro:robotiq_c2_model>
 </robot>

File: urdf/xtion/xtion.urdf.xacro (robot description, xacro)
@@ -15,9 +15,9 @@
         <inertial>
           <mass value="0.200" />
-          <origin xyz="0 0 0" rpy="0 0 0" />
+          <origin xyz="0 0 0" rpy="1.5708 0 1.5708" />
           <inertia ixx="5.8083e-4" ixy="0" ixz="0" iyy="3.0833e-5" iyz="0" izz="5.9083e-4" />
         </inertial>
         <visual>
-          <origin xyz="0 0 0" rpy="0 0 0" />
+          <origin xyz="0 0 0" rpy="1.5708 0 1.5708" />
           <geometry>
               <mesh filename="package://sara_description/meshes/xtion.STL" scale="0.001 0.001 0.001"/>
@@ -25,5 +25,5 @@
         </visual>
         <collision>
-          <origin xyz="0 0 0" rpy="0 0 0" />
+          <origin xyz="0 0 0" rpy="1.5708 0 1.5708" />
           <geometry>
             <box size="0.035 0.185 0.025"/>
