Commit message: wip

File: urdf/sara.urdf.xacro (robot description, xacro)
@@ -1,4 +1,4 @@
 <?xml version="1.0"?>
-<robot xmlns:xacro="http://ros.org/wiki/xacro" name="sara" >
+<robot name="sara" xmlns:xacro="http://www.ros.org/wiki/xacro">
     <xacro:arg name="sim" default="true"/>
     <xacro:property name="sim" value="$(arg sim)"/>
@@ -12,53 +12,24 @@
     <xacro:include filename="$(find sara_description)/urdf/base_v2/base.urdf.xacro"/>
     <xacro:include filename="$(find sara_description)/urdf/hokuyo/hokuyo.urdf.xacro"/>
-    <xacro:include filename="$(find sara_description)/urdf/mecanum_wheel/mecanum_wheel.urdf.xacro"/>
-    <xacro:include filename="$(find robotiq_140_description)/urdf/robotiq_arg2f_140_model_macro.xacro" />
-    <xacro:if value="${sim}">
+    <xacro:macro name="robot">
+        <!-- BASE FOOTPRINT -->
+        <link name="sara_base_footprint">
+            <visual>
+                <origin xyz="0 0 0" rpy="0 0 0" />
+                <geometry>
+                    <box size="0.001 0.001 0.001" />
+                </geometry>
+            </visual>
+        </link>
+        <joint name="sara_base_footprint_joint" type="fixed">
+            <origin xyz="0 0 0" rpy="0 0 0" /> <!-- ${wheel_radius} property must be defined inside wheel description -->
+            <parent link="sara_base_footprint"/>
+            <child link="base_link" />
+        </joint>
+        <!-- Base -->
+        <xacro:sara_base sim="${sim}"/>
+        <!-- Bring in simulation data for Gazebo. -->
         <xacro:include filename="$(find sara_description)/urdf/sara.gazebo.xacro" />
-        <xacro:sara_gazebo/>
-    </xacro:if>
-    <!-- Base -->
-    <xacro:sara_base_v2 sim="${sim}"/>
-    <!-- hokuyo -->
-    <xacro:hokuyo prefix="front_" parent="base" sim="${sim}">
-        <origin xyz="0.2516879 0 0" rpy="0 0 0" />
-    </xacro:hokuyo>
-    <!-- Wheels -->
-    <xacro:four_mecanum_wheels parent="base" x_center="0.22735" y_center="0.23" sim="${sim}"/>
-    <!-- Linear Actuator -->
-    <xacro:sara_linear_actuator_v1 parent="base" sim="${sim}">
-        <origin xyz="0 0 0.1" rpy="0 0 0" />
-    </xacro:sara_linear_actuator_v1>
-    <!-- Torso -->
-    <xacro:sara_torso_v1 parent="actuator" sim="${sim}">
-        <origin xyz="0.1999806 0 0.61595" rpy="0 0 0" />
-    </xacro:sara_torso_v1>
-    <!-- Neck -->
-    <xacro:sara_neck_v1 parent="torso" sim="${sim}">
-        <origin xyz="0.032295 0 0.10036" rpy="0 0 0"/>
-    </xacro:sara_neck_v1>
-    <!-- Head -->
-    <xacro:sara_head_v1 parent="neck" sim="${sim}">
-        <origin xyz="0 0 0.1214" rpy="-1.57 0 0"/>
-    </xacro:sara_head_v1>
-    <!-- Head Xtion -->
-    <xacro:asus_head_xtion prefix="head_" parent="head" sim="${sim}">
-        <origin xyz="0.0776104 -0.13 0" rpy="1.57 0 0" />
-    </xacro:asus_head_xtion>
-    <!-- Arm -->
-    <xacro:sara_arm_v2 prefix="right_" parent="torso" sim="${sim}">
-        <origin xyz="0 -0.1437625 0.01166" rpy="0 -1.57 0"/>
-    </xacro:sara_arm_v2>
-    <!-- End Effector -->
-    <!-- Gripper 85 (round base)
-    <xacro:include filename="$(find robotiq_85_description)/urdf/robotiq_85_gripper.urdf.xacro"/>
-    <xacro:robotiq_85_gripper prefix="right_" parent="right_socket_link">
-        <origin xyz="0 0 -0.02989" rpy="0 1.5708 0"/>
-    </xacro:robotiq_85_gripper>-->
-    <!-- Gripper C2 (old model)
-    <xacro:include filename="$(find robotiq_c2_description)/urdf/robotiq_c2_model_macro.xacro"/>
-    <xacro:robotiq_c2_model prefix="right_" parent="right_socket_link">
-        <origin xyz="0 0 -0.02989" rpy="0 1.5708 0"/>
-    </xacro:robotiq_c2_model>-->
-    <xacro:robotiq_arg2f_140 prefix="right_"/>
+    </xacro:macro>
+    <xacro:robot/>
 </robot>
