Commit message: configure les controlleurs et ajoute un monde de test

File: urdf/arm_v2/arm.gazebo.xacro (robot description, xacro)
@@ -12,9 +12,9 @@
     <gazebo reference="${prefix}forearm_upper_link">
       <turnGravityOff>false</turnGravityOff>
-      <selfCollide>false</selfCollide>
+      <selfCollide>true</selfCollide>
     </gazebo>
     <gazebo reference="${prefix}upper_arm_lower_link">
       <turnGravityOff>false</turnGravityOff>
-      <selfCollide>false</selfCollide>
+      <selfCollide>true</selfCollide>
     </gazebo>
     <gazebo reference="${prefix}forearm_lower_link">
@@ -24,5 +24,5 @@
     <gazebo reference="${prefix}wrist_upper_link">
       <turnGravityOff>false</turnGravityOff>
-      <selfCollide>false</selfCollide>
+      <selfCollide>true</selfCollide>
     </gazebo>
     <gazebo reference="${prefix}wrist_lower_link">

File: urdf/arm_v2/arm.transmission.xacro (robot description, xacro)
@@ -1,68 +1,66 @@
 <?xml version="1.0"?>
 <robot xmlns:xacro="http://ros.org/wiki/xacro">
-  <xacro:macro name="sara_arm_transmission_v2" params="prefix">
     <transmission name="${prefix}shoulder_roll_trans" type="SimpleTransmission">
-      <type>transmission_interface/SimpleTransmission</type>
-      <actuator name="${prefix}shoulder_roll_motor">
-        <mechanicalReduction>1</mechanicalReduction>
-      </actuator>
-      <joint name="${prefix}shoulder_roll_joint">
-  	     <hardwareInterface>VelocityJointInterface</hardwareInterface>
-      </joint>
+        <type>transmission_interface/SimpleTransmission</type>
+        <actuator name="${prefix}shoulder_roll_motor">
+            <mechanicalReduction>1</mechanicalReduction>
+        </actuator>
+        <joint name="${prefix}shoulder_roll_joint">
+            <hardwareInterface>hardware_interface/EffortJointInterface</hardwareInterface>
+        </joint>
     </transmission>
     <transmission name="${prefix}shoulder_pitch_trans" type="SimpleTransmission">
-      <type>transmission_interface/SimpleTransmission</type>
-      <actuator name="${prefix}shoulder_pitch_motor">
-  	     <mechanicalReduction>1</mechanicalReduction>
-      </actuator>
-      <joint name="${prefix}shoulder_pitch_joint">
-      	 <hardwareInterface>VelocityJointInterface</hardwareInterface>
-      </joint>
+        <type>transmission_interface/SimpleTransmission</type>
+        <actuator name="${prefix}shoulder_pitch_motor">
+            <mechanicalReduction>1</mechanicalReduction>
+        </actuator>
+        <joint name="${prefix}shoulder_pitch_joint">
+            <hardwareInterface>hardware_interface/EffortJointInterface</hardwareInterface>
+        </joint>
     </transmission>
     <transmission name="${prefix}shoulder_yaw_trans" type="SimpleTransmission">
-      <type>transmission_interface/SimpleTransmission</type>
-      <actuator name="${prefix}shoulder_yaw_motor">
-        <mechanicalReduction>1</mechanicalReduction>
-      </actuator>
-      <joint name="${prefix}shoulder_yaw_joint">
-        <hardwareInterface>VelocityJointInterface</hardwareInterface>
-      </joint>
+        <type>transmission_interface/SimpleTransmission</type>
+        <actuator name="${prefix}shoulder_yaw_motor">
+            <mechanicalReduction>1</mechanicalReduction>
+        </actuator>
+        <joint name="${prefix}shoulder_yaw_joint">
+            <hardwareInterface>hardware_interface/EffortJointInterface</hardwareInterface>
+        </joint>
     </transmission>
     <transmission name="${prefix}elbow_pitch_trans" type="SimpleTransmission">
-      <type>transmission_interface/SimpleTransmission</type>
-      <actuator name="${prefix}elbow_pitch_motor">
-        <mechanicalReduction>1</mechanicalReduction>
-      </actuator>
-      <joint name="${prefix}elbow_pitch_joint">
-        <hardwareInterface>VelocityJointInterface</hardwareInterface>
-      </joint>
+        <type>transmission_interface/SimpleTransmission</type>
+        <actuator name="${prefix}elbow_pitch_motor">
+            <mechanicalReduction>1</mechanicalReduction>
+        </actuator>
+        <joint name="${prefix}elbow_pitch_joint">
+            <hardwareInterface>hardware_interface/EffortJointInterface</hardwareInterface>
+        </joint>
     </transmission>
     <transmission name="${prefix}elbow_yaw_trans" type="SimpleTransmission">
-      <type>transmission_interface/SimpleTransmission</type>
-      <actuator name="${prefix}elbow_yaw_motor">
-   	 <mechanicalReduction>1</mechanicalReduction>
-      </actuator>
-      <joint name="${prefix}elbow_yaw_joint">
-      	 <hardwareInterface>VelocityJointInterface</hardwareInterface>
-      </joint>
+        <type>transmission_interface/SimpleTransmission</type>
+        <actuator name="${prefix}elbow_yaw_motor">
+            <mechanicalReduction>1</mechanicalReduction>
+        </actuator>
+        <joint name="${prefix}elbow_yaw_joint">
+            <hardwareInterface>hardware_interface/EffortJointInterface</hardwareInterface>
+        </joint>
     </transmission>
     <transmission name="${prefix}wrist_pitch_trans" type="SimpleTransmission">
-      <type>transmission_interface/SimpleTransmission</type>
-      <actuator name="${prefix}wrist_pitch_motor">
-      	 <mechanicalReduction>1</mechanicalReduction>
-      </actuator>
-      <joint name="${prefix}wrist_pitch_joint">
-      	 <hardwareInterface>VelocityJointInterface</hardwareInterface>
-      </joint>
+        <type>transmission_interface/SimpleTransmission</type>
+        <actuator name="${prefix}wrist_pitch_motor">
+            <mechanicalReduction>1</mechanicalReduction>
+        </actuator>
+        <joint name="${prefix}wrist_pitch_joint">
+            <hardwareInterface>hardware_interface/EffortJointInterface</hardwareInterface>
+        </joint>
     </transmission>
     <transmission name="${prefix}wrist_roll_trans" type="SimpleTransmission">
-      <type>transmission_interface/SimpleTransmission</type>
-      <actuator name="${prefix}wrist_roll_motor">
-      	 <mechanicalReduction>1</mechanicalReduction>
-      </actuator>
-      <joint name="${prefix}wrist_roll_joint">
-      	 <hardwareInterface>VelocityJointInterface</hardwareInterface>
-      </joint>
+        <type>transmission_interface/SimpleTransmission</type>
+        <actuator name="${prefix}wrist_roll_motor">
+            <mechanicalReduction>1</mechanicalReduction>
+        </actuator>
+        <joint name="${prefix}wrist_roll_joint">
+            <hardwareInterface>hardware_interface/EffortJointInterface</hardwareInterface>
+        </joint>
     </transmission>
-  </xacro:macro>
 </robot>

File: urdf/arm_v2/arm.urdf.xacro (robot description, xacro)
@@ -6,5 +6,7 @@
             <xacro:include filename="$(find sara_description)/urdf/arm_v2/arm.gazebo.xacro"/>
             <xacro:sara_arm_gazebo_v2 prefix="${prefix}"/>
+            <xacro:include filename="$(find sara_description)/urdf/arm_v2/arm.transmission.xacro" />
         </xacro:if>
+<!---->
         <joint name="${prefix}shoulder_roll_joint" type="revolute">
             <parent link="${parent}_link"/>
@@ -230,5 +232,5 @@
         <joint name="${prefix}wrist_roll_joint" type="revolute">
             <parent link="${prefix}wrist_lower_link"/>
-            <child link="${prefix}socket_link"/>
+            <child link="${prefix}last_link"/>
             <dynamics damping="0.1"/>
             <limit effort="10000.0" lower="-1.45" upper="1.45" velocity="1"/>
@@ -236,5 +238,5 @@
             <axis xyz="1 0 0"/>
         </joint>
-        <link name="${prefix}socket_link">
+        <link name="${prefix}last_link">
             <visual>
                 <geometry>
@@ -260,53 +262,10 @@
             </inertial>
         </link>
-        <!-- Robotiq Coupler -->
-        <!--  + Height added by the coupler: 8mm -->
-        <!--  + Reference frame: at the middle (4mm) -->
-        <link name="robotiq_coupler">
-            <visual>
-                <geometry>
-                    <mesh filename="package://robotiq_description/meshes/robotiq_85_coupler.stl"/>
-                </geometry>
-                <material name="flat_black"/>
-            </visual>
-            <collision>
-                <geometry>
-                    <mesh filename="package://robotiq_description/meshes/robotiq_85_coupler.stl"/>
-                </geometry>
-            </collision>
-            <inertial>
-                <origin xyz="2.073e-05   1.45286e-03  -1.1049e-03" rpy="0 0 0"/>
-                <mass value="0.168"/>
-                <inertia ixx="6.69695624e-05" ixy="5.21511788e-09" ixz="-2.74383009e-08"
-                         iyy="7.85088161e-05" iyz="5.41105193e-07" izz="1.41819717e-04"/>
-            </inertial>
-        </link>
-        <joint name="robotiq_coupler_joint" type="fixed">
-            <origin xyz="0 0 -0.07" rpy="0 ${pi} ${-pi/2.0}"/>
-            <parent link="right_socket_link"/>
-            <child link="robotiq_coupler"/>
-        </joint>
-        <gazebo reference="robotiq_coupler">
-            <mu1>0.9</mu1>
-            <mu2>0.9</mu2>
-            <material>Gazebo/FlatBlack</material>
-        </gazebo>
-        <!-- Attach the robotiq 85 gripper -->
-        <xacro:robotiq_85_gripper prefix="" parent="robotiq_coupler">
-            <origin xyz="0 0 0.004" rpy="0 ${-pi/2} ${pi}"/>
-        </xacro:robotiq_85_gripper>
-        <!-- Gazebo grasping plugin -->
-        <gazebo>
-            <gripper name="gazebo_gripper">
-                <grasp_check>
-                    <attach_steps>2</attach_steps>    <!-- default: 20 -->
-                    <detach_steps>2</detach_steps>    <!-- default: 40 -->
-                    <min_contact_count>3</min_contact_count>
-                </grasp_check>
-                <gripper_link>robotiq_85_left_finger_tip_link</gripper_link>
-                <gripper_link>robotiq_85_right_finger_tip_link</gripper_link>
-                <palm_link>robotiq_85_base_link</palm_link>
-            </gripper>
-        </gazebo>
+        <joint name="${prefix}socket_joint" type="fixed">
+            <parent link="${prefix}last_link"/>
+            <child link="${prefix}socket_link"/>
+            <origin xyz="0 0 -0.055" rpy="${PI/2} ${PI/2} 0"/>
+        </joint>
+        <link name="${prefix}socket_link"/>
     </xacro:macro>
 </robot>

File: urdf/base_v2/base.gazebo.xacro (robot description, xacro)
@@ -1,8 +1,10 @@
 <?xml version="1.0"?>
-<robot xmlns:xacro="http://www.ros.org/wiki/xacro">
-   <gazebo reference="chassis">
+<robot xmlns:xacro="http://ros.org/wiki/xacro">
+   <gazebo reference="chassis_link">
       <material>Gazebo/DarkGrey</material>
       <mu1>0.0</mu1>
       <mu2>0.0</mu2>
+      <turnGravityOff>false</turnGravityOff>
+      <selfCollide>true</selfCollide>
    </gazebo>
 </robot>

File: urdf/base_v2/base.urdf.xacro (robot description, xacro)
@@ -6,7 +6,8 @@
       <joint name="base_to_chassis" type="fixed">
           <parent link="${parent}_link"/>
-          <child link="chassis"/>
+          <child link="chassis_link"/>
+          <origin xyz="0 0 0" />
       </joint>
-      <link name="chassis">
+      <link name="chassis_link">
       <inertial>
           <mass value="125.0" />

File: urdf/head_v1/head.gazebo.xacro (robot description, xacro)
@@ -1,4 +1,4 @@
 <?xml version="1.0"?>
-<robot xmlns:xacro="http://www.ros.org/wiki/xacro">
+<robot xmlns:xacro="http://ros.org/wiki/xacro">
    <xacro:macro name="sara_head_gazebo">
       <gazebo reference="head_link">

File: urdf/head_v1/head.transmission.xacro (robot description, xacro)
@@ -1,14 +1,12 @@
 <?xml version="1.0"?>
 <robot xmlns:xacro="http://ros.org/wiki/xacro">
-   <xacro:macro name="sara_head_pitch_transmission_v1">
-      <transmission name="head_pitch_trans" type="SimpleTransmission">
-         <type>transmission_interface/SimpleTransmission</type>
-         <actuator name="head_pitch_motor">
+    <transmission name="head_pitch_trans" type="SimpleTransmission">
+        <type>transmission_interface/SimpleTransmission</type>
+        <actuator name="head_pitch_motor">
             <mechanicalReduction>1</mechanicalReduction>
-         </actuator>
-         <joint name="head_pitch_joint">
-            <hardwareInterface>PositionJointInterface</hardwareInterface>
-         </joint>
-      </transmission>
-   </xacro:macro>
+        </actuator>
+        <joint name="head_pitch_joint">
+            <hardwareInterface>hardware_interface/EffortJointInterface</hardwareInterface>
+        </joint>
+    </transmission>
 </robot>

File: urdf/head_v1/head.urdf.xacro (robot description, xacro)
@@ -1,8 +1,9 @@
 <?xml version="1.0"?>
-<robot xmlns:xacro="http://www.ros.org/wiki/xacro">
+<robot xmlns:xacro="http://ros.org/wiki/xacro">
     <xacro:macro name="sara_head" params="parent *origin sim">
         <xacro:if value="${sim}">
             <xacro:include filename="$(find sara_description)/urdf/head_v1/head.gazebo.xacro"/>
             <xacro:sara_head_gazebo/>
+            <xacro:include filename="$(find sara_description)/urdf/head_v1/head.transmission.xacro" />
         </xacro:if>
         <joint name="head_pitch_joint" type="revolute">
@@ -23,10 +24,4 @@
                 </material>
             </visual>
-            <collision>
-                <geometry>
-                    <mesh filename="package://sara_description/meshes/tete.STL" scale="0.001 0.001 0.001"/>
-                </geometry>
-                <origin xyz="0 0 0" rpy="1.5708 -1.5708 1.5708"/>
-            </collision>
             <inertial>
                 <mass value="2.60401968"/>

File: urdf/head_xtion/head_xtion.gazebo.xacro (robot description, xacro)
@@ -51,9 +51,9 @@
                <pointCloudTopicName>${prefix}xtion/depth/points</pointCloudTopicName>
                <frameName>${prefix}xtion_depth_optical_frame</frameName>
-               <distortion_k1>0.0</distortion_k1>
-               <distortion_k2>0.0</distortion_k2>
-               <distortion_k3>0.0</distortion_k3>
-               <distortion_t1>0.0</distortion_t1>
-               <distortion_t2>0.0</distortion_t2>
+               <distortion_k1>0.1</distortion_k1>
+               <distortion_k2>0.1</distortion_k2>
+               <distortion_k3>0.1</distortion_k3>
+               <distortion_t1>0.1</distortion_t1>
+               <distortion_t2>0.1</distortion_t2>
             </plugin>
          </sensor>

File: urdf/head_xtion/head_xtion.urdf.xacro (robot description, xacro)
@@ -1,4 +1,4 @@
 <?xml version="1.0"?>
-<robot xmlns:xacro="http://www.ros.org/wiki/xacro">
+<robot xmlns:xacro="http://ros.org/wiki/xacro">
     <xacro:property name="M_PI" value="3.1415926535897931"/>
     <xacro:macro name="asus_head_xtion" params="prefix parent *origin sim">

File: urdf/hokuyo/hokuyo.gazebo.xacro (robot description, xacro)
@@ -1,4 +1,4 @@
 <?xml version="1.0"?>
-<robot xmlns:xacro="http://www.ros.org/wiki/xacro">
+<robot xmlns:xacro="http://ros.org/wiki/xacro">
     <xacro:macro name="hokuyo_gazebo" params="prefix">
         <!-- hokuyo -->
@@ -19,5 +19,5 @@
                     </scan>
                     <range>
-                        <min>0.26</min>
+                        <min>0.28</min>
                         <max>10.0</max>
                         <resolution>0.01</resolution>

File: urdf/hokuyo/hokuyo.urdf.xacro (robot description, xacro)
@@ -1,4 +1,4 @@
 <?xml version="1.0"?>
-<robot xmlns:xacro="http://www.ros.org/wiki/xacro">
+<robot xmlns:xacro="http://ros.org/wiki/xacro">
     <xacro:macro name="hokuyo" params="prefix parent *origin sim">
         <xacro:if value="${sim}">

File: urdf/linear_actuator_v1/actuator.gazebo.xacro (robot description, xacro)
@@ -1,8 +1,8 @@
 <?xml version="1.0"?>
-<robot xmlns:xacro="http://www.ros.org/wiki/xacro">
+<robot xmlns:xacro="http://ros.org/wiki/xacro">
     <xacro:macro name="sara_linear_actuator_gazebo" params="prefix">
         <gazebo reference="${prefix}actuator_link">
             <turnGravityOff>false</turnGravityOff>
-            <selfCollide>true</selfCollide>
+            <selfCollide>false</selfCollide>
         </gazebo>
     </xacro:macro>

File: urdf/linear_actuator_v1/actuator.transmission.xacro (robot description, xacro)
@@ -1,68 +1,12 @@
 <?xml version="1.0"?>
 <robot xmlns:xacro="http://ros.org/wiki/xacro">
-  <xacro:macro name="sara_arm_transmission_v2" params="prefix">
-    <transmission name="${prefix}shoulder_roll_trans" type="SimpleTransmission">
-      <type>transmission_interface/SimpleTransmission</type>
-      <actuator name="${prefix}shoulder_roll_motor">
-        <mechanicalReduction>1</mechanicalReduction>
-      </actuator>
-      <joint name="${prefix}shoulder_roll_joint">
-  	     <hardwareInterface>VelocityJointInterface</hardwareInterface>
-      </joint>
+    <transmission name="${prefix}_actuator_trans" type="SimpleTransmission">
+        <type>transmission_interface/SimpleTransmission</type>
+        <actuator name="${prefix}_actuator_motor">
+            <mechanicalReduction>1</mechanicalReduction>
+        </actuator>
+        <joint name="${prefix}_actuator_joint">
+            <hardwareInterface>hardware_interface/EffortJointInterface</hardwareInterface>
+        </joint>
     </transmission>
-    <transmission name="${prefix}shoulder_pitch_trans" type="SimpleTransmission">
-      <type>transmission_interface/SimpleTransmission</type>
-      <actuator name="${prefix}shoulder_pitch_motor">
-  	     <mechanicalReduction>1</mechanicalReduction>
-      </actuator>
-      <joint name="${prefix}shoulder_pitch_joint">
-      	 <hardwareInterface>VelocityJointInterface</hardwareInterface>
-      </joint>
-    </transmission>
-    <transmission name="${prefix}shoulder_yaw_trans" type="SimpleTransmission">
-      <type>transmission_interface/SimpleTransmission</type>
-      <actuator name="${prefix}shoulder_yaw_motor">
-        <mechanicalReduction>1</mechanicalReduction>
-      </actuator>
-      <joint name="${prefix}shoulder_yaw_joint">
-        <hardwareInterface>VelocityJointInterface</hardwareInterface>
-      </joint>
-    </transmission>
-    <transmission name="${prefix}elbow_pitch_trans" type="SimpleTransmission">
-      <type>transmission_interface/SimpleTransmission</type>
-      <actuator name="${prefix}elbow_pitch_motor">
-        <mechanicalReduction>1</mechanicalReduction>
-      </actuator>
-      <joint name="${prefix}elbow_pitch_joint">
-        <hardwareInterface>VelocityJointInterface</hardwareInterface>
-      </joint>
-    </transmission>
-    <transmission name="${prefix}elbow_yaw_trans" type="SimpleTransmission">
-      <type>transmission_interface/SimpleTransmission</type>
-      <actuator name="${prefix}elbow_yaw_motor">
-   	 <mechanicalReduction>1</mechanicalReduction>
-      </actuator>
-      <joint name="${prefix}elbow_yaw_joint">
-      	 <hardwareInterface>VelocityJointInterface</hardwareInterface>
-      </joint>
-    </transmission>
-    <transmission name="${prefix}wrist_pitch_trans" type="SimpleTransmission">
-      <type>transmission_interface/SimpleTransmission</type>
-      <actuator name="${prefix}wrist_pitch_motor">
-      	 <mechanicalReduction>1</mechanicalReduction>
-      </actuator>
-      <joint name="${prefix}wrist_pitch_joint">
-      	 <hardwareInterface>VelocityJointInterface</hardwareInterface>
-      </joint>
-    </transmission>
-    <transmission name="${prefix}wrist_roll_trans" type="SimpleTransmission">
-      <type>transmission_interface/SimpleTransmission</type>
-      <actuator name="${prefix}wrist_roll_motor">
-      	 <mechanicalReduction>1</mechanicalReduction>
-      </actuator>
-      <joint name="${prefix}wrist_roll_joint">
-      	 <hardwareInterface>VelocityJointInterface</hardwareInterface>
-      </joint>
-    </transmission>
-  </xacro:macro>
 </robot>

File: urdf/linear_actuator_v1/actuator.urdf.xacro (robot description, xacro)
@@ -1,4 +1,4 @@
 <?xml version="1.0"?>
-<robot xmlns:xacro="http://www.ros.org/wiki/xacro">
+<robot xmlns:xacro="http://ros.org/wiki/xacro">
     <xacro:macro name="sara_linear_actuator" params="prefix parent *origin sim">
         <xacro:if value="${sim}">
@@ -6,5 +6,6 @@
             <xacro:sara_linear_actuator_gazebo prefix="${prefix}"/>
         </xacro:if>
-        <joint name="${parent}_actuator_joint" type="prismatic">
+        <xacro:include filename="$(find sara_description)/urdf/linear_actuator_v1/actuator.transmission.xacro" />
+        <joint name="${prefix}_actuator_joint" type="prismatic">
             <parent link="${parent}_link"/>
             <child link="actuator_link"/>

File: urdf/neck_v1/neck.gazebo.xacro (robot description, xacro)
@@ -1,6 +1,6 @@
 <?xml version="1.0"?>
-<robot xmlns:xacro="http://www.ros.org/wiki/xacro">
+<robot xmlns:xacro="http://ros.org/wiki/xacro">
    <xacro:macro name="sara_neck_gazebo">
-      <gazebo reference="neck_link">
+      <gazebo reference="neck_linke">
          <turnGravityOff>false</turnGravityOff>
          <selfCollide>false</selfCollide>

File: urdf/neck_v1/neck.transmission.xacro (robot description, xacro)
@@ -1,14 +1,12 @@
 <?xml version="1.0"?>
 <robot xmlns:xacro="http://ros.org/wiki/xacro">
-   <xacro:macro name="sara_head_yaw_transmission_v1">
-      <transmission name="head_yaw_trans" type="SimpleTransmission">
-         <type>transmission_interface/SimpleTransmission</type>
-         <actuator name="head_yaw_motor">
+    <transmission name="head_yaw_trans" type="SimpleTransmission">
+        <type>transmission_interface/SimpleTransmission</type>
+        <actuator name="head_yaw_motor">
             <mechanicalReduction>1</mechanicalReduction>
-         </actuator>
-         <joint name="head_yaw_joint">
-            <hardwareInterface>PositionJointInterface</hardwareInterface>
-         </joint>
-      </transmission>
-   </xacro:macro>
+        </actuator>
+        <joint name="head_yaw_joint">
+            <hardwareInterface>hardware_interface/EffortJointInterface</hardwareInterface>
+        </joint>
+    </transmission>
 </robot>

File: urdf/neck_v1/neck.urdf.xacro (robot description, xacro)
@@ -1,8 +1,9 @@
 <?xml version="1.0"?>
-<robot xmlns:xacro="http://www.ros.org/wiki/xacro">
+<robot xmlns:xacro="http://ros.org/wiki/xacro">
     <xacro:macro name="sara_neck" params="parent *origin sim">
         <xacro:if value="${sim}">
             <xacro:include filename="$(find sara_description)/urdf/neck_v1/neck.gazebo.xacro"/>
             <xacro:sara_neck_gazebo/>
+            <xacro:include filename="$(find sara_description)/urdf/neck_v1/neck.transmission.xacro" />
         </xacro:if>
         <joint name="head_yaw_joint" type="revolute">
@@ -23,10 +24,4 @@
                 </material>
             </visual>
-            <collision>
-                <geometry>
-                    <mesh filename="package://sara_description/meshes/couV2.STL" scale="0.001 0.001 0.001"/>
-                </geometry>
-                <origin xyz="0 0 0" rpy="1.5708 0 1.5708"/>
-            </collision>
             <inertial>
                 <mass value="2"/>
