Commit message: configure les controlleurs et ajoute un monde de test

File: urdf/sara.gazebo.xacro (robot description, xacro)
@@ -1,10 +1,12 @@
 <?xml version="1.0"?>
-<robot>
+<robot xmlns:xacro="http://ros.org/wiki/xacro">
+   <xacro:macro name="sara_gazebo">
       <gazebo>
          <static>false</static>
          <plugin name="gazebo_ros_control" filename="libgazebo_ros_control.so">
-            <robotNamespace>/sara_simulation</robotNamespace>
+            <robotNamespace>/</robotNamespace>
+            <controlPeriod>0.002</controlPeriod>
             <robotSimType>gazebo_ros_control/DefaultRobotHWSim</robotSimType>
-            <legacyModeNS>false</legacyModeNS>
+            <legacyModeNS>true</legacyModeNS>
          </plugin>
          <plugin name="ridgeback_ros_force_based_move" filename="libridgeback_ros_force_based_move.so">
@@ -23,3 +25,4 @@
          </plugin>
       </gazebo>
+   </xacro:macro>
 </robot>

File: urdf/sara.urdf.xacro (robot description, xacro)
@@ -4,4 +4,6 @@
     <xacro:arg name="sim" default="true"/>
     <xacro:property name="sim" value="$(arg sim)"/>
+    <xacro:arg name="ns" default="/"/>
+    <xacro:property name="ns" value="$(arg ns)"/>
     <xacro:include filename="$(find sara_description)/urdf/linear_actuator_v1/actuator.urdf.xacro"/>
     <xacro:include filename="$(find sara_description)/urdf/torso_v1/torso.urdf.xacro"/>
@@ -12,10 +14,19 @@
     <xacro:include filename="$(find sara_description)/urdf/base_v2/base.urdf.xacro"/>
     <xacro:include filename="$(find sara_description)/urdf/hokuyo/hokuyo.urdf.xacro"/>
+    <xacro:include filename="$(find sara_description)/robotiq_2f_85/urdf/robotiq_2f_85_macro.xacro" />
     <link name="base_link"></link>
     <!-- Base -->
     <xacro:sara_base parent="base"/>
+    <!-- hokuyo -->
+    <xacro:hokuyo prefix="front_" parent="chassis" sim="${sim}">
+        <origin xyz="0.2516879 0 -0.005" rpy="0 0 0" />
+    </xacro:hokuyo>
+    <!-- Linear Actuator -->
+    <xacro:sara_linear_actuator prefix="front" parent="chassis" sim="${sim}">
+        <origin xyz="0 0 0.1" rpy="0 0 0" />
+    </xacro:sara_linear_actuator>
     <!-- Torso -->
-    <xacro:sara_torso parent="base" sim="${sim}">
-        <origin xyz="0.1999806 0 1.189" rpy="0 0 0" />
+    <xacro:sara_torso parent="actuator" sim="${sim}">
+        <origin xyz="0.1999806 0 0.5256" rpy="0 0 0" />
     </xacro:sara_torso>
     <!-- Neck -->
@@ -25,5 +36,5 @@
     <!-- Head -->
     <xacro:sara_head parent="neck" sim="${sim}">
-        <origin xyz="0 0 0.0927" rpy="-1.57 0 0"/>
+        <origin xyz="0 0 0.0927" rpy="${-PI/2} 0 0"/>
     </xacro:sara_head>
     <!-- Head Xtion -->
@@ -33,7 +44,17 @@
     <!-- Arm -->
     <xacro:sara_arm prefix="right_" parent="torso" sim="${sim}">
-        <origin xyz="0 -0.1437625 0.01166" rpy="0 -1.57 0"/>
+        <origin xyz="0 -0.1437625 0.01166" rpy="0 ${-PI/2} 0"/>
     </xacro:sara_arm>
+    <!-- Gripper -->
+    <xacro:load_gripper parent="right_socket_link">
+        <origin xyz="0 0 0" rpy="0 0 0"/>
+    </xacro:load_gripper>
+    <!-- Gripper physic -->
+    <xacro:if value="${sim}">
+        <xacro:include filename="$(find sara_description)/robotiq_2f_85/urdf/robotiq_2f_85_transmission_macro.xacro" />
+        <xacro:load_gazebo_gripper_transmissions/>
+    </xacro:if>
     <!-- Bring in simulation data for Gazebo. -->
     <xacro:include filename="$(find sara_description)/urdf/sara.gazebo.xacro" />
+    <xacro:sara_gazebo/>
 </robot>
