Commit message: Ajoute les librairies tiers pour les doigts

File: description/robotiq_2f_85/urdf/robotiq_2f_85_macro.xacro (robot description, xacro)
@@ -11,10 +11,10 @@
             <visual>
                 <geometry>
-                    <mesh filename="package://kortex_description/grippers/robotiq_2f_85/meshes/visual/robotiq_85_base_link.dae"/>
-                </geometry>
-            </visual>
-            <collision>
-                <geometry>
-                    <mesh filename="package://kortex_description/grippers/robotiq_2f_85/meshes/collision/robotiq_85_base_link.stl"/>
+                    <mesh filename="package://sara_description/robotiq_2f_85/meshes/visual/robotiq_85_base_link.dae"/>
+                </geometry>
+            </visual>
+            <collision>
+                <geometry>
+                    <mesh filename="package://sara_description/robotiq_2f_85/meshes/collision/robotiq_85_base_link.stl"/>
                 </geometry>
             </collision>
@@ -52,10 +52,10 @@
             <visual>
                 <geometry>
-                    <mesh filename="package://kortex_description/grippers/robotiq_2f_85/meshes/visual/robotiq_85_knuckle_link.dae"/>
-                </geometry>
-            </visual>
-            <collision>
-                <geometry>
-                    <mesh filename="package://kortex_description/grippers/robotiq_2f_85/meshes/collision/robotiq_85_knuckle_link.stl"/>
+                    <mesh filename="package://sara_description/robotiq_2f_85/meshes/visual/robotiq_85_knuckle_link.dae"/>
+                </geometry>
+            </visual>
+            <collision>
+                <geometry>
+                    <mesh filename="package://sara_description/robotiq_2f_85/meshes/collision/robotiq_85_knuckle_link.stl"/>
                 </geometry>
             </collision>
@@ -78,10 +78,10 @@
             <visual>
                 <geometry>
-                    <mesh filename="package://kortex_description/grippers/robotiq_2f_85/meshes/visual/robotiq_85_knuckle_link.dae"/>
-                </geometry>
-            </visual>
-            <collision>
-                <geometry>
-                    <mesh filename="package://kortex_description/grippers/robotiq_2f_85/meshes/collision/robotiq_85_knuckle_link.stl"/>
+                    <mesh filename="package://sara_description/robotiq_2f_85/meshes/visual/robotiq_85_knuckle_link.dae"/>
+                </geometry>
+            </visual>
+            <collision>
+                <geometry>
+                    <mesh filename="package://sara_description/robotiq_2f_85/meshes/collision/robotiq_85_knuckle_link.stl"/>
                 </geometry>
             </collision>
@@ -114,10 +114,10 @@
             <visual>
                 <geometry>
-                    <mesh filename="package://kortex_description/grippers/robotiq_2f_85/meshes/visual/robotiq_85_finger_link.dae"/>
-                </geometry>
-            </visual>
-            <collision>
-                <geometry>
-                    <mesh filename="package://kortex_description/grippers/robotiq_2f_85/meshes/collision/robotiq_85_finger_link.stl"/>
+                    <mesh filename="package://sara_description/robotiq_2f_85/meshes/visual/robotiq_85_finger_link.dae"/>
+                </geometry>
+            </visual>
+            <collision>
+                <geometry>
+                    <mesh filename="package://sara_description/robotiq_2f_85/meshes/collision/robotiq_85_finger_link.stl"/>
                 </geometry>
             </collision>
@@ -140,10 +140,10 @@
             <visual>
                 <geometry>
-                    <mesh filename="package://kortex_description/grippers/robotiq_2f_85/meshes/visual/robotiq_85_finger_link.dae"/>
-                </geometry>
-            </visual>
-            <collision>
-                <geometry>
-                    <mesh filename="package://kortex_description/grippers/robotiq_2f_85/meshes/collision/robotiq_85_finger_link.stl"/>
+                    <mesh filename="package://sara_description/robotiq_2f_85/meshes/visual/robotiq_85_finger_link.dae"/>
+                </geometry>
+            </visual>
+            <collision>
+                <geometry>
+                    <mesh filename="package://sara_description/robotiq_2f_85/meshes/collision/robotiq_85_finger_link.stl"/>
                 </geometry>
             </collision>
@@ -182,10 +182,10 @@
             <visual>
                 <geometry>
-                    <mesh filename="package://kortex_description/grippers/robotiq_2f_85/meshes/visual/robotiq_85_inner_knuckle_link.dae"/>
-                </geometry>
-            </visual>
-            <collision>
-                <geometry>
-                    <mesh filename="package://kortex_description/grippers/robotiq_2f_85/meshes/collision/robotiq_85_inner_knuckle_link.stl"/>
+                    <mesh filename="package://sara_description/robotiq_2f_85/meshes/visual/robotiq_85_inner_knuckle_link.dae"/>
+                </geometry>
+            </visual>
+            <collision>
+                <geometry>
+                    <mesh filename="package://sara_description/robotiq_2f_85/meshes/collision/robotiq_85_inner_knuckle_link.stl"/>
                 </geometry>
             </collision>
@@ -208,10 +208,10 @@
             <visual>
                 <geometry>
-                    <mesh filename="package://kortex_description/grippers/robotiq_2f_85/meshes/visual/robotiq_85_inner_knuckle_link.dae"/>
-                </geometry>
-            </visual>
-            <collision>
-                <geometry>
-                    <mesh filename="package://kortex_description/grippers/robotiq_2f_85/meshes/collision/robotiq_85_inner_knuckle_link.stl"/>
+                    <mesh filename="package://sara_description/robotiq_2f_85/meshes/visual/robotiq_85_inner_knuckle_link.dae"/>
+                </geometry>
+            </visual>
+            <collision>
+                <geometry>
+                    <mesh filename="package://sara_description/robotiq_2f_85/meshes/collision/robotiq_85_inner_knuckle_link.stl"/>
                 </geometry>
             </collision>
@@ -250,10 +250,10 @@
             <visual>
                 <geometry>
-                    <mesh filename="package://kortex_description/grippers/robotiq_2f_85/meshes/visual/robotiq_85_finger_tip_link.dae"/>
-                </geometry>
-            </visual>
-            <collision>
-                <geometry>
-                    <mesh filename="package://kortex_description/grippers/robotiq_2f_85/meshes/collision/robotiq_85_finger_tip_link.stl"/>
+                    <mesh filename="package://sara_description/robotiq_2f_85/meshes/visual/robotiq_85_finger_tip_link.dae"/>
+                </geometry>
+            </visual>
+            <collision>
+                <geometry>
+                    <mesh filename="package://sara_description/robotiq_2f_85/meshes/collision/robotiq_85_finger_tip_link.stl"/>
                 </geometry>
             </collision>
@@ -276,10 +276,10 @@
             <visual>
                 <geometry>
-                    <mesh filename="package://kortex_description/grippers/robotiq_2f_85/meshes/visual/robotiq_85_finger_tip_link.dae"/>
-                </geometry>
-            </visual>
-            <collision>
-                <geometry>
-                    <mesh filename="package://kortex_description/grippers/robotiq_2f_85/meshes/collision/robotiq_85_finger_tip_link.stl"/>
+                    <mesh filename="package://sara_description/robotiq_2f_85/meshes/visual/robotiq_85_finger_tip_link.dae"/>
+                </geometry>
+            </visual>
+            <collision>
+                <geometry>
+                    <mesh filename="package://sara_description/robotiq_2f_85/meshes/collision/robotiq_85_finger_tip_link.stl"/>
                 </geometry>
             </collision>
